File: sheets/10_power_input.kicad_sch (KiCad schematic)
At the start: 36 parts, among them J1 MSTB 2,5/5-GF-5,08, J2 MSTB 2,5/2-GF-5,08, Q101 STD18NF25, Q102 IPD30N10S3L-34, U101 LM74930QRGERQ1

Commit message: fixed and review
Parts:
- F101: footprint (none) -> INCLI-VA:FUSE-SMD_L6.1-W2.5-1
- J1: footprint Connector_Phoenix_MSTB:PhoenixContact_MSTB_2,5_5-GF-5,08_1x05_P5.08mm_Horizontal_ThreadedFlange -> Connector_Phoenix_MC:PhoenixContact_MCV_1,5_5-GF-3.81_1x05_P3.81mm_Vertical_ThreadedFlange
- J2: footprint Connector_Phoenix_MSTB:PhoenixContact_MSTB_2,5_2-GF-5,08_1x02_P5.08mm_Horizontal_ThreadedFlange -> Connector_Phoenix_MC:PhoenixContact_MCV_1,5_2-GF-3.81_1x02_P3.81mm_Vertical_ThreadedFlange
Changed lines of the file:
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@@
 			)
 		)
-		(property "Footprint" ""
+		(property "Footprint" "INCLI-VA:FUSE-SMD_L6.1-W2.5-1"
 			(at 123.19 76.2 0)
 			(hide yes)
@@
 			)
 		)
-		(property "Datasheet" ""
+		(property "Datasheet" "https://www.lcsc.com/datasheet/C3159902.pdf"
 			(at 123.19 76.2 0)
 			(hide yes)
@@
 			)
 		)
-		(property "Footprint" "Connector_Phoenix_MSTB:PhoenixContact_MSTB_2,5_5-GF-5,08_1x05_P5.08mm_Horizontal_ThreadedFlange"
+		(property "Footprint" "Connector_Phoenix_MC:PhoenixContact_MCV_1,5_5-GF-3.81_1x05_P3.81mm_Vertical_ThreadedFlange"
 			(at 100.33 81.28 0)
 			(hide yes)
@@
 			)
 		)
-		(property "Footprint" "Connector_Phoenix_MSTB:PhoenixContact_MSTB_2,5_2-GF-5,08_1x02_P5.08mm_Horizontal_ThreadedFlange"
+		(property "Footprint" "Connector_Phoenix_MC:PhoenixContact_MCV_1,5_2-GF-3.81_1x02_P3.81mm_Vertical_ThreadedFlange"
 			(at 100.33 114.3 0)
 			(hide yes)
