File: sheets/10_power_input.kicad_sch (KiCad schematic)
At the start: 36 parts, among them J1 MSTBV 2,5/5-GF-5,08, J2 MSTBV 2,5/2-GF-5,08, Q101 STD18NF25, Q102 IPD30N10S3L-34, U101 LM74930QRGERQ1

Commit message: [Claude Code] PCB: placement-v1 - desacoples de U601, lazo del buck, C105 J16 Panasonic y zonas sin barniz
- C601 a 1.1 mm del pin VIO (ADI Rev. D: pista <= 2 mm); C604, C607/C608 reordenados.
- L201 y C203 mas cerca de U201 (SW 2.8 mm, BOOT 1.1 mm).
- C105: huella INCLI-VA:CP_Elec_Panasonic_J16_VibProof (land antivibracion J16, acepta
  EEE-FK1H102AV y EEE-FK1H102AM); MPN PROD EEE-FK1H102AV.
- Coating: zonas a enmascarar en User.Comments y rotulo "SIN BARNIZ".
- PENDIENTES: decisiones del usuario cerradas, requisitos de la caja y plan de ruteo.
- DRC 0 errores, paridad 0. ERC sin cambios.

Co-Authored-By: Claude Opus 5.5 <noreply@anthropic.com>
Parts:
- C105: footprint Capacitor_SMD:CP_Elec_16x17.5 -> INCLI-VA:CP_Elec_Panasonic_J16_VibProof; Alt_MPN EEE-FK1H102AV -> EEE-FK1H102AM; MPN EEE-FK1H102AM -> EEE-FK1H102AV; Notes Hold-up: DNP en PROTO, montado en PROD (load dump suprimido de 24 V <= 350 ms y arranque en frio de 12 V). Panasonic serie FK, AEC-Q200, 1000 uF / 50 V, 105 C, cuerpo 16 x 16.5 mm, 2 terminales: FIJAR CON ADHESIVO (vibracion). Alt_MPN EEE-FK1H102AV (FK antivibracion, 30 G) requiere su land pattern con terminales de anclaje: no se pudo verificar (datasheet Panasonic no accesible). Verificar el land pattern J16 contra CP_Elec_16x17.5 antes de produccion. Requiere C109 = 100 nF (inrush). -> Hold-up: DNP en PROTO, montado en PROD (load dump suprimido de 24 V <= 350 ms y arranque en frio de 12 V). PROD: EEE-FK1H102AV, Panasonic FK antivibracion (terminales de soporte), AEC-Q200, 1000 uF / 50 V, 105 C, J16 (16 x 16.8 mm, altura max. 17.3 mm). Huella INCLI-VA:CP_Elec_Panasonic_J16_VibProof = land antivibracion J16 de Panasonic (FK, 01-Sep-25); su columna central contiene el land estandar J16, asi que EEE-FK1H102AM (Alt_MPN, sin soporte: fijar con adhesivo) entra en la misma huella. Disponibilidad del AV a verificar. Requiere C109 = 100 nF (inrush).
Changed lines of the file:
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@@
 			)
 		)
-		(property "Footprint" "Capacitor_SMD:CP_Elec_16x17.5"
+		(property "Footprint" "INCLI-VA:CP_Elec_Panasonic_J16_VibProof"
 			(at 252.73 80.01 0)
 			(hide yes)
@@
 			)
 		)
-		(property "Datasheet" "https://www.mouser.com/ProductDetail/Panasonic/EEE-FK1H102AM"
+		(property "Datasheet" "https://industrial.panasonic.com/cdbs/www-data/pdf/RDE0000/ABA0000C1181.pdf"
 			(at 252.73 80.01 0)
 			(hide yes)
@@
 			)
 		)
-		(property "MPN" "EEE-FK1H102AM"
+		(property "MPN" "EEE-FK1H102AV"
 			(at 252.73 80.01 0)
 			(hide yes)
@@
 			)
 		)
-		(property "Notes" "Hold-up: DNP en PROTO, montado en PROD (load dump suprimido de 24 V <= 350 ms y arranque en frio de 12 V). Panasonic serie FK, AEC-Q200, 1000 uF / 50 V, 105 C, cuerpo 16 x 16.5 mm, 2 terminales: FIJAR CON ADHESIVO (vibracion). Alt_MPN EEE-FK1H102AV (FK antivibracion, 30 G) requiere su land pattern con terminales de anclaje: no se pudo verificar (datasheet Panasonic no accesible). Verificar el land pattern J16 contra CP_Elec_16x17.5 antes de produccion. Requiere C109 = 100 nF (inrush)."
+		(property "Notes" "Hold-up: DNP en PROTO, montado en PROD (load dump suprimido de 24 V <= 350 ms y arranque en frio de 12 V). PROD: EEE-FK1H102AV, Panasonic FK antivibracion (terminales de soporte), AEC-Q200, 1000 uF / 50 V, 105 C, J16 (16 x 16.8 mm, altura max. 17.3 mm). Huella INCLI-VA:CP_Elec_Panasonic_J16_VibProof = land antivibracion J16 de Panasonic (FK, 01-Sep-25); su columna central contiene el land estandar J16, asi que EEE-FK1H102AM (Alt_MPN, sin soporte: fijar con adhesivo) entra en la misma huella. Disponibilidad del AV a verificar. Requiere C109 = 100 nF (inrush)."
 			(at 252.73 80.01 0)
 			(hide yes)
@@
 			)
 		)
-		(property "Alt_MPN" "EEE-FK1H102AV"
+		(property "Alt_MPN" "EEE-FK1H102AM"
 			(at 252.73 80.01 0)
 			(hide yes)

Commit message: [Claude Code] esquema+PCB: campos LCSC y sustitutos PROTO del BOM (pcb-v1-rc2)
- Esquema (solo campos, ocultos): LCSC en todos los componentes; MPN_PROTO,
  LCSC_PROTO y Manufacturer_PROTO con los sustitutos aceptados; Notes con
  compra y montaje (Q101, Q102, F101, L201, U503 a mano desde DigiKey/Mouser).
  MPN (PROD), valores, huellas y conexiones sin cambios. LCSC Part -> LCSC.
- PCB: mismos campos en las 145 huellas, insertados como texto (equivalente
  a F8 solo para campos); nada cambia fuera de las huellas.
- ERC por hoja igual que antes (0 errores, 5 avisos). DRC 0 errores / 3 avisos
  aceptados, 0 sin rutear, paridad 0 (antes de sincronizar: 145).
- etapa6_fab.py usa los campos _PROTO y genera bom_jlc_lcsc.csv; este y
  cpl_jlc.csv salen idénticos (60 líneas, 123 piezas). Gerbers sin cambios
  de contenido.

Co-Authored-By: Claude Opus 5.5 <noreply@anthropic.com>
Parts:
- C101: LCSC (none) -> C3887150; LCSC_PROTO (none) -> C106025; MPN_PROTO (none) -> C1206X104K451T; Manufacturer_PROTO (none) -> IHHEC; Notes 1206 / 450 V: C_IN en VBAT_F, ve hasta 202 V. MPN a verificar (disponibilidad y especificación) antes de congelar el BOM. -> 1206 / 450 V: C_IN en VBAT_F, ve hasta 202 V. MPN a verificar (disponibilidad y especificación) antes de congelar el BOM. PROTO (2026-10-30): IHHEC C1206X104K451T (LCSC C106025), sin AEC-Q200, solo para el prototipo. PROD: este MPN (AEC-Q200); sin stock en JLC/LCSC, comprar en DigiKey/Mouser.
- C102: LCSC (none) -> C2168321; LCSC_PROTO (none) -> C13832; MPN_PROTO (none) -> CL31B105KCHNNNE; Manufacturer_PROTO (none) -> Samsung; Notes C_VS >= 1 uF (ref. TI). 1206 por 100 V. MPN a verificar (disponibilidad y especificación) antes de congelar el BOM. -> C_VS >= 1 uF (ref. TI). 1206 por 100 V. MPN a verificar (disponibilidad y especificación) antes de congelar el BOM. PROTO (2026-10-30): Samsung CL31B105KCHNNNE (LCSC C13832, JLC extended), misma especificación, sin AEC-Q200.
- C103: LCSC (none) -> C2168321; LCSC_PROTO (none) -> C13832; MPN_PROTO (none) -> CL31B105KCHNNNE; Manufacturer_PROTO (none) -> Samsung; Notes C_CS (ref. TI). 1206 por 100 V. MPN a verificar (disponibilidad y especificación) antes de congelar el BOM. -> C_CS (ref. TI). 1206 por 100 V. MPN a verificar (disponibilidad y especificación) antes de congelar el BOM. PROTO (2026-10-30): Samsung CL31B105KCHNNNE (LCSC C13832, JLC extended), misma especificación, sin AEC-Q200.
- C104: LCSC (none) -> C344077; LCSC_PROTO (none) -> C164068; MPN_PROTO (none) -> VZH470M2ATR-1010; Manufacturer_PROTO (none) -> Lelon; Notes C_OUT (ex C3). 100 V 105 C AEC-Q200. LCSC C344077. -> C_OUT (ex C3). 100 V 105 C AEC-Q200. LCSC C344077. PROTO (2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
- C105: LCSC (none) -> C2164039; Notes Hold-up: DNP en PROTO, montado en PROD (load dump suprimido de 24 V <= 350 ms y arranque en frio de 12 V). PROD: EEE-FK1H102AV, Panasonic FK antivibracion (terminales de soporte), AEC-Q200, 1000 uF / 50 V, 105 C, J16 (16 x 16.8 mm, altura max. 17.3 mm). Huella INCLI-VA:CP_Elec_Panasonic_J16_VibProof = land antivibracion J16 de Panasonic (FK, 01-Sep-25); su columna central contiene el land estandar J16, asi que EEE-FK1H102AM (Alt_MPN, sin soporte: fijar con adhesivo) entra en la misma huella. Disponibilidad del AV a verificar. Requiere C109 = 100 nF (inrush). -> Hold-up: DNP en PROTO, montado en PROD (load dump suprimido de 24 V <= 350 ms y arranque en frio de 12 V). PROD: EEE-FK1H102AV, Panasonic FK antivibracion (terminales de soporte), AEC-Q200, 1000 uF / 50 V, 105 C, J16 (16 x 16.8 mm, altura max. 17.3 mm). Huella INCLI-VA:CP_Elec_Panasonic_J16_VibProof = land antivibracion J16 de Panasonic (FK, 01-Sep-25); su columna central contiene el land estandar J16, asi que EEE-FK1H102AM (Alt_MPN, sin soporte: fijar con adhesivo) entra en la misma huella. Disponibilidad del AV a verificar. Requiere C109 = 100 nF (inrush). PROD (2026-10-30): sin stock suficiente en JLC/LCSC para 100 placas; comprar en DigiKey/Mouser.
- C106: LCSC_PROTO (none) -> C138687; MPN_PROTO (none) -> CL32B106KBJNNNE; Manufacturer_PROTO (none) -> Samsung; Notes 1210: 10 uF / 50 V en +VPROT (<= 40 V). MPN a verificar (disponibilidad y especificación) antes de congelar el BOM. -> 1210: 10 uF / 50 V en +VPROT (<= 40 V). MPN a verificar (disponibilidad y especificación) antes de congelar el BOM. PROTO (2026-10-30): Samsung CL32B106KBJNNNE (LCSC C138687, JLC extended), misma especificación, sin AEC-Q200.
- C107, C109: LCSC (none) -> C415406
- C108: LCSC (none) -> C85864; LCSC_PROTO (none) -> C14663; MPN_PROTO (none) -> CC0603KRX7R9BB104; Manufacturer_PROTO (none) -> Yageo; Notes C_CAP entre CAP y VS (bomba de carga). -> C_CAP entre CAP y VS (bomba de carga). PROTO (2026-10-30): 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
- C110: LCSC (none) -> C380380; LCSC_PROTO (none) -> C31658; MPN_PROTO (none) -> CL10B683KB8NNNC; Manufacturer_PROTO (none) -> Samsung; Notes C_TMR: breaker ~1 ms, reintento ~1.5 s. MPN a verificar (disponibilidad y especificación) antes de congelar el BOM. -> C_TMR: breaker ~1 ms, reintento ~1.5 s. MPN a verificar (disponibilidad y especificación) antes de congelar el BOM. PROTO (2026-10-30): Samsung CL10B683KB8NNNC (LCSC C31658, JLC preferred), misma especificación, sin AEC-Q200.
- D101: LCSC (none) -> C2927419
- D102: LCSC (none) -> C438109
- D103: LCSC (none) -> C366557
- D104: LCSC (none) -> C8661
- F101: LCSC (none) -> C3159902; Notes Bourns SF-2410FPA200W-2: 2 A rapido, 250 VDC, AEC-Q200 (LCSC C3159902). Fusible de falla grave: el breaker del LM74930 actua antes (1 A). Huella INCLI-VA:Fuse_Bourns_SF-2410 segun el 'Recommended Pad Layout' de Bourns (pads 2.8 x 3.15 mm, separacion 3.0 mm). -> Bourns SF-2410FPA200W-2: 2 A rapido, 250 VDC, AEC-Q200 (LCSC C3159902). Fusible de falla grave: el breaker del LM74930 actua antes (1 A). Huella INCLI-VA:Fuse_Bourns_SF-2410 segun el 'Recommended Pad Layout' de Bourns (pads 2.8 x 3.15 mm, separacion 3.0 mm). Compra (2026-10-30): sin stock en JLC/LCSC; comprar en DigiKey/Mouser y soldar a mano (PROTO y PROD). Sustituto rechazado: protección de entrada, el prototipo valida el diseño de producción.
- J1: LCSC (none) -> C7164734; Notes Header vertical MSTBV 2,5/5-GF-5,08 (1777109) con brida roscada; enchufe MSTB 2,5/5-STF-5,08 (1778014). Pines: 1 V+, 2 GND_VEH, 3 CAN_H, 4 CAN_L, 5 CAN_GND. 320 V / 12 A. Cableado interno hasta el conector circular de 8 hilos de la caja. -> Header vertical MSTBV 2,5/5-GF-5,08 (1777109) con brida roscada; enchufe MSTB 2,5/5-STF-5,08 (1778014). Pines: 1 V+, 2 GND_VEH, 3 CAN_H, 4 CAN_L, 5 CAN_GND. 320 V / 12 A. Cableado interno hasta el conector circular de 8 hilos de la caja. Montaje: soldar a mano; comprar en LCSC (C7164734).
- J2: LCSC (none) -> C480552; Notes Header vertical MSTBV 2,5/2-GF-5,08 (1777073, VERIFICAR en phoenixcontact.com) con brida roscada; enchufe MSTB 2,5/2-STF-5,08 (1777989). Pines: 1 DO1, 2 DO2 (low-side; drenador hasta 58 V + pico inductivo recortado < 100 V). Colocar la proteccion de 70_output junto a J2. -> Header vertical MSTBV 2,5/2-GF-5,08 (1777073, VERIFICAR en phoenixcontact.com) con brida roscada; enchufe MSTB 2,5/2-STF-5,08 (1777989). Pines: 1 DO1, 2 DO2 (low-side; drenador hasta 58 V + pico inductivo recortado < 100 V). Colocar la proteccion de 70_output junto a J2. Montaje: soldar a mano; comprar en LCSC (C480552).
- L101: LCSC (none) -> C2046332
- Q101: LCSC (none) -> C183634; Notes FET de corte (HGATE), 250 V: bloquea el load dump de 202 V. VGS +-20 V. MPN a verificar (disponibilidad y especificación) antes de congelar el BOM. -> FET de corte (HGATE), 250 V: bloquea el load dump de 202 V. VGS +-20 V. MPN a verificar (disponibilidad y especificación) antes de congelar el BOM. Compra (2026-10-30): sin stock en JLC/LCSC; comprar en DigiKey/Mouser y soldar a mano (PROTO y PROD). Sustituto rechazado: protección de entrada, el prototipo valida el diseño de producción.
- Q102: LCSC (none) -> C148263; Notes FET de diodo ideal (DGATE), 100 V: ve ~79 V en el pulso 1 (32 V + recorte de D102). -> FET de diodo ideal (DGATE), 100 V: ve ~79 V en el pulso 1 (32 V + recorte de D102). Compra (2026-10-30): sin stock en JLC/LCSC; comprar en DigiKey/Mouser y soldar a mano (PROTO y PROD). Sustituto rechazado: protección de entrada, el prototipo valida el diseño de producción.
- R102: LCSC (none) -> C469651
- R103: LCSC (none) -> C2076185
- R104: LCSC (none) -> C144653; LCSC_PROTO (none) -> C23185; MPN_PROTO (none) -> 0603WAF499JT5E; Manufacturer_PROTO (none) -> UNI-ROYAL; Notes R_SET entre CS+ y R_SENSE (TI: 50 ohm). -> R_SET entre CS+ y R_SENSE (TI: 50 ohm). PROTO (2026-10-30):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
- R105: LCSC (none) -> C125923; LCSC_PROTO (none) -> C22775; MPN_PROTO (none) -> 0603WAF1000T5E; Manufacturer_PROTO (none) -> UNI-ROYAL; Notes R_G en serie con C_dVdT. -> R_G en serie con C_dVdT. PROTO (2026-10-30): UNI-ROYAL 0603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
- R106: LCSC (none) -> C116674; LCSC_PROTO (none) -> C25803; MPN_PROTO (none) -> 0603WAF1003T5E; Manufacturer_PROTO (none) -> UNI-ROYAL; Notes (none) -> PROTO (2026-10-30): UNI-ROYAL 0603WAF1003T5E (LCSC C25803, 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
- R107: LCSC (none) -> C144630
- R108, R112: LCSC (none) -> C144484; LCSC_PROTO (none) -> C114947; MPN_PROTO (none) -> RC1206FR-0751KL; Notes 1206 por tensión/potencia: ~101 V y 0.2 W con load dump de 202 V. -> 1206 por tensión/potencia: ~101 V y 0.2 W con load dump de 202 V. PROTO (2026-10-30): Yageo RC1206FR-0751KL (LCSC C114947, JLC extended), misma especificación, sin AEC-Q200.
- R109: LCSC (none) -> C227657; LCSC_PROTO (none) -> C100797; MPN_PROTO (none) -> CR0603FA1621G; Manufacturer_PROTO (none) -> LIZ; Notes Corte por OV: 0.6 V x (1 + 102k/1.62k) = 38.4 V. -> Corte por OV: 0.6 V x (1 + 102k/1.62k) = 38.4 V. PROTO (202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
- R110: LCSC (none) -> C227994; LCSC_PROTO (none) -> C165742; MPN_PROTO (none) -> RC0603FR-0760K4L; Notes R_ILIM: 12 x 50 / (1 A x 10 mohm) = 60 k -> breaker a 1 A. -> R_ILIM: 12 x 50 / (1 A x 10 mohm) = 60 k -> breaker a 1 A. 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
- R111: LCSC (none) -> C116677; LCSC_PROTO (none) -> C25804; MPN_PROTO (none) -> 0603WAF1002T5E; Manufacturer_PROTO (none) -> UNI-ROYAL; Notes Pull-up de FLT (drenador abierto) a +3V3_D: PWR_FLT_N va directo a un GPIO del ESP32 (opcion B). -> Pull-up de FLT (drenador abierto) a +3V3_D: PWR_FLT_N va directo a un GPIO del ESP32 (opcion B). PROTO (2026-10-30): UNI-ROYAL 0603WAF1002T5E (LCSC C25804, JLC basic), misma especificación, sin AEC-Q200.
- U101: LCSC (none) -> C22428070

Commit message: [Claude Code] bom: compra principal en LCSC + DigiKey/Mouser; consolidación de pasivos
- Plan: JLC solo PCB + stencil Top; componentes de LCSC soldados a mano.
- Consolidación (solo valor/campos): R702/R752 4k7 → 2.2k; 23 × 100 nF a un
  MPN de 100 V X7R; PROTO 1 µF 50 V y 10 µF 25 V X7R. BOM PROTO 70 → 68 líneas.
- LCSC_BOM_COMPLETO_PROTO.csv: 6 juegos, 62 líneas, USD 552.43 (3 juegos: 286.65).
- DIGIKEY_MOUSER.csv: L201, U503, Q101, Q102, F101 (0 en LCSC), ≈ USD 99.54.
- Resumen de costos en BOM_SOURCING.md; archivos de JLC al día como alternativa.
- DRC 0 errores / 3 avisos aceptados, paridad 0, ERC 0 / 5.

Co-Authored-By: Claude Opus 5.5 <noreply@anthropic.com>
Parts:
- C107: LCSC_PROTO (none) -> C88219; MPN_PROTO (none) -> 0603B104K101NT; Manufacturer_PROTO (none) -> FH; Notes 100 V en 0603. MPN a verificar (disponibilidad y especificación) antes de congelar el BOM. -> 100 V en 0603. MPN a verificar (disponibilidad y especificación) antes de congelar el BOM. PROTO (2026-10-30, consolidacion): un solo MPN para los 100 nF 0603: 100 V X7R (FH 0603B104K101NT, LCSC C88219), sin AEC-Q200. PROD: Murata GCM188R72A104KA64D (100 V, AEC-Q200). Mismo valor y tolerancia.
- C108: LCSC C85864 -> C415406; LCSC_PROTO C14663 -> C88219; MPN GCM188R71H104KA57D -> GCM188R72A104KA64D; MPN_PROTO CC0603KRX7R9BB104 -> 0603B104K101NT; Manufacturer_PROTO Yageo -> FH; Notes C_CAP entre CAP y VS (bomba de carga). PROTO (2026-10-30): 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 -> C_CAP entre CAP y VS (bomba de carga). PROTO (2026-10-30, c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
- C109: LCSC_PROTO (none) -> C88219; MPN_PROTO (none) -> 0603B104K101NT; Manufacturer_PROTO (none) -> FH; Notes C_dVdT (TI ec. 2): Iinrush = C_OUT x 55 uA / C_dVdT. Con C105 montado (~1.07 mF): 0.59 A < breaker 1 A (con 10 nF eran 5.9 A y disparaba). Sin C105: ~34 mA. Arranque ~60 ms. 100 V en 0603. -> C_dVdT (TI ec. 2): Iinrush = C_OUT x 55 uA / C_dVdT. Con C105 montado (~1.07 mF): 0.59 A < breaker 1 A (con 10 nF eran 5.9 A y disparaba). Sin C105: ~34 mA. Arranque ~60 ms. 100 V en 0603. PROTO (2026-10-30, consolidacion): un solo MPN para los 100 nF 0603: 100 V X7R (FH 0603B104K101NT, LCSC C88219), sin AEC-Q200. PROD: Murata GCM188R72A104KA64D (100 V, AEC-Q200). Mismo valor y tolerancia.
Changed lines of the file:
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@@
 			)
 		)
-		(property "MPN" "GCM188R71H104KA57D"
+		(property "MPN" "GCM188R72A104KA64D"
 			(at 168.91 166.37 0)
 			(hide yes)
@@
 			)
 		)
-		(property "Notes" "C_CAP entre CAP y VS (bomba de carga). PROTO (2026-10-30): Yageo CC0603KRX7R9BB104 (LCSC C14663, JLC basic), misma especificación, sin AEC-Q200."
+		(property "Notes" "C_CAP entre CAP y VS (bomba de carga). PROTO (2026-10-30, consolidacion): un solo MPN para los 100 nF 0603: 100 V X7R (FH 0603B104K101NT, LCSC C88219), sin AEC-Q200. PROD: Murata GCM188R72A104KA64D (100 V, AEC-Q200). Mismo valor y tolerancia."
 			(at 168.91 166.37 0)
 			(hide yes)
@@
 			)
 		)
-		(property "LCSC" "C85864"
-			(at 168.91 166.37 0)
-			(hide yes)
-			(show_name no)
-			(do_not_autoplace no)
-			(effects
-				(font
-					(size 1.27 1.27)
-				)
-			)
-		)
-		(property "MPN_PROTO" "CC0603KRX7R9BB104"
-			(at 168.91 166.37 0)
-			(hide yes)
-			(show_name no)
-			(do_not_autoplace no)
-			(effects
-				(font
-					(size 1.27 1.27)
-				)
-			)
-		)
-		(property "Manufacturer_PROTO" "Yageo"
-			(at 168.91 166.37 0)
-			(hide yes)
-			(show_name no)
-			(do_not_autoplace no)
-			(effects
-				(font
-					(size 1.27 1.27)
-				)
-			)
-		)
-		(property "LCSC_PROTO" "C14663"
+		(property "LCSC" "C415406"
+			(at 168.91 166.37 0)
+			(hide yes)
+			(show_name no)
+			(do_not_autoplace no)
+			(effects
+				(font
+					(size 1.27 1.27)
+				)
+			)
+		)
+		(property "MPN_PROTO" "0603B104K101NT"
+			(at 168.91 166.37 0)
+			(hide yes)
+			(show_name no)
+			(do_not_autoplace no)
+			(effects
+				(font
+					(size 1.27 1.27)
+				)
+			)
+		)
+		(property "Manufacturer_PROTO" "FH"
+			(at 168.91 166.37 0)
+			(hide yes)
+			(show_name no)
+			(do_not_autoplace no)
+			(effects
+				(font
+					(size 1.27 1.27)
+				)
+			)
+		)
+		(property "LCSC_PROTO" "C88219"
 			(at 168.91 166.37 0)
 			(hide yes)
@@
 			)
 		)
-		(property "Notes" "C_dVdT (TI ec. 2): Iinrush = C_OUT x 55 uA / C_dVdT. Con C105 montado (~1.07 mF): 0.59 A < breaker 1 A (con 10 nF eran 5.9 A y disparaba). Sin C105: ~34 mA. Arranque ~60 ms. 100 V en 0603."
+		(property "Notes" "C_dVdT (TI ec. 2): Iinrush = C_OUT x 55 uA / C_dVdT. Con C105 montado (~1.07 mF): 0.59 A < breaker 1 A (con 10 nF eran 5.9 A y disparaba). Sin C105: ~34 mA. Arranque ~60 ms. 100 V en 0603. PROTO (2026-10-30, consolidacion): un solo MPN para los 100 nF 0603: 100 V X7R (FH 0603B104K101NT, LCSC C88219), sin AEC-Q200. PROD: Murata GCM188R72A104KA64D (100 V, AEC-Q200). Mismo valor y tolerancia."
 			(at 189.23 173.99 0)
 			(hide yes)
@@
 		)
 		(property "LCSC" "C415406"
+			(at 189.23 173.99 0)
+			(hide yes)
+			(show_name no)
+			(do_not_autoplace no)
+			(effects
+				(font
+					(size 1.27 1.27)
+				)
+			)
+		)
+		(property "MPN_PROTO" "0603B104K101NT"
+			(at 189.23 173.99 0)
+			(hide yes)
+			(show_name no)
+			(do_not_autoplace no)
+			(effects
+				(font
+					(size 1.27 1.27)
+				)
+			)
+		)
+		(property "Manufacturer_PROTO" "FH"
+			(at 189.23 173.99 0)
+			(hide yes)
+			(show_name no)
+			(do_not_autoplace no)
+			(effects
+				(font
+					(size 1.27 1.27)
+				)
+			)
+		)
+		(property "LCSC_PROTO" "C88219"
 			(at 189.23 173.99 0)
 			(hide yes)
@@
 			)
 		)
-		(property "Notes" "100 V en 0603. MPN a verificar (disponibilidad y especificación) antes de congelar el BOM."
+		(property "Notes" "100 V en 0603. MPN a verificar (disponibilidad y especificación) antes de congelar el BOM. PROTO (2026-10-30, consolidacion): un solo MPN para los 100 nF 0603: 100 V X7R (FH 0603B104K101NT, LCSC C88219), sin AEC-Q200. PROD: Murata GCM188R72A104KA64D (100 V, AEC-Q200). Mismo valor y tolerancia."
 			(at 288.29 80.01 0)
 			(hide yes)
@@
 			(at 288.29 80.01 0)
 			(hide yes)
+			(show_name no)
+			(do_not_autoplace no)
+			(effects
+				(font
+					(size 1.27 1.27)
+				)
+			)
+		)
+		(property "MPN_PROTO" "0603B104K101NT"
+			(at 288.29 80.01 0)
+			(hide yes)
+			(show_name no)
+			(do_not_autoplace no)
+			(effects
+				(font
+					(size 1.27 1.27)
+				)
+			)
+		)
+		(property "Manufacturer_PROTO" "FH"
+			(at 288.29 80.01 0)
+			(hide yes)
+			(show_name no)
+			(do_not_autoplace no)
+			(effects
+				(font
+					(size 1.27 1.27)
+				)
+			)
+		)
+		(property "LCSC_PROTO" "C88219"
+			(at 288.29 80.01 0)
+			(hide yes)

Commit message: [Claude Code] rc6: grupo A de la revisión externa y JLCDFM (pcb-v1-rc6)
Esquema (hoja 10), aprobado por el usuario:
- R-01: UVLO desde VBAT_F (R113 + R106 51k 1206, cara inferior junto a TP102),
  R107 9.53k (corte 6.44 V), U101.3 (SW) con no-connect. TI SNOSDF6 fig. 8-1.
- R-02: D104 = BAV23C (Diode:BAV70): A2-K es el D1 de VA a VS de TI.
  PROTO Diodes BAV23C-7-F (C150732); PROD Nexperia BAV23C,215.
- R-26: TP105 VS, TP106 VA, TP107 UVLO (cara inferior).
- Notes C-1..C-14, R-17, R-29; README, REVISION_CODEX, BOM_SOURCING.

PCB, sin mover componentes existentes:
- UVLO por B.Cu (y90 -> x111 -> y74.5) con 10 vías de costura GND_VEH.
- VA a D104.2 por x = 132.1.
- J-01 vías a 0.15 mm de los pads (excepción C403.2), J-02 tramos a
  >= 0.11 mm de las aberturas (excepciones de la misma red), J-03 64 textos
  fuera de vías, pads y orificios.
- DRC 0 errores / 3 avisos aceptados, 0 sin rutear, paridad 0; ERC 0 / 5;
  verify_etapa3/5 OK; 710 teardrops; fab/proto/ y BOM de LCSC regenerados.

Datasheets agregados en docs/datasheets/ (STD18NF25, BAS21, BAV23C, BAV23A_C_S,
BAV23C-7-F y los renombrados por el usuario). Scripts en scripts/rc6/.

Co-Authored-By: Claude Opus 5.5 <noreply@anthropic.com>
Parts:
- added R113: 51k, Resistor_SMD:R_1206_3216Metric, symbol Device:R
- added TP105: VS, TestPoint:TestPoint_Pad_D1.5mm, symbol Connector:TestPoint
- added TP106: VA, TestPoint:TestPoint_Pad_D1.5mm, symbol Connector:TestPoint
- added TP107: UVLO, TestPoint:TestPoint_Pad_D1.5mm, symbol Connector:TestPoint
- C109: Notes C_dVdT (TI ec. 2): Iinrush = C_OUT x 55 uA / C_dVdT. Con C105 montado (~1.07 mF): 0.59 A < breaker 1 A (con 10 nF eran 5.9 A y disparaba). Sin C105: ~34 mA. Arranque ~60 ms. 100 V en 0603. PROTO (2026-10-30, consolidacion): un solo MPN para los 100 nF 0603: 100 V X7R (FH 0603B104K101NT, LCSC C88219), sin AEC-Q200. PROD: Murata GCM188R72A104KA64D (100 V, AEC-Q200). Mismo valor y tolerancia. -> C_dVdT (TI ec. 2): Iinrush = C_OUT x 55 uA / C_dVdT. Con C105 montado (~1.07 mF): 0.59 A más la carga del buck durante la rampa (~0.15-0.25 A) contra el breaker de 0.88-1.07 A (V(SNS_TH) 1.08-1.32 V): margen de ~0.1 A, ensayar en PROD (rev. B: 220-330 nF) (con 10 nF eran 5.9 A y disparaba). Sin C105: ~34 mA. Arranque ~60 ms. 100 V en 0603. PROTO (2026-10-30, consolidacion): un solo MPN para los 100 nF 0603: 100 V X7R (FH 0603B104K101NT, LCSC C88219), sin AEC-Q200. PROD: Murata GCM188R72A104KA64D (100 V, AEC-Q200). Mismo valor y tolerancia.
- D104: value BAS21 -> BAV23C; symbol Diode:BAS21 -> Diode:BAV70; LCSC C8661 -> C282370; LCSC_PROTO (none) -> C150732; MPN BAS21,215 -> BAV23C,215; MPN_PROTO (none) -> BAV23C-7-F; Manufacturer_PROTO (none) -> Diodes Incorporated; Notes Bloqueo de VS en polaridad inversa (D1 de la ref. TI). -> D104 = BAV23C (doble, cátodo común): A1-K bloquea VS en pol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
- J2: Notes Header vertical MSTBV 2,5/2-GF-5,08 (1777073, VERIFICAR en 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 -> Header vertical MSTBV 2,5/2-GF-5,08 (1777073, confirmado) c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
- R106: value 100k -> 51k; footprint Resistor_SMD:R_0603_1608Metric -> Resistor_SMD:R_1206_3216Metric; LCSC C116674 -> C144484; LCSC_PROTO C25803 -> C114947; MPN AC0603FR-07100KL -> AC1206FR-0751KL; MPN_PROTO 0603WAF1003T5E -> RC1206FR-0751KL; Manufacturer_PROTO UNI-ROYAL -> (none); Notes PROTO (2026-10-30): UNI-ROYAL 0603WAF1003T5E (LCSC C25803, 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 -> R1 de UVLO (TI SNOSDF6 fig. 8-1, R1 a VBAT): R113 + R106 en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
- R107: value 9.31k -> 9.53k; LCSC C144630 -> C228113; LCSC_PROTO (none) -> C23127; MPN AC0603FR-079K31L -> AC0603FR-079K53L; MPN_PROTO (none) -> 0603WAF9531T5E; Manufacturer_PROTO (none) -> UNI-ROYAL; Notes UVLO de caída ~6.5 V. -> R2 de UVLO. Con R113 + R106 = 102 kΩ desde VBAT_F: corte 0.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
Connections:
- net UVLO: now also TP107.1
- net VA: now also D104.2 (A), TP106.1
- net VBAT_F: now also R113.1
- net VS: now also TP105.1
- net SW: no longer names the net of U101.3 (SW)
- net SW: no longer R106.1
- new net: R106.1, R113.2
- no-connect marks 1 -> 2
