File: sheets/20_isolation.kicad_sch (KiCad schematic)
At the start: 16 parts, among them U201 TPS7A1650QDGNRQ1, U202 ISO7763FQDWRQ1

Commit message: fixed and review
Parts:
- removed PS201: EC4AW8-48S05, Converter_DCDC:Converter_DCDC_TRACO_THD_15-xxxxWIN_THT, symbol INCLI-VA:EC4AW8-48S05
- added PS201: URB2405YMD-10WR3, INCLI-VA:PWRM-TH_URBXXXXYMD_10WR3, symbol INCLI-VA:URB2405YMD-10WR3_C5369754
Connections:
- net +5V_ISO: now also PS201.3 (+VO)
- net +VPROT: now also PS201.2 (+Vin)
- net GND_ISO: now also PS201.5 (GND)
- net GND_VEH: now also PS201.1 (-Vin)
- no-connect marks 4 -> 5
Other:
- moved on the sheet: C201, C202, C203, C204, C205, C206, TP201, U201
