File: sheets/30_regulation.kicad_sch (KiCad schematic)
At the start: 25 parts, among them U301 TPS62A02QDRLRQ1, U302 LP5907QMFX-3.3Q1

Commit message: fixed and review
Other:
- moved on the sheet: C301, C302, C303, C304, C306, C307, C309, C310, FB301, L301, R301, R302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
