File: sheets/30_regulation.kicad_sch (KiCad schematic)
At the start: 25 parts, among them U301 TPS62A02QDRLRQ1, U302 LP5907QMFX-3.3Q1

Commit message: [Claude Code] esquema+PCB: campos LCSC y sustitutos PROTO del BOM (pcb-v1-rc2)
- Esquema (solo campos, ocultos): LCSC en todos los componentes; MPN_PROTO,
  LCSC_PROTO y Manufacturer_PROTO con los sustitutos aceptados; Notes con
  compra y montaje (Q101, Q102, F101, L201, U503 a mano desde DigiKey/Mouser).
  MPN (PROD), valores, huellas y conexiones sin cambios. LCSC Part -> LCSC.
- PCB: mismos campos en las 145 huellas, insertados como texto (equivalente
  a F8 solo para campos); nada cambia fuera de las huellas.
- ERC por hoja igual que antes (0 errores, 5 avisos). DRC 0 errores / 3 avisos
  aceptados, 0 sin rutear, paridad 0 (antes de sincronizar: 145).
- etapa6_fab.py usa los campos _PROTO y genera bom_jlc_lcsc.csv; este y
  cpl_jlc.csv salen idénticos (60 líneas, 123 piezas). Gerbers sin cambios
  de contenido.

Co-Authored-By: Claude Opus 5.5 <noreply@anthropic.com>
Parts:
- C301: LCSC (none) -> C126586
- C302: LCSC (none) -> C85864; LCSC_PROTO (none) -> C14663; MPN_PROTO (none) -> CC0603KRX7R9BB104; Manufacturer_PROTO (none) -> Yageo; Notes Desacople de alta frecuencia en VIN de U301, pegado a los pines. -> Desacople de alta frecuencia en VIN de U301, pegado a los pines. PROTO (2026-10-30): Yageo CC0603KRX7R9BB104 (LCSC C14663, JLC basic), misma especificación, sin AEC-Q200.
- C303: LCSC (none) -> C126542; LCSC_PROTO (none) -> C1634; MPN_PROTO (none) -> CL10C100JB8NNNC; Manufacturer_PROTO (none) -> Samsung; Notes C_FF en paralelo con R303: valor de TI para 3.3 V con R2 = 100k (SLUSFG7 9.2.2.2). C0G. -> C_FF en paralelo con R303: valor de TI para 3.3 V con R2 = 100k (SLUSFG7 9.2.2.2). C0G. PROTO (2026-10-30): Samsung CL10C100JB8NNNC (LCSC C1634, JLC basic), misma especificación, sin AEC-Q200.
- C304: LCSC (none) -> C907991
- C306, C307: LCSC (none) -> C161212
- C309: LCSC (none) -> C85864; LCSC_PROTO (none) -> C14663; MPN_PROTO (none) -> CC0603KRX7R9BB104; Manufacturer_PROTO (none) -> Yageo; Notes Filtro/reserva de carga del muestreo del ADC1 en VMON_5V. -> Filtro/reserva de carga del muestreo del ADC1 en VMON_5V. P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
- C310: LCSC (none) -> C85864; LCSC_PROTO (none) -> C14663; MPN_PROTO (none) -> CC0603KRX7R9BB104; Manufacturer_PROTO (none) -> Yageo; Notes Filtro/reserva de carga del muestreo del ADC1 en VMON_3V3. -> Filtro/reserva de carga del muestreo del ADC1 en VMON_3V3. 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
- FB301: LCSC (none) -> C80165
- L301: LCSC (none) -> C4555951
- R301: LCSC (none) -> C116674; LCSC_PROTO (none) -> C25803; MPN_PROTO (none) -> 0603WAF1003T5E; Manufacturer_PROTO (none) -> UNI-ROYAL; Notes EN de U301 a +5V_VEH: el buck arranca con el riel (EN no puede quedar flotante, TI). -> EN de U301 a +5V_VEH: el buck arranca con el riel (EN no puede quedar flotante, TI). PROTO (2026-10-30): UNI-ROYAL 0603WAF1003T5E (LCSC C25803, JLC basic), misma especificación, sin AEC-Q200.
- R302: LCSC (none) -> C116674; LCSC_PROTO (none) -> C25803; MPN_PROTO (none) -> 0603WAF1003T5E; Manufacturer_PROTO (none) -> UNI-ROYAL; Notes Pull-up de PG (drenador abierto, máx 5.5 V) a +3V3_D. -> Pull-up de PG (drenador abierto, máx 5.5 V) a +3V3_D. PROTO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
- R303: LCSC (none) -> C227908; LCSC_PROTO (none) -> C101055; MPN_PROTO (none) -> CR0603FA4533G; Manufacturer_PROTO (none) -> LIZ; Notes Divisor de FB superior: VOUT = 0.6 V x (1 + 453k/100k) = 3.318 V. -> Divisor de FB superior: VOUT = 0.6 V x (1 + 453k/100k) = 3.318 V. PROTO (2026-10-30): LIZ CR0603FA4533G (LCSC C101055, JLC extended), misma especificación, sin AEC-Q200.
- R304: LCSC (none) -> C116674; LCSC_PROTO (none) -> C25803; MPN_PROTO (none) -> 0603WAF1003T5E; Manufacturer_PROTO (none) -> UNI-ROYAL; Notes Divisor de FB inferior (TI: R2 <= 400k; 100k para usar C_FF = 10 pF). -> Divisor de FB inferior (TI: R2 <= 400k; 100k para usar C_FF = 10 pF). PROTO (2026-10-30): UNI-ROYAL 0603WAF1003T5E (LCSC C25803, JLC basic), misma especificación, sin AEC-Q200.
- R305: LCSC (none) -> C116674; LCSC_PROTO (none) -> C25803; MPN_PROTO (none) -> 0603WAF1003T5E; Manufacturer_PROTO (none) -> UNI-ROYAL; Notes Divisor VMON_5V: 5 V x 49.9k/149.9k = 1.66 V (5.5 V -> 1.83 V). -> Divisor VMON_5V: 5 V x 49.9k/149.9k = 1.66 V (5.5 V -> 1.83 V). PROTO (2026-10-30): UNI-ROYAL 0603WAF1003T5E (LCSC C25803, JLC basic), misma especificación, sin AEC-Q200.
- R306: LCSC (none) -> C144654; LCSC_PROTO (none) -> C23184; MPN_PROTO (none) -> 0603WAF4992T5E; Manufacturer_PROTO (none) -> UNI-ROYAL; Notes Divisor VMON_5V: 5 V x 49.9k/149.9k = 1.66 V (5.5 V -> 1.83 V). -> Divisor VMON_5V: 5 V x 49.9k/149.9k = 1.66 V (5.5 V -> 1.83 V). PROTO (2026-10-30): UNI-ROYAL 0603WAF4992T5E (LCSC C23184, JLC basic), misma especificación, sin AEC-Q200.
- R307, R308: LCSC (none) -> C116674; LCSC_PROTO (none) -> C25803; MPN_PROTO (none) -> 0603WAF1003T5E; Manufacturer_PROTO (none) -> UNI-ROYAL; Notes Divisor VMON_3V3: 3.3 V x 1/2 = 1.65 V. -> Divisor VMON_3V3: 3.3 V x 1/2 = 1.65 V. PROTO (2026-10-30):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
- U301: LCSC (none) -> C49259289
- U302: LCSC (none) -> C130005

Commit message: [Claude Code] bom: compra principal en LCSC + DigiKey/Mouser; consolidación de pasivos
- Plan: JLC solo PCB + stencil Top; componentes de LCSC soldados a mano.
- Consolidación (solo valor/campos): R702/R752 4k7 → 2.2k; 23 × 100 nF a un
  MPN de 100 V X7R; PROTO 1 µF 50 V y 10 µF 25 V X7R. BOM PROTO 70 → 68 líneas.
- LCSC_BOM_COMPLETO_PROTO.csv: 6 juegos, 62 líneas, USD 552.43 (3 juegos: 286.65).
- DIGIKEY_MOUSER.csv: L201, U503, Q101, Q102, F101 (0 en LCSC), ≈ USD 99.54.
- Resumen de costos en BOM_SOURCING.md; archivos de JLC al día como alternativa.
- DRC 0 errores / 3 avisos aceptados, paridad 0, ERC 0 / 5.

Co-Authored-By: Claude Opus 5.5 <noreply@anthropic.com>
Parts:
- C301: LCSC_PROTO (none) -> C3039694; MPN_PROTO (none) -> CL21B106KAYQNNE; Manufacturer_PROTO (none) -> Samsung; Notes C_IN del buck, 10 V X7R. 0805 (no 0603) por pérdida de capacitancia por DC bias a 5 V. Pegado a VIN/GND de U301. MPN a verificar (disponibilidad y especificación) antes de congelar el BOM. -> C_IN del buck, 10 V X7R. 0805 (no 0603) por pérdida de capacitancia por DC bias a 5 V. Pegado a VIN/GND de U301. MPN a verificar (disponibilidad y especificación) antes de congelar el BOM. PROTO (2026-10-30, consolidacion): Samsung CL21B106KAYQNNE (25 V X7R, LCSC C3039694), sin AEC-Q200: el original no tiene stock en lcsc.com.
- C302: LCSC C85864 -> C415406; LCSC_PROTO C14663 -> C88219; MPN GCM188R71H104KA57D -> GCM188R72A104KA64D; MPN_PROTO CC0603KRX7R9BB104 -> 0603B104K101NT; Manufacturer_PROTO Yageo -> FH; Notes Desacople de alta frecuencia en VIN de U301, pegado a los pines. PROTO (2026-10-30): Yageo CC0603KRX7R9BB104 (LCSC C14663, JLC basic), misma especificación, sin AEC-Q200. -> Desacople de alta frecuencia en VIN de U301, pegado a los pines. PROTO (2026-10-30, consolidacion): un solo MPN para los 100 nF 0603: 100 V X7R (FH 0603B104K101NT, LCSC C88219), sin AEC-Q200. PROD: Murata GCM188R72A104KA64D (100 V, AEC-Q200). Mismo valor y tolerancia.
- C306: LCSC_PROTO (none) -> C559769; MPN_PROTO (none) -> CC0603KRX7R9BB105; Manufacturer_PROTO (none) -> Yageo; Notes C_IN del LDO (TI: 1 uF cerámico). -> C_IN del LDO (TI: 1 uF cerámico). PROTO (2026-10-30, consol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
- C307: LCSC_PROTO (none) -> C559769; MPN_PROTO (none) -> CC0603KRX7R9BB105; Manufacturer_PROTO (none) -> Yageo; Notes C_OUT del LDO (TI: >= 1 uF efectivo). -> C_OUT del LDO (TI: >= 1 uF efectivo). PROTO (2026-10-30, co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
- C309: LCSC C85864 -> C415406; LCSC_PROTO C14663 -> C88219; MPN GCM188R71H104KA57D -> GCM188R72A104KA64D; MPN_PROTO CC0603KRX7R9BB104 -> 0603B104K101NT; Manufacturer_PROTO Yageo -> FH; Notes Filtro/reserva de carga del muestreo del ADC1 en VMON_5V. PROTO (2026-10-30): Yageo CC0603KRX7R9BB104 (LCSC C14663, JLC basic), misma especificación, sin AEC-Q200. -> Filtro/reserva de carga del muestreo del ADC1 en VMON_5V. PROTO (2026-10-30, consolidacion): un solo MPN para los 100 nF 0603: 100 V X7R (FH 0603B104K101NT, LCSC C88219), sin AEC-Q200. PROD: Murata GCM188R72A104KA64D (100 V, AEC-Q200). Mismo valor y tolerancia.
- C310: LCSC C85864 -> C415406; LCSC_PROTO C14663 -> C88219; MPN GCM188R71H104KA57D -> GCM188R72A104KA64D; MPN_PROTO CC0603KRX7R9BB104 -> 0603B104K101NT; Manufacturer_PROTO Yageo -> FH; Notes Filtro/reserva de carga del muestreo del ADC1 en VMON_3V3. PROTO (2026-10-30): Yageo CC0603KRX7R9BB104 (LCSC C14663, JLC basic), misma especificación, sin AEC-Q200. -> Filtro/reserva de carga del muestreo del ADC1 en VMON_3V3. PROTO (2026-10-30, consolidacion): un solo MPN para los 100 nF 0603: 100 V X7R (FH 0603B104K101NT, LCSC C88219), sin AEC-Q200. PROD: Murata GCM188R72A104KA64D (100 V, AEC-Q200). Mismo valor y tolerancia.
Changed lines of the file:
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@@
 			)
 		)
-		(property "MPN" "GCM188R71H104KA57D"
+		(property "MPN" "GCM188R72A104KA64D"
 			(at 105.41 95.25 0)
 			(hide yes)
@@
 			)
 		)
-		(property "Notes" "Desacople de alta frecuencia en VIN de U301, pegado a los pines. PROTO (2026-10-30): Yageo CC0603KRX7R9BB104 (LCSC C14663, JLC basic), misma especificación, sin AEC-Q200."
+		(property "Notes" "Desacople de alta frecuencia en VIN de U301, pegado a los pines. PROTO (2026-10-30, consolidacion): un solo MPN para los 100 nF 0603: 100 V X7R (FH 0603B104K101NT, LCSC C88219), sin AEC-Q200. PROD: Murata GCM188R72A104KA64D (100 V, AEC-Q200). Mismo valor y tolerancia."
 			(at 105.41 95.25 0)
 			(hide yes)
@@
 			)
 		)
-		(property "LCSC" "C85864"
+		(property "LCSC" "C415406"
 			(at 105.41 95.25 0)
 			(hide yes)
@@
 			)
 		)
-		(property "MPN_PROTO" "CC0603KRX7R9BB104"
+		(property "MPN_PROTO" "0603B104K101NT"
 			(at 105.41 95.25 0)
 			(hide yes)
@@
 			)
 		)
-		(property "Manufacturer_PROTO" "Yageo"
+		(property "Manufacturer_PROTO" "FH"
 			(at 105.41 95.25 0)
 			(hide yes)
@@
 			)
 		)
-		(property "LCSC_PROTO" "C14663"
+		(property "LCSC_PROTO" "C88219"
 			(at 105.41 95.25 0)
 			(hide yes)
@@
 			)
 		)
-		(property "Notes" "C_IN del LDO (TI: 1 uF cerámico)."
+		(property "Notes" "C_IN del LDO (TI: 1 uF cerámico). PROTO (2026-10-30, consolidacion): Yageo CC0603KRX7R9BB105 (50 V X7R, LCSC C559769), sin AEC-Q200: mas stock y menos perdida por DC bias."
 			(at 110.49 194.31 0)
 			(hide yes)
@@
 			)
 		)
+		(property "MPN_PROTO" "CC0603KRX7R9BB105"
+			(at 110.49 194.31 0)
+			(hide yes)
+			(show_name no)
+			(do_not_autoplace no)
+			(effects
+				(font
+					(size 1.27 1.27)
+				)
+			)
+		)
+		(property "Manufacturer_PROTO" "Yageo"
+			(at 110.49 194.31 0)
+			(hide yes)
+			(show_name no)
+			(do_not_autoplace no)
+			(effects
+				(font
+					(size 1.27 1.27)
+				)
+			)
+		)
+		(property "LCSC_PROTO" "C559769"
+			(at 110.49 194.31 0)
+			(hide yes)
+			(show_name no)
+			(do_not_autoplace no)
+			(effects
+				(font
+					(size 1.27 1.27)
+				)
+			)
+		)
 		(pin "1"
 		)
@@
 			)
 		)
-		(property "Notes" "C_IN del buck, 10 V X7R. 0805 (no 0603) por pérdida de capacitancia por DC bias a 5 V. Pegado a VIN/GND de U301. MPN a verificar (disponibilidad y especificación) antes de congelar el BOM."
+		(property "Notes" "C_IN del buck, 10 V X7R. 0805 (no 0603) por pérdida de capacitancia por DC bias a 5 V. Pegado a VIN/GND de U301. MPN a verificar (disponibilidad y especificación) antes de congelar el BOM. PROTO (2026-10-30, consolidacion): Samsung CL21B106KAYQNNE (25 V X7R, LCSC C3039694), sin AEC-Q200: el original no tiene stock en lcsc.com."
 			(at 95.25 95.25 0)
 			(hide yes)
@@
 			)
 		)
+		(property "MPN_PROTO" "CL21B106KAYQNNE"
+			(at 95.25 95.25 0)
+			(hide yes)
+			(show_name no)
+			(do_not_autoplace no)
+			(effects
+				(font
+					(size 1.27 1.27)
+				)
+			)
+		)
+		(property "Manufacturer_PROTO" "Samsung"
+			(at 95.25 95.25 0)
+			(hide yes)
+			(show_name no)
+			(do_not_autoplace no)
+			(effects
+				(font
+					(size 1.27 1.27)
+				)
+			)
+		)
+		(property "LCSC_PROTO" "C3039694"
+			(at 95.25 95.25 0)
+			(hide yes)
+			(show_name no)
+			(do_not_autoplace no)
+			(effects
+				(font
+					(size 1.27 1.27)
+				)
+			)
+		)
 		(pin "1"
 		)
@@
 			)
 		)
-		(property "Notes" "C_OUT del LDO (TI: >= 1 uF efectivo)."
+		(property "Notes" "C_OUT del LDO (TI: >= 1 uF efectivo). PROTO (2026-10-30, consolidacion): Yageo CC0603KRX7R9BB105 (50 V X7R, LCSC C559769), sin AEC-Q200: mas stock y menos perdida por DC bias."
 			(at 156.21 194.31 0)
 			(hide yes)
@@
 			)
 		)
+		(property "MPN_PROTO" "CC0603KRX7R9BB105"
+			(at 156.21 194.31 0)
+			(hide yes)
+			(show_name no)
+			(do_not_autoplace no)
+			(effects
+				(font
+					(size 1.27 1.27)
+				)
+			)
+		)
+		(property "Manufacturer_PROTO" "Yageo"
+			(at 156.21 194.31 0)
+			(hide yes)
+			(show_name no)
+			(do_not_autoplace no)
+			(effects
+				(font
+					(size 1.27 1.27)
+				)
+			)
+		)
+		(property "LCSC_PROTO" "C559769"
+			(at 156.21 194.31 0)
+			(hide yes)
+			(show_name no)
+			(do_not_autoplace no)
+			(effects
+				(font
+					(size 1.27 1.27)
+				)
+			)
+		)
 		(pin "1"
 		)
@@
 			)
 		)
-		(property "MPN" "GCM188R71H104KA57D"
+		(property "MPN" "GCM188R72A104KA64D"
 			(at 356.87 158.75 0)
 			(hide yes)
@@
 			)
 		)
-		(property "Notes" "Filtro/reserva de carga del muestreo del ADC1 en VMON_3V3. PROTO (2026-10-30): Yageo CC0603KRX7R9BB104 (LCSC C14663, JLC basic), misma especificación, sin AEC-Q200."
+		(property "Notes" "Filtro/reserva de carga del muestreo del ADC1 en VMON_3V3. PROTO (2026-10-30, consolidacion): un solo MPN para los 100 nF 0603: 100 V X7R (FH 0603B104K101NT, LCSC C88219), sin AEC-Q200. PROD: Murata GCM188R72A104KA64D (100 V, AEC-Q200). Mismo valor y tolerancia."
 			(at 356.87 158.75 0)
 			(hide yes)
@@
 			)
 		)
-		(property "LCSC" "C85864"
+		(property "LCSC" "C415406"
 			(at 356.87 158.75 0)
 			(hide yes)
@@
 			)
 		)
-		(property "MPN_PROTO" "CC0603KRX7R9BB104"
+		(property "MPN_PROTO" "0603B104K101NT"
 			(at 356.87 158.75 0)
 			(hide yes)
@@
 			)
 		)
-		(property "Manufacturer_PROTO" "Yageo"
+		(property "Manufacturer_PROTO" "FH"
 			(at 356.87 158.75 0)
 			(hide yes)
@@
 			)
 		)
-		(property "LCSC_PROTO" "C14663"
+		(property "LCSC_PROTO" "C88219"
 			(at 356.87 158.75 0)
 			(hide yes)
@@
 			)
 		)
-		(property "MPN" "GCM188R71H104KA57D"
+		(property "MPN" "GCM188R72A104KA64D"
 			(at 318.77 158.75 0)
 			(hide yes)
@@
 			)
 		)
-		(property "Notes" "Filtro/reserva de carga del muestreo del ADC1 en VMON_5V. PROTO (2026-10-30): Yageo CC0603KRX7R9BB104 (LCSC C14663, JLC basic), misma especificación, sin AEC-Q200."
+		(property "Notes" "Filtro/reserva de carga del muestreo del ADC1 en VMON_5V. PROTO (2026-10-30, consolidacion): un solo MPN para los 100 nF 0603: 100 V X7R (FH 0603B104K101NT, LCSC C88219), sin AEC-Q200. PROD: Murata GCM188R72A104KA64D (100 V, AEC-Q200). Mismo valor y tolerancia."
 			(at 318.77 158.75 0)
 			(hide yes)
@@
 			)
 		)
-		(property "LCSC" "C85864"
+		(property "LCSC" "C415406"
 			(at 318.77 158.75 0)
 			(hide yes)
@@
 			)
 		)
-		(property "MPN_PROTO" "CC0603KRX7R9BB104"
+		(property "MPN_PROTO" "0603B104K101NT"
 			(at 318.77 158.75 0)
 			(hide yes)
@@
 			)
 		)
-		(property "Manufacturer_PROTO" "Yageo"
+		(property "Manufacturer_PROTO" "FH"
 			(at 318.77 158.75 0)
 			(hide yes)
@@
 			)
 		)
-		(property "LCSC_PROTO" "C14663"
+		(property "LCSC_PROTO" "C88219"
 			(at 318.77 158.75 0)
 			(hide yes)

Commit message: [Claude Code] rc6: grupo A de la revisión externa y JLCDFM (pcb-v1-rc6)
Esquema (hoja 10), aprobado por el usuario:
- R-01: UVLO desde VBAT_F (R113 + R106 51k 1206, cara inferior junto a TP102),
  R107 9.53k (corte 6.44 V), U101.3 (SW) con no-connect. TI SNOSDF6 fig. 8-1.
- R-02: D104 = BAV23C (Diode:BAV70): A2-K es el D1 de VA a VS de TI.
  PROTO Diodes BAV23C-7-F (C150732); PROD Nexperia BAV23C,215.
- R-26: TP105 VS, TP106 VA, TP107 UVLO (cara inferior).
- Notes C-1..C-14, R-17, R-29; README, REVISION_CODEX, BOM_SOURCING.

PCB, sin mover componentes existentes:
- UVLO por B.Cu (y90 -> x111 -> y74.5) con 10 vías de costura GND_VEH.
- VA a D104.2 por x = 132.1.
- J-01 vías a 0.15 mm de los pads (excepción C403.2), J-02 tramos a
  >= 0.11 mm de las aberturas (excepciones de la misma red), J-03 64 textos
  fuera de vías, pads y orificios.
- DRC 0 errores / 3 avisos aceptados, 0 sin rutear, paridad 0; ERC 0 / 5;
  verify_etapa3/5 OK; 710 teardrops; fab/proto/ y BOM de LCSC regenerados.

Datasheets agregados en docs/datasheets/ (STD18NF25, BAS21, BAV23C, BAV23A_C_S,
BAV23C-7-F y los renombrados por el usuario). Scripts en scripts/rc6/.

Co-Authored-By: Claude Opus 5.5 <noreply@anthropic.com>
Parts:
- C304: Notes C_OUT del buck, 10 V X7R. 0805 por DC bias. Presupuesto de 47 uF en +3V3_D (TI sin Bode): 22 uF aquí + 22 uF + 100 nF en el módulo (40_mcu) + ~0.5 uF de desacoples = ~44.6 uF. MPN a verificar (disponibilidad y especificación) antes de congelar el BOM. -> C_OUT del buck, 10 V X7R. 0805 por DC bias. Presupuesto de 47 uF en +3V3_D (TI sin Bode): 22 uF aquí + 22 uF + 100 nF en el módulo (40_mcu) + ~0.5 uF de desacoples = ~44.6 uF, más 10 uF de C605 (hoja 60) = ~54.6 uF nominal; con DC bias probablemente < 47 uF: verificar el escalón 0.1 -> 0.6 A en el bring-up. MPN a verificar (disponibilidad y especificación) antes de congelar el BOM.
Changed lines of the file:
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@@
 			)
 		)
-		(property "Notes" "C_OUT del buck, 10 V X7R. 0805 por DC bias. Presupuesto de 47 uF en +3V3_D (TI sin Bode): 22 uF aquí + 22 uF + 100 nF en el módulo (40_mcu) + ~0.5 uF de desacoples = ~44.6 uF. MPN a verificar (disponibilidad y especificación) antes de congelar el BOM."
+		(property "Notes" "C_OUT del buck, 10 V X7R. 0805 por DC bias. Presupuesto de 47 uF en +3V3_D (TI sin Bode): 22 uF aquí + 22 uF + 100 nF en el módulo (40_mcu) + ~0.5 uF de desacoples = ~44.6 uF, más 10 uF de C605 (hoja 60) = ~54.6 uF nominal; con DC bias probablemente < 47 uF: verificar el escalón 0.1 -> 0.6 A en el bring-up. MPN a verificar (disponibilidad y especificación) antes de congelar el BOM."
 			(at 189.23 102.87 0)
 			(hide yes)
