File: sheets/70_output_ch.kicad_sch (KiCad schematic)
At the start: 17 parts, among them Q701 FDD7N25LZ, Q702 BC817-40, Q703 BC807-40

Commit message: fixed and review
Other:
- moved on the sheet: C701, D701, D702, D703, Q701, Q702, Q703, R701, R702, R703, R704, R705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
