File: sheets/70_output_ch.kicad_sch (KiCad schematic)
At the start: 21 parts, among them Q701 DMN10H220LQ, Q702 BC817-40, Q703 BC807-40, U701 74AHCT1G126

Commit message: [Codex] Integra cierre de Claude y valida sincronizacion previa al layout
Parts:
- C701, C702, D701, D702, D703, D704, Q702, Q703, R701, R702, R703, R704, R705, R706, R707, R708, R709, R710, R711: Variant (none) -> OUT
- Q701: MPN_PROTO (none) -> DMN10H220L-7; Variant (none) -> OUT
- U701: MPN_PROTO (none) -> SN74AHCT1G126DBVR; Variant (none) -> OUT
