File: sheets/70_output_ch.kicad_sch (KiCad schematic)
At the start: 12 parts, among them Q701 DMN10H220LQ, U701 74AHCT1G126

Commit message: [Claude Code] rc6: grupo A de la revisión externa y JLCDFM (pcb-v1-rc6)
Esquema (hoja 10), aprobado por el usuario:
- R-01: UVLO desde VBAT_F (R113 + R106 51k 1206, cara inferior junto a TP102),
  R107 9.53k (corte 6.44 V), U101.3 (SW) con no-connect. TI SNOSDF6 fig. 8-1.
- R-02: D104 = BAV23C (Diode:BAV70): A2-K es el D1 de VA a VS de TI.
  PROTO Diodes BAV23C-7-F (C150732); PROD Nexperia BAV23C,215.
- R-26: TP105 VS, TP106 VA, TP107 UVLO (cara inferior).
- Notes C-1..C-14, R-17, R-29; README, REVISION_CODEX, BOM_SOURCING.

PCB, sin mover componentes existentes:
- UVLO por B.Cu (y90 -> x111 -> y74.5) con 10 vías de costura GND_VEH.
- VA a D104.2 por x = 132.1.
- J-01 vías a 0.15 mm de los pads (excepción C403.2), J-02 tramos a
  >= 0.11 mm de las aberturas (excepciones de la misma red), J-03 64 textos
  fuera de vías, pads y orificios.
- DRC 0 errores / 3 avisos aceptados, 0 sin rutear, paridad 0; ERC 0 / 5;
  verify_etapa3/5 OK; 710 teardrops; fab/proto/ y BOM de LCSC regenerados.

Datasheets agregados en docs/datasheets/ (STD18NF25, BAS21, BAV23C, BAV23A_C_S,
BAV23C-7-F y los renombrados por el usuario). Scripts en scripts/rc6/.

Co-Authored-By: Claude Opus 5.5 <noreply@anthropic.com>
Parts:
- D703: Notes Diagnostico (DNP en prototipo): limita DIAG a 3.3 V para el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 -> Diagnostico (DNP en prototipo): protege el GPIO del ESP32. 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
- R708, R709: Notes 1206 por tension: el drenador llega a ~250 V; dos en serie,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 -> 1206 por tension: Q701/Q751 son de 100 V y D701/D751 recort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
Changed lines of the file:
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@@
 			)
 		)
-		(property "Notes" "1206 por tension: el drenador llega a ~250 V; dos en serie, ~125 V cada una."
+		(property "Notes" "1206 por tension: Q701/Q751 son de 100 V y D701/D751 recortan a <= 93.6 V (lo de ~250 V venía del FDD7N25LZ); el 1206 sigue dando margen."
 			(at 248.92 106.68 0)
 			(hide yes)
@@
 			)
 		)
-		(property "Notes" "Diagnostico (DNP en prototipo): limita DIAG a 3.3 V para el GPIO del ESP32 (antes 5V1 para el ISO7763)."
+		(property "Notes" "Diagnostico (DNP en prototipo): protege el GPIO del ESP32. Con ~30 uA (drenador a 12 V) el zener no fija 3.3 V y DIAG puede leer bajo con la carga presente (hallazgo R-05): rediseñar en la rev. B."
 			(at 259.08 114.3 0)
 			(hide yes)
@@
 			)
 		)
-		(property "Notes" "1206 por tension: el drenador llega a ~250 V; dos en serie, ~125 V cada una."
+		(property "Notes" "1206 por tension: Q701/Q751 son de 100 V y D701/D751 recortan a <= 93.6 V (lo de ~250 V venía del FDD7N25LZ); el 1206 sigue dando margen."
 			(at 248.92 99.06 0)
 			(hide yes)
