File: sheets/60_can.kicad_sch (KiCad schematic)
At the start: 2 parts, among them U1 ADM3055E

Commit message: order pcb
Parts:
- added C1, C7: 0.01uF, symbol Device:C
- added C10, C2, C4, C8: 0.1uF, symbol Device:C
- added C11, C3, C5, C6: 10uF, symbol Device:C
- added C9: 4700pF, symbol Device:C
- added FB1, FB2: FerriteBead, symbol Device:FerriteBead
- added R2, R3: 60.4, symbol Device:R
Connections:
- net +3V3_D: now also U1.4 (V_{IO}), C1.1, C2.1, C5.1
- net +5V_ISO: now also U1.3 (V_{CC}), C3.1, C4.1, C6.1
- net BUS_CAN_H: now also U1.14 (CANH), R2.1
- net BUS_CAN_L: now also U1.13 (CANL), R3.2
- net CAN_RX: now also U1.5 (RXD)
- net CAN_STBY: now also U1.8 (STBY)
- net CAN_TX: now also U1.7 (TXD)
- net GND_CAN: now also U1.11 (GND_{2}), U1.15 (GND_{2}), U1.18 (GND_{ISO}), U1.20 (GND_{ISO}), C10.2, C11.2, C7.2, C8.2, C9.2, FB2.1, FB2.2
- net GND_ISO: now also U1.1 (GND_{1}), U1.10 (GND_{1}), U1.2 (GND_{1}), C1.2, C2.2, C3.2, C4.2, C5.2, C6.2
- net V_SOIN: now reaches U1.16 (V_{ISOIN})
- net V_SOIN: now also C11.1, C7.1, C8.1, FB1.2
- net V_SOOUT: now reaches U1.19 (V_{ISOOUT})
- net V_SOOUT: now also C10.1, FB1.1
- new net: C9.1, R2.2, R3.1
- no-connect marks 0 -> 2
Other:
- note removed: "INTERFAZ DE LA HOJA (pines jerárquicos)"
- note removed: "RIELES USADOS EN ESTA HOJA"
- moved on the sheet: R1, U1
