File: sheets/60_can.kicad_sch (KiCad schematic)
At the start: 19 parts, among them U601 ADM3055E

Commit message: [Claude Code] etapa 6: correcciones de la revisión independiente
- Stencil y pasta de gerbers sin aperturas en los 12 componentes DNP.
- Notes de C602 corregido (cadena tras C601, ~6 mm, aceptado).
- «K» de cátodo en serigrafía junto a D101-D103, D701 y D751.
- verify_etapa5: teardrops entre filas de U601 (0); regla ISO registrada como verificada.
- CPL/BOM de JLC (cpl_jlc.csv, bom_jlc.csv) sin THT ni U401, con rotaciones por
  familia (JLCKicadTools) y posición al centro de pads; cpl_proto.csv eliminado.
- Registrados como aceptados: H5 sin acero, par CAN asimétrico, C104 a 1.6 mm del
  borde y placa sin V-cut. Hallazgos 2 (imán) y 4 (courtyards) esperan aprobación.
DRC 0 errores / 3 avisos aceptados, 0 sin rutear, paridad 0; ERC sin cambios.

Co-Authored-By: Claude Opus 5.5 <noreply@anthropic.com>
Parts:
- C602: Notes VIO: 0.01 uF + 0.1 uF (ADM3055E Rev. D, tabla 10). < 2 mm d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 -> VIO: 0.01 uF + 0.1 uF (ADM3055E Rev. D, tabla 10). En caden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
Changed lines of the file:
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@@
 			)
 		)
-		(property "Notes" "VIO: 0.01 uF + 0.1 uF (ADM3055E Rev. D, tabla 10). < 2 mm del pin."
+		(property "Notes" "VIO: 0.01 uF + 0.1 uF (ADM3055E Rev. D, tabla 10). En cadena detrás de C601 (pin VIO → C601 10 nF → C602 100 nF), a ~6 mm del pin; ubicación aceptada por el usuario (2026-10-29)."
 			(at 109.22 175.26 0)
 			(hide yes)
