File: sheets/60_can.kicad_sch (KiCad schematic)
At the start: 19 parts, among them U601 ADM3055E

Commit message: [Claude Code] esquema+PCB: campos LCSC y sustitutos PROTO del BOM (pcb-v1-rc2)
- Esquema (solo campos, ocultos): LCSC en todos los componentes; MPN_PROTO,
  LCSC_PROTO y Manufacturer_PROTO con los sustitutos aceptados; Notes con
  compra y montaje (Q101, Q102, F101, L201, U503 a mano desde DigiKey/Mouser).
  MPN (PROD), valores, huellas y conexiones sin cambios. LCSC Part -> LCSC.
- PCB: mismos campos en las 145 huellas, insertados como texto (equivalente
  a F8 solo para campos); nada cambia fuera de las huellas.
- ERC por hoja igual que antes (0 errores, 5 avisos). DRC 0 errores / 3 avisos
  aceptados, 0 sin rutear, paridad 0 (antes de sincronizar: 145).
- etapa6_fab.py usa los campos _PROTO y genera bom_jlc_lcsc.csv; este y
  cpl_jlc.csv salen idénticos (60 líneas, 123 piezas). Gerbers sin cambios
  de contenido.

Co-Authored-By: Claude Opus 5.5 <noreply@anthropic.com>
Parts:
- C601: LCSC (none) -> C85863; LCSC_PROTO (none) -> C57112; MPN_PROTO (none) -> 0603B103K500NT; Manufacturer_PROTO (none) -> FH; Notes VIO: 0.01 uF + 0.1 uF (ADM3055E Rev. D, tabla 10). < 2 mm del pin. -> VIO: 0.01 uF + 0.1 uF (ADM3055E Rev. D, tabla 10). < 2 mm del pin. PROTO (2026-10-30): FH 0603B103K500NT (LCSC C57112, JLC basic), misma especificación, sin AEC-Q200.
- C602: LCSC (none) -> C85864; LCSC_PROTO (none) -> C14663; MPN_PROTO (none) -> CC0603KRX7R9BB104; Manufacturer_PROTO (none) -> Yageo; Notes VIO: 0.01 uF + 0.1 uF (ADM3055E Rev. D, tabla 10). En cadena detrás de C601 (pin VIO → C601 10 nF → C602 100 nF), a ~6 mm del pin; ubicación aceptada por el usuario (2026-10-29). -> VIO: 0.01 uF + 0.1 uF (ADM3055E Rev. D, tabla 10). En cadena detrás de C601 (pin VIO → C601 10 nF → C602 100 nF), a ~6 mm del pin; ubicación aceptada por el usuario (2026-10-29). PROTO (2026-10-30): Yageo CC0603KRX7R9BB104 (LCSC C14663, JLC basic), misma especificación, sin AEC-Q200.
- C603, C605, C606: LCSC (none) -> C126586
- C604: LCSC (none) -> C85864; LCSC_PROTO (none) -> C14663; MPN_PROTO (none) -> CC0603KRX7R9BB104; Manufacturer_PROTO (none) -> Yageo; Notes VCC: 10 uF + 0.1 uF (tabla 10). < 2 mm del pin. -> VCC: 10 uF + 0.1 uF (tabla 10). < 2 mm del pin. PROTO (2026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
- C607: LCSC (none) -> C85863; LCSC_PROTO (none) -> C57112; MPN_PROTO (none) -> 0603B103K500NT; Manufacturer_PROTO (none) -> FH; Notes VISOIN: 0.01 uF + 0.1 uF a GND2 (tabla 10). -> VISOIN: 0.01 uF + 0.1 uF a GND2 (tabla 10). PROTO (2026-10-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
- C608: LCSC (none) -> C85864; LCSC_PROTO (none) -> C14663; MPN_PROTO (none) -> CC0603KRX7R9BB104; Manufacturer_PROTO (none) -> Yageo; Notes VISOIN: 0.01 uF + 0.1 uF a GND2 (tabla 10). -> VISOIN: 0.01 uF + 0.1 uF a GND2 (tabla 10). PROTO (2026-10-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
- C609: LCSC (none) -> C426631
- C610: LCSC (none) -> C161217; LCSC_PROTO (none) -> C21120; MPN_PROTO (none) -> CL10B224KA8NNNC; Manufacturer_PROTO (none) -> Samsung; Notes VISOOUT: 0.22 uF + 10 uF a GNDISO (tabla 10). -> VISOOUT: 0.22 uF + 10 uF a GNDISO (tabla 10). PROTO (2026-1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
- D601: LCSC (none) -> C5736151
- FB601, FB602: LCSC (none) -> C113020
- R601: LCSC (none) -> C116677; LCSC_PROTO (none) -> C25804; MPN_PROTO (none) -> 0603WAF1002T5E; Manufacturer_PROTO (none) -> UNI-ROYAL; Notes Pull-down de SILENT (el ADM3055E ya tiene pull-down interno; refuerza el modo normal). -> Pull-down de SILENT (el ADM3055E ya tiene pull-down interno; refuerza el modo normal). PROTO (2026-10-30): UNI-ROYAL 0603WAF1002T5E (LCSC C25804, JLC basic), misma especificación, sin AEC-Q200.
- R602, R603: LCSC (none) -> C144645
- R604: LCSC (none) -> C116677; LCSC_PROTO (none) -> C25804; MPN_PROTO (none) -> 0603WAF1002T5E; Manufacturer_PROTO (none) -> UNI-ROYAL; Notes Pull-up de STBY a VIO: el transceiver arranca en standby (bus en silencio) hasta que el firmware baje CAN_STBY. Decision 60_can #5. -> Pull-up de STBY a VIO: el transceiver arranca en standby (bus en silencio) hasta que el firmware baje CAN_STBY. Decision 60_can #5. PROTO (2026-10-30): UNI-ROYAL 0603WAF1002T5E (LCSC C25804, JLC basic), misma especificación, sin AEC-Q200.
- R605: LCSC (none) -> C141796; LCSC_PROTO (none) -> C21189; MPN_PROTO (none) -> 0603WAF0000T5E; Manufacturer_PROTO (none) -> UNI-ROYAL; Notes RS a GND2: 0 ohm = velocidad completa (tabla 10). Para control de pendiente (EMI) montar 47k. -> RS a GND2: 0 ohm = velocidad completa (tabla 10). Para control de pendiente (EMI) montar 47k. PROTO (2026-10-30): UNI-ROYAL 0603WAF0000T5E (LCSC C21189, JLC basic), misma especificación, sin AEC-Q200.
- U601: LCSC (none) -> C658104; LCSC_PROTO (none) -> C658105; MPN_PROTO (none) -> ADM3055EBRIZ-RL; Notes ADM3055E Rev. D: RS a GND2 por R605, AUXIN a GND1 (sin uso), AUXOUT sin conexion. GNDISO por FB602 a GND2. Verificar el land pattern SOIC-20W contra el plano RI-20-1. -> ADM3055E Rev. D: RS a GND2 por R605, AUXIN a GND1 (sin uso), AUXOUT sin conexion. GNDISO por FB602 a GND2. Verificar el land pattern SOIC-20W contra el plano RI-20-1. PROTO (2026-10-30): ADM3055EBRIZ-RL (LCSC C658105), mismo CI en carrete; JLC tenía 55 u. PROD (100 u): comprar ADM3055EBRIZ en DigiKey/Mouser.

Commit message: [Claude Code] bom: compra principal en LCSC + DigiKey/Mouser; consolidación de pasivos
- Plan: JLC solo PCB + stencil Top; componentes de LCSC soldados a mano.
- Consolidación (solo valor/campos): R702/R752 4k7 → 2.2k; 23 × 100 nF a un
  MPN de 100 V X7R; PROTO 1 µF 50 V y 10 µF 25 V X7R. BOM PROTO 70 → 68 líneas.
- LCSC_BOM_COMPLETO_PROTO.csv: 6 juegos, 62 líneas, USD 552.43 (3 juegos: 286.65).
- DIGIKEY_MOUSER.csv: L201, U503, Q101, Q102, F101 (0 en LCSC), ≈ USD 99.54.
- Resumen de costos en BOM_SOURCING.md; archivos de JLC al día como alternativa.
- DRC 0 errores / 3 avisos aceptados, paridad 0, ERC 0 / 5.

Co-Authored-By: Claude Opus 5.5 <noreply@anthropic.com>
Parts:
- C602: LCSC C85864 -> C415406; LCSC_PROTO C14663 -> C88219; MPN GCM188R71H104KA57D -> GCM188R72A104KA64D; MPN_PROTO CC0603KRX7R9BB104 -> 0603B104K101NT; Manufacturer_PROTO Yageo -> FH; Notes VIO: 0.01 uF + 0.1 uF (ADM3055E Rev. D, tabla 10). En cadena detrás de C601 (pin VIO → C601 10 nF → C602 100 nF), a ~6 mm del pin; ubicación aceptada por el usuario (2026-10-29). PROTO (2026-10-30): Yageo CC0603KRX7R9BB104 (LCSC C14663, JLC basic), misma especificación, sin AEC-Q200. -> VIO: 0.01 uF + 0.1 uF (ADM3055E Rev. D, tabla 10). En cadena detrás de C601 (pin VIO → C601 10 nF → C602 100 nF), a ~6 mm del pin; ubicación aceptada por el usuario (2026-10-29). PROTO (2026-10-30, consolidacion): un solo MPN para los 100 nF 0603: 100 V X7R (FH 0603B104K101NT, LCSC C88219), sin AEC-Q200. PROD: Murata GCM188R72A104KA64D (100 V, AEC-Q200). Mismo valor y tolerancia.
- C603: LCSC_PROTO (none) -> C3039694; MPN_PROTO (none) -> CL21B106KAYQNNE; Manufacturer_PROTO (none) -> Samsung; Notes VCC (isoPower): 10 uF + 0.1 uF (tabla 10). Picos de 180-260 mA. 0805 por DC bias a 5 V. -> VCC (isoPower): 10 uF + 0.1 uF (tabla 10). Picos de 180-260 mA. 0805 por DC bias a 5 V. PROTO (2026-10-30, consolidacion): Samsung CL21B106KAYQNNE (25 V X7R, LCSC C3039694), sin AEC-Q200: el original no tiene stock en lcsc.com.
- C604: LCSC C85864 -> C415406; LCSC_PROTO C14663 -> C88219; MPN GCM188R71H104KA57D -> GCM188R72A104KA64D; MPN_PROTO CC0603KRX7R9BB104 -> 0603B104K101NT; Manufacturer_PROTO Yageo -> FH; Notes VCC: 10 uF + 0.1 uF (tabla 10). < 2 mm del pin. PROTO (2026-10-30): Yageo CC0603KRX7R9BB104 (LCSC C14663, JLC basic), misma especificación, sin AEC-Q200. -> VCC: 10 uF + 0.1 uF (tabla 10). < 2 mm del pin. PROTO (2026-10-30, consolidacion): un solo MPN para los 100 nF 0603: 100 V X7R (FH 0603B104K101NT, LCSC C88219), sin AEC-Q200. PROD: Murata GCM188R72A104KA64D (100 V, AEC-Q200). Mismo valor y tolerancia.
- C605: LCSC_PROTO (none) -> C3039694; MPN_PROTO (none) -> CL21B106KAYQNNE; Manufacturer_PROTO (none) -> Samsung; Notes Reserva local de +3V3_D en VIO (no la exige el datasheet). 0805 por DC bias. -> Reserva local de +3V3_D en VIO (no la exige el datasheet). 0805 por DC bias. PROTO (2026-10-30, consolidacion): Samsung CL21B106KAYQNNE (25 V X7R, LCSC C3039694), sin AEC-Q200: el original no tiene stock en lcsc.com.
- C606: LCSC_PROTO (none) -> C3039694; MPN_PROTO (none) -> CL21B106KAYQNNE; Manufacturer_PROTO (none) -> Samsung; Notes VISOOUT: 0.22 uF + 10 uF a GNDISO (tabla 10). 0805 por DC bias. -> VISOOUT: 0.22 uF + 10 uF a GNDISO (tabla 10). 0805 por DC bias. PROTO (2026-10-30, consolidacion): Samsung CL21B106KAYQNNE (25 V X7R, LCSC C3039694), sin AEC-Q200: el original no tiene stock en lcsc.com.
- C608: LCSC C85864 -> C415406; LCSC_PROTO C14663 -> C88219; MPN GCM188R71H104KA57D -> GCM188R72A104KA64D; MPN_PROTO CC0603KRX7R9BB104 -> 0603B104K101NT; Manufacturer_PROTO Yageo -> FH; Notes VISOIN: 0.01 uF + 0.1 uF a GND2 (tabla 10). PROTO (2026-10-30): Yageo CC0603KRX7R9BB104 (LCSC C14663, JLC basic), misma especificación, sin AEC-Q200. -> VISOIN: 0.01 uF + 0.1 uF a GND2 (tabla 10). PROTO (2026-10-30, consolidacion): un solo MPN para los 100 nF 0603: 100 V X7R (FH 0603B104K101NT, LCSC C88219), sin AEC-Q200. PROD: Murata GCM188R72A104KA64D (100 V, AEC-Q200). Mismo valor y tolerancia.
Changed lines of the file:
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@@
 			)
 		)
-		(property "MPN" "GCM188R71H104KA57D"
+		(property "MPN" "GCM188R72A104KA64D"
 			(at 295.91 160.02 0)
 			(hide yes)
@@
 			)
 		)
-		(property "Notes" "VISOIN: 0.01 uF + 0.1 uF a GND2 (tabla 10). PROTO (2026-10-30): Yageo CC0603KRX7R9BB104 (LCSC C14663, JLC basic), misma especificación, sin AEC-Q200."
+		(property "Notes" "VISOIN: 0.01 uF + 0.1 uF a GND2 (tabla 10). PROTO (2026-10-30, consolidacion): un solo MPN para los 100 nF 0603: 100 V X7R (FH 0603B104K101NT, LCSC C88219), sin AEC-Q200. PROD: Murata GCM188R72A104KA64D (100 V, AEC-Q200). Mismo valor y tolerancia."
 			(at 295.91 160.02 0)
 			(hide yes)
@@
 			)
 		)
-		(property "LCSC" "C85864"
+		(property "LCSC" "C415406"
 			(at 295.91 160.02 0)
 			(hide yes)
@@
 			)
 		)
-		(property "MPN_PROTO" "CC0603KRX7R9BB104"
+		(property "MPN_PROTO" "0603B104K101NT"
 			(at 295.91 160.02 0)
 			(hide yes)
@@
 			)
 		)
-		(property "Manufacturer_PROTO" "Yageo"
+		(property "Manufacturer_PROTO" "FH"
 			(at 295.91 160.02 0)
 			(hide yes)
@@
 			)
 		)
-		(property "LCSC_PROTO" "C14663"
+		(property "LCSC_PROTO" "C88219"
 			(at 295.91 160.02 0)
 			(hide yes)
@@
 			)
 		)
-		(property "Notes" "Reserva local de +3V3_D en VIO (no la exige el datasheet). 0805 por DC bias."
+		(property "Notes" "Reserva local de +3V3_D en VIO (no la exige el datasheet). 0805 por DC bias. PROTO (2026-10-30, consolidacion): Samsung CL21B106KAYQNNE (25 V X7R, LCSC C3039694), sin AEC-Q200: el original no tiene stock en lcsc.com."
 			(at 82.55 175.26 0)
 			(hide yes)
@@
 			)
 		)
+		(property "MPN_PROTO" "CL21B106KAYQNNE"
+			(at 82.55 175.26 0)
+			(hide yes)
+			(show_name no)
+			(do_not_autoplace no)
+			(effects
+				(font
+					(size 1.27 1.27)
+				)
+			)
+		)
+		(property "Manufacturer_PROTO" "Samsung"
+			(at 82.55 175.26 0)
+			(hide yes)
+			(show_name no)
+			(do_not_autoplace no)
+			(effects
+				(font
+					(size 1.27 1.27)
+				)
+			)
+		)
+		(property "LCSC_PROTO" "C3039694"
+			(at 82.55 175.26 0)
+			(hide yes)
+			(show_name no)
+			(do_not_autoplace no)
+			(effects
+				(font
+					(size 1.27 1.27)
+				)
+			)
+		)
 		(pin "1"
 		)
@@
 			)
 		)
-		(property "MPN" "GCM188R71H104KA57D"
+		(property "MPN" "GCM188R72A104KA64D"
 			(at 109.22 175.26 0)
 			(hide yes)
@@
 			)
 		)
-		(property "Notes" "VIO: 0.01 uF + 0.1 uF (ADM3055E Rev. D, tabla 10). En cadena detrás de C601 (pin VIO → C601 10 nF → C602 100 nF), a ~6 mm del pin; ubicación aceptada por el usuario (2026-10-29). PROTO (2026-10-30): Yageo CC0603KRX7R9BB104 (LCSC C14663, JLC basic), misma especificación, sin AEC-Q200."
+		(property "Notes" "VIO: 0.01 uF + 0.1 uF (ADM3055E Rev. D, tabla 10). En cadena detrás de C601 (pin VIO → C601 10 nF → C602 100 nF), a ~6 mm del pin; ubicación aceptada por el usuario (2026-10-29). PROTO (2026-10-30, consolidacion): un solo MPN para los 100 nF 0603: 100 V X7R (FH 0603B104K101NT, LCSC C88219), sin AEC-Q200. PROD: Murata GCM188R72A104KA64D (100 V, AEC-Q200). Mismo valor y tolerancia."
 			(at 109.22 175.26 0)
 			(hide yes)
@@
 			)
 		)
-		(property "LCSC" "C85864"
+		(property "LCSC" "C415406"
 			(at 109.22 175.26 0)
 			(hide yes)
@@
 			)
 		)
-		(property "MPN_PROTO" "CC0603KRX7R9BB104"
+		(property "MPN_PROTO" "0603B104K101NT"
 			(at 109.22 175.26 0)
 			(hide yes)
@@
 			)
 		)
-		(property "Manufacturer_PROTO" "Yageo"
+		(property "Manufacturer_PROTO" "FH"
 			(at 109.22 175.26 0)
 			(hide yes)
@@
 			)
 		)
-		(property "LCSC_PROTO" "C14663"
+		(property "LCSC_PROTO" "C88219"
 			(at 109.22 175.26 0)
 			(hide yes)
@@
 			)
 		)
-		(property "MPN" "GCM188R71H104KA57D"
+		(property "MPN" "GCM188R72A104KA64D"
 			(at 121.92 140.97 0)
 			(hide yes)
@@
 			)
 		)
-		(property "Notes" "VCC: 10 uF + 0.1 uF (tabla 10). < 2 mm del pin. PROTO (2026-10-30): Yageo CC0603KRX7R9BB104 (LCSC C14663, JLC basic), misma especificación, sin AEC-Q200."
+		(property "Notes" "VCC: 10 uF + 0.1 uF (tabla 10). < 2 mm del pin. PROTO (2026-10-30, consolidacion): un solo MPN para los 100 nF 0603: 100 V X7R (FH 0603B104K101NT, LCSC C88219), sin AEC-Q200. PROD: Murata GCM188R72A104KA64D (100 V, AEC-Q200). Mismo valor y tolerancia."
 			(at 121.92 140.97 0)
 			(hide yes)
@@
 			)
 		)
-		(property "LCSC" "C85864"
+		(property "LCSC" "C415406"
 			(at 121.92 140.97 0)
 			(hide yes)
@@
 			)
 		)
-		(property "MPN_PROTO" "CC0603KRX7R9BB104"
+		(property "MPN_PROTO" "0603B104K101NT"
 			(at 121.92 140.97 0)
 			(hide yes)
@@
 			)
 		)
-		(property "Manufacturer_PROTO" "Yageo"
+		(property "Manufacturer_PROTO" "FH"
 			(at 121.92 140.97 0)
 			(hide yes)
@@
 			)
 		)
-		(property "LCSC_PROTO" "C14663"
+		(property "LCSC_PROTO" "C88219"
 			(at 121.92 140.97 0)
 			(hide yes)
@@
 			)
 		)
-		(property "Notes" "VISOOUT: 0.22 uF + 10 uF a GNDISO (tabla 10). 0805 por DC bias."
+		(property "Notes" "VISOOUT: 0.22 uF + 10 uF a GNDISO (tabla 10). 0805 por DC bias. PROTO (2026-10-30, consolidacion): Samsung CL21B106KAYQNNE (25 V X7R, LCSC C3039694), sin AEC-Q200: el original no tiene stock en lcsc.com."
 			(at 259.08 195.58 0)
 			(hide yes)
@@
 			)
 		)
+		(property "MPN_PROTO" "CL21B106KAYQNNE"
+			(at 259.08 195.58 0)
+			(hide yes)
+			(show_name no)
+			(do_not_autoplace no)
+			(effects
+				(font
+					(size 1.27 1.27)
+				)
+			)
+		)
+		(property "Manufacturer_PROTO" "Samsung"
+			(at 259.08 195.58 0)
+			(hide yes)
+			(show_name no)
+			(do_not_autoplace no)
+			(effects
+				(font
+					(size 1.27 1.27)
+				)
+			)
+		)
+		(property "LCSC_PROTO" "C3039694"
+			(at 259.08 195.58 0)
+			(hide yes)
+			(show_name no)
+			(do_not_autoplace no)
+			(effects
+				(font
+					(size 1.27 1.27)
+				)
+			)
+		)
 		(pin "1"
 		)
@@
 			)
 		)
-		(property "Notes" "VCC (isoPower): 10 uF + 0.1 uF (tabla 10). Picos de 180-260 mA. 0805 por DC bias a 5 V."
+		(property "Notes" "VCC (isoPower): 10 uF + 0.1 uF (tabla 10). Picos de 180-260 mA. 0805 por DC bias a 5 V. PROTO (2026-10-30, consolidacion): Samsung CL21B106KAYQNNE (25 V X7R, LCSC C3039694), sin AEC-Q200: el original no tiene stock en lcsc.com."
 			(at 109.22 140.97 0)
 			(hide yes)
@@
 			(at 109.22 140.97 0)
 			(hide yes)
+			(show_name no)
+			(do_not_autoplace no)
+			(effects
+				(font
+					(size 1.27 1.27)
+				)
+			)
+		)
+		(property "MPN_PROTO" "CL21B106KAYQNNE"
+			(at 109.22 140.97 0)
+			(hide yes)
+			(show_name no)
+			(do_not_autoplace no)
+			(effects
+				(font
+					(size 1.27 1.27)
+				)
+			)
+		)
+		(property "Manufacturer_PROTO" "Samsung"
+			(at 109.22 140.97 0)
+			(hide yes)
+			(show_name no)
+			(do_not_autoplace no)
+			(effects
+				(font
+					(size 1.27 1.27)
+				)
+			)
+		)
+		(property "LCSC_PROTO" "C3039694"
+			(at 109.22 140.97 0)
+			(hide yes)
