File: sheets/60_can.kicad_sch (KiCad schematic)
At the start: 19 parts, among them U601 ADM3055E

Commit message: [Claude Code] rc7: JP601, selector de terminación CAN por puente de soldadura (pcb-v1-rc7)
- Hoja 60: JP601 (Jumper:SolderJumper_2_Open, abierto) en serie con R602; red nueva
  /60_can/CAN_TERM_H. Abierto = sin terminación; unido con estaño = 120 Ω. Fuera de BOM y CPL.
- PCB: JP601 en la cara inferior (114.6, 125.3), dentro de la isla GND_CAN, vías V1/V2,
  «TERM CAN» en B.Silkscreen. Sin mover componentes. CAN_TERM_H en ISO_CAN_barrera.
- ERC 0 errores / 5 avisos conocidos; DRC 0 errores / 3 avisos aceptados; paridad 0;
  716 teardrops; fab/proto regenerado.

Co-Authored-By: Claude Opus 5.5 <noreply@anthropic.com>
Parts:
- added JP601: TERM_CAN, Jumper:SolderJumper-2_P1.3mm_Open_RoundedPad1.0x1.5mm, symbol Jumper:SolderJumper_2_Open
- R602, R603: Notes Terminacion partida 2 x 60.4 ohm + C609. Montar solo en nod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 -> Terminacion partida 2 x 60.4 ohm + C609, siempre montada; s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
Connections:
- net BUS_CAN_H: now also JP601.1 (A); no longer R602.1
- new net CAN_TERM_H: JP601.2 (B), R602.1
Other:
- note added: "JP601 TERM CAN (cara inferior): abierto = sin terminacion; unido con estano = 120 ohm (nodo en el extremo del bus). Configurar en banco, antes de la caja."
Changed lines of the file:
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@@
 		(comment 2 "Inclinómetro de chasis CAN/BLE — INCLI-VA")
 	)
-	(text "BLOQUE 60 - CAN AISLADO (ADM3055E, barrera 2)   [Variant=CAN]\nFuente: datasheet ADI ADM3055E/ADM3057E Rev. D (tablas 10 y 12, PCB layout).\n\n  U601  ADM3055EBRIZ: CAN aislado con isoPower. VCC <- +5V_VEH (180 mA tip / 260 mA max en dominante), VIO <- +3V3_D.\n  Desacople (tabla 10): VCC 10 uF + 0.1 uF | VIO 0.01 + 0.1 uF | VISOIN 0.01 + 0.1 uF | VISOOUT 0.22 + 10 uF a GNDISO.\n  FB601 VISOOUT -> VISOIN y FB602 GNDISO -> GND2 (~2 kohm a 100 MHz-1 GHz; reducen emisiones, no son funcionales).\n  RS -> GND2 por R605 (0 ohm = velocidad completa; 47k = control de pendiente).  AUXIN -> GND1 (sin uso), AUXOUT sin conexion.\n  STBY: pull-up R604 -> arranca en standby hasta que el firmware baje CAN_STBY.  SILENT: pull-down R601 (normal).\n  Terminacion partida R602 + R603 + C609: montar solo en nodos de extremo del bus.\n  D601 ESD2CAN24-Q1 (SOT-23): DNP. El ADM3055E ya integra IEC 61000-4-2 +-8 kV y +-40 V de falla en CANH/CANL.\n\nCAN clasico (J1939) desde el TWAI del ESP32-S3: CAN_TX/CAN_RX directo al ADM3055E.\nLayout: capacitores a < 2 mm de los pines; verificar el land pattern SOIC-20W contra el plano RI-20-1 (creepage de la barrera 2)."
+	(text "BLOQUE 60 - CAN AISLADO (ADM3055E, barrera 2)   [Variant=CAN]\nFuente: datasheet ADI ADM3055E/ADM3057E Rev. D (tablas 10 y 12, PCB layout).\n\n  U601  ADM3055EBRIZ: CAN aislado con isoPower. VCC <- +5V_VEH (180 mA tip / 260 mA max en dominante), VIO <- +3V3_D.\n  Desacople (tabla 10): VCC 10 uF + 0.1 uF | VIO 0.01 + 0.1 uF | VISOIN 0.01 + 0.1 uF | VISOOUT 0.22 + 10 uF a GNDISO.\n  FB601 VISOOUT -> VISOIN y FB602 GNDISO -> GND2 (~2 kohm a 100 MHz-1 GHz; reducen emisiones, no son funcionales).\n  RS -> GND2 por R605 (0 ohm = velocidad completa; 47k = control de pendiente).  AUXIN -> GND1 (sin uso), AUXOUT sin conexion.\n  STBY: pull-up R604 -> arranca en standby hasta que el firmware baje CAN_STBY.  SILENT: pull-down R601 (normal).\n  Terminacion partida R602 + R603 + C609 (siempre montada) con JP601 en serie con R602: abierto = sin terminacion,\n  unido con estano = 120 ohm (nodo en el extremo del bus). JP601 en la cara inferior; se configura en banco, antes de la caja.\n  D601 ESD2CAN24-Q1 (SOT-23): DNP. El ADM3055E ya integra IEC 61000-4-2 +-8 kV y +-40 V de falla en CANH/CANL.\n\nCAN clasico (J1939) desde el TWAI del ESP32-S3: CAN_TX/CAN_RX directo al ADM3055E.\nLayout: capacitores a < 2 mm de los pines; verificar el land pattern SOIC-20W contra el plano RI-20-1 (creepage de la barrera 2)."
 		(exclude_from_sim no)
 		(at 20.32 20.32 0)
@@
 	(wire
 		(pts
-			(xy 284.48 101.6) (xy 281.94 101.6)
-		)
-		(stroke
-			(width 0)
-			(type default)
-		)
-	)
-	(wire
-		(pts
 			(xy 304.8 119.38) (xy 304.8 116.84)
 		)
@@
 	(hierarchical_label "BUS_CAN_H"
 		(shape bidirectional)
-		(at 281.94 101.6 180)
+		(at 274.32 101.6 180)
 		(effects
 			(font
@@
 		)
 	)
+	(label "CAN_TERM_H"
+		(at 284.48 101.6 0)
+		(effects
+			(font
+				(size 1.27 1.27)
+			)
+			(justify left bottom)
+		)
+	)
+	(text "JP601 TERM CAN (cara inferior): abierto = sin terminacion;\nunido con estano = 120 ohm (nodo en el extremo del bus).\nConfigurar en banco, antes de la caja."
+		(exclude_from_sim no)
+		(at 260.35 91.44 0)
+		(effects
+			(font
+				(size 1.27 1.27)
+			)
+			(justify left bottom)
+		)
+	)
+	(symbol
+		(lib_id "Jumper:SolderJumper_2_Open")
+		(at 279.4 101.6 0)
+		(unit 1)
+		(body_style 1)
+		(exclude_from_sim no)
+		(in_bom no)
+		(on_board yes)
+		(in_pos_files no)
+		(dnp no)
+		(property "Reference" "JP601"
+			(at 279.4 99.06 0)
+			(show_name no)
+			(do_not_autoplace no)
+			(effects
+				(font
+					(size 1.27 1.27)
+				)
+			)
+		)
+		(property "Value" "TERM_CAN"
+			(at 279.4 104.14 0)
+			(show_name no)
+			(do_not_autoplace no)
+			(effects
+				(font
+					(size 1.27 1.27)
+				)
+			)
+		)
+		(property "Footprint" "Jumper:SolderJumper-2_P1.3mm_Open_RoundedPad1.0x1.5mm"
+			(at 279.4 101.6 0)
+			(hide yes)
+			(show_name no)
+			(do_not_autoplace no)
+			(effects
+				(font
+					(size 1.27 1.27)
+				)
+			)
+		)
+		(property "Datasheet" "~"
+			(at 279.4 101.6 0)
+			(hide yes)
+			(show_name no)
+			(do_not_autoplace no)
+			(effects
+				(font
+					(size 1.27 1.27)
+				)
+			)
+		)
+		(property "Description" "Solder Jumper, 2-pole, open"
+			(at 279.4 101.6 0)
+			(hide yes)
+			(show_name no)
+			(do_not_autoplace no)
+			(effects
+				(font
+					(size 1.27 1.27)
+				)
+			)
+		)
+		(property "MPN" "N/A (puente de soldadura en el PCB)"
+			(at 279.4 101.6 0)
+			(hide yes)
+			(show_name no)
+			(do_not_autoplace no)
+			(effects
+				(font
+					(size 1.27 1.27)
+				)
+			)
+		)
+		(property "Manufacturer" "N/A (cobre de la placa)"
+			(at 279.4 101.6 0)
+			(hide yes)
+			(show_name no)
+			(do_not_autoplace no)
+			(effects
+				(font
+					(size 1.27 1.27)
+				)
+			)
+		)
+		(property "Notes" "Selector de terminacion CAN (puente de soldadura, ABIERTO por defecto), en serie con R602, cara inferior. Abierto = sin terminacion. Unido con estano = terminacion partida de 120 ohm activa (nodo en el extremo del bus). Se configura en banco, antes de montar la placa en la caja. Sin componente: fuera del BOM y del CPL. Con JP601 abierto, CANL sigue viendo R603 + C609 a GND_CAN (carga de modo comun asimetrica, sin carga en DC)."
+			(at 279.4 101.6 0)
+			(hide yes)
+			(show_name no)
+			(do_not_autoplace no)
+			(effects
+				(font
+					(size 1.27 1.27)
+				)
+			)
+		)
+		(property "Variant" "CAN"
+			(at 279.4 101.6 0)
+			(hide yes)
+			(show_name no)
+			(do_not_autoplace no)
+			(effects
+				(font
+					(size 1.27 1.27)
+				)
+			)
+		)
+		(pin "1"
+		)
+		(pin "2"
+		)
+		(instances
+			(project "INCLI-VA"
+				(path "/7fd92c2b-4254-4d73-93ba-bfde861bede3/3036af0c-b072-4a36-8ec1-d374aba21569"
+					(reference "JP601")
+					(unit 1)
+				)
+			)
+		)
+	)
 	(symbol
 		(lib_id "INCLI-VA:GND_VEH")
@@
 			)
 		)
-		(property "Notes" "Terminacion partida 2 x 60.4 ohm + C609. Montar solo en nodos de extremo del bus."
+		(property "Notes" "Terminacion partida 2 x 60.4 ohm + C609, siempre montada; se activa uniendo JP601 (en serie con R602). JP601 abierto = sin terminacion."
 			(at 284.48 127 0)
 			(hide yes)
@@
 			)
 		)
-		(property "Notes" "Terminacion partida 2 x 60.4 ohm + C609. Montar solo en nodos de extremo del bus (si el nodo no termina, R602/R603/C609 DNP)."
+		(property "Notes" "Terminacion partida 2 x 60.4 ohm + C609, siempre montada; se activa uniendo JP601 (en serie con R602). JP601 abierto = sin terminacion."
 			(at 284.48 107.95 0)
 			(hide yes)
