File: sheets/40_mcu_esp32s3.kicad_sch (KiCad schematic)
At the start: 20 parts, among them J401 USB4105-GF-A, J402 UART0, SW401 RESET, SW402 BOOT, U401 ESP32-S3-WROOM-1-N8R2, U402 USBLC6-2SC6

Commit message: [Claude Code] 80_supervision: TPS3828-33-Q1, LED y VAR_ID; J1/J2 verticales; contorno con muesca
- 80_supervision: U801 TPS3828-33QDBVRQ1 (supervisor de +3V3_D + watchdog,
  WDI <- IO17), R802 0 ohm, R801 DNP; LED verde/rojo DNP en PROD (caja
  opaca); VAR_ID0/1 (CAN/OUT) y VAR_ID2 (IO8, CABIN, DNP).
- WD_EN eliminado (IO18 libre); VAR_ID2 ocupa su pin en las hojas 40/80 y la raíz.
- 10_power_input: J1/J2 MSTBV 2,5 GF 5.08 verticales (1777109 / 1777073).
- lib: se borran los símbolos URB2405 y TPS7A1650; U101: vías del EP a Ø 0.45 mm.
- PCB: contorno único con muesca de 8 x 35 mm para la antena (antes, dos
  rectángulos superpuestos); serigrafía de U401 recortada en la muesca.
- ERC: 0 errores, 1 aviso intencional (U101_RTN).

Co-Authored-By: Claude Opus 5.5 <noreply@anthropic.com>
Connections:
- net VAR_ID2: now reaches U401.12 (IO8)
- net WD_EN: no longer names the net of U401.11 (IO18)
Changed lines of the file:
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@@
 		)
 	)
-	(text "ASIGNACIÓN DE PINES (aprobada 2026-10-27; fuentes: WROOM-1 v1.8 tabla 3-1, ESP32-S3 Series v2.2 tablas 2-1 y 2-2)\nCriterios: VMON solo en ADC1 (ADC2 no se puede usar con WiFi). GPIO1–14, 17, 18: glitch BAJO de ~60 µs al encender → solo CS, SCK,\nMOSI, LEDs, entradas resistivas o analógicas, WDI/WD_EN. Señales críticas en pines sin glitch ni pull: IO21, IO35–38, IO40–42, IO47/48.\nSPI en los pines IO MUX de FSPI. Strapping (0, 3, 45, 46), USB (19/20) y UART0 (43/44) reservados.\n\nIO12 SPI_SCK   IO11 SPI_MOSI   IO13 SPI_MISO   IO10 CS_INC (FSPICS0)   IO9 CS_IMU   IO14 CS_ROT\nIO40 IMU_INT1  IO41 IMU_INT2   (sin glitch: salida push-pull del IMU)\nIO47 CAN_TX (sin glitch: un bajo sería un dominante en el bus)   IO48 CAN_RX   IO21 CAN_STBY   IO42 CAN_SILENT\nIO35 DO1_EN  IO36 DO2_EN (sin glitch ni pull; R203/R204 en hoja 20)   IO37 DO1_DIAG  IO38 DO2_DIAG  IO39 PWR_FLT_N\nIO1 VMON_5V (ADC1_CH0)   IO2 VMON_3V3 (ADC1_CH1)   IO4 VAR_ID0   IO5 VAR_ID1   IO6 LED_G   IO7 LED_R\nIO17 WDI   IO18 WD_EN (requiere pull-down en la hoja 80)   Libres: IO8, IO15, IO16.\nRiesgo: IO39–42 son el JTAG por pads; se usa el JTAG por USB. No habilitar el JTAG por pads con eFuse."
+	(text "ASIGNACIÓN DE PINES (aprobada 2026-10-27; fuentes: WROOM-1 v1.8 tabla 3-1, ESP32-S3 Series v2.2 tablas 2-1 y 2-2)\nCriterios: VMON solo en ADC1 (ADC2 no se puede usar con WiFi). GPIO1–14, 17, 18: glitch BAJO de ~60 µs al encender → solo CS, SCK,\nMOSI, LEDs, entradas resistivas o analógicas, WDI/WD_EN. Señales críticas en pines sin glitch ni pull: IO21, IO35–38, IO40–42, IO47/48.\nSPI en los pines IO MUX de FSPI. Strapping (0, 3, 45, 46), USB (19/20) y UART0 (43/44) reservados.\n\nIO12 SPI_SCK   IO11 SPI_MOSI   IO13 SPI_MISO   IO10 CS_INC (FSPICS0)   IO9 CS_IMU   IO14 CS_ROT\nIO40 IMU_INT1  IO41 IMU_INT2   (sin glitch: salida push-pull del IMU)\nIO47 CAN_TX (sin glitch: un bajo sería un dominante en el bus)   IO48 CAN_RX   IO21 CAN_STBY   IO42 CAN_SILENT\nIO35 DO1_EN  IO36 DO2_EN (sin glitch ni pull; R203/R204 en hoja 20)   IO37 DO1_DIAG  IO38 DO2_DIAG  IO39 PWR_FLT_N\nIO1 VMON_5V (ADC1_CH0)   IO2 VMON_3V3 (ADC1_CH1)   IO4 VAR_ID0   IO5 VAR_ID1   IO6 LED_G   IO7 LED_R\nIO17 WDI (TPS3828, hoja 80)   IO8 VAR_ID2 (CABIN)   Libres: IO15, IO16, IO18.\nRiesgo: IO39–42 son el JTAG por pads; se usa el JTAG por USB. No habilitar el JTAG por pads con eFuse."
 		(exclude_from_sim no)
 		(at 21.336 227.838 0)
@@
 	)
 	(no_connect
-		(at 185.42 142.24)
-	)
-	(no_connect
 		(at 292.1 76.2)
 	)
@@
 	(wire
 		(pts
-			(xy 215.9 124.46) (xy 220.98 124.46)
-		)
-		(stroke
-			(width 0)
-			(type default)
-		)
-	)
-	(wire
-		(pts
 			(xy 350.52 121.92) (xy 355.6 121.92)
 		)
@@
 		)
 	)
-	(hierarchical_label "WD_EN"
-		(shape output)
-		(at 220.98 124.46 0)
-		(effects
-			(font
-				(size 1.27 1.27)
-			)
-			(justify left)
-		)
-	)
 	(hierarchical_label "VMON_5V"
 		(shape input)
@@
 		)
 	)
+	(no_connect
+		(at 215.9 124.46)
+	)
+	(wire
+		(pts
+			(xy 185.42 142.24) (xy 180.34 142.24)
+		)
+		(stroke
+			(width 0)
+			(type default)
+		)
+	)
+	(hierarchical_label "VAR_ID2"
+		(shape input)
+		(at 180.34 142.24 180)
+		(effects
+			(font
+				(size 1.27 1.27)
+			)
+			(justify right)
+		)
+	)
