File: sheets/40_mcu_esp32s3.kicad_sch (KiCad schematic)
At the start: 19 parts, among them J401 USB4105-GF-A, J402 UART0, SW401 RESET, SW402 BOOT, U401 ESP32-S3-WROOM-1-N8R2, U402 USBLC6-2SC6

Commit message: [Claude Code] esquema+PCB: campos LCSC y sustitutos PROTO del BOM (pcb-v1-rc2)
- Esquema (solo campos, ocultos): LCSC en todos los componentes; MPN_PROTO,
  LCSC_PROTO y Manufacturer_PROTO con los sustitutos aceptados; Notes con
  compra y montaje (Q101, Q102, F101, L201, U503 a mano desde DigiKey/Mouser).
  MPN (PROD), valores, huellas y conexiones sin cambios. LCSC Part -> LCSC.
- PCB: mismos campos en las 145 huellas, insertados como texto (equivalente
  a F8 solo para campos); nada cambia fuera de las huellas.
- ERC por hoja igual que antes (0 errores, 5 avisos). DRC 0 errores / 3 avisos
  aceptados, 0 sin rutear, paridad 0 (antes de sincronizar: 145).
- etapa6_fab.py usa los campos _PROTO y genera bom_jlc_lcsc.csv; este y
  cpl_jlc.csv salen idénticos (60 líneas, 123 piezas). Gerbers sin cambios
  de contenido.

Co-Authored-By: Claude Opus 5.5 <noreply@anthropic.com>
Parts:
- C401: LCSC (none) -> C907991
- C402: LCSC (none) -> C85864; LCSC_PROTO (none) -> C14663; MPN_PROTO (none) -> CC0603KRX7R9BB104; Manufacturer_PROTO (none) -> Yageo; Notes Desacople de alta frecuencia, pegado al pin 3V3 del módulo. -> Desacople de alta frecuencia, pegado al pin 3V3 del módulo.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
- C403: LCSC (none) -> C161212
- C404: LCSC (none) -> C85864; LCSC_PROTO (none) -> C14663; MPN_PROTO (none) -> CC0603KRX7R9BB104; Manufacturer_PROTO (none) -> Yageo; Notes Desacople VBUS del USBLC6-2SC6: 100 nF, X7R, 50 V, 0603; no alimenta el riel +5V. Agregado despues de placement-v1, autorizado en etapa 3. -> Desacople VBUS del USBLC6-2SC6: 100 nF, X7R, 50 V, 0603; no alimenta el riel +5V. Agregado despues de placement-v1, autorizado en etapa 3. PROTO (2026-10-30): Yageo CC0603KRX7R9BB104 (LCSC C14663, JLC basic), misma especificación, sin AEC-Q200.
- J401: LCSC (none) -> C3020560; Notes USB-C solo USB 2.0 para el USB-Serial-JTAG del ESP32-S3 (GPIO19/20). Programación, consola y JTAG. Masa = GND_VEH: SIN aislamiento (opción B), la PC comparte masa con el vehículo; en el vehículo usar aislador USB/UART o laptop a batería. Blindaje a GND_VEH. -> USB-C solo USB 2.0 para el USB-Serial-JTAG del ESP32-S3 (GPIO19/20). Programación, consola y JTAG. Masa = GND_VEH: SIN aislamiento (opción B), la PC comparte masa con el vehículo; en el vehículo usar aislador USB/UART o laptop a batería. Blindaje a GND_VEH. Montaje: soldar a mano; comprar en LCSC (C3020560).
- J402: LCSC (none) -> C2915006; LCSC_PROTO (none) -> C49257; MPN_PROTO (none) -> 2.54-1*3PPin; Manufacturer_PROTO (none) -> BOOMELE; Notes UART0 para logs: 1 = TXD0 (IO43, sale del MCU), 2 = RXD0 (IO44), 3 = GND_VEH. Adaptador USB-UART de 3.3 V. -> UART0 para logs: 1 = TXD0 (IO43, sale del MCU), 2 = RXD0 (IO44), 3 = GND_VEH. Adaptador USB-UART de 3.3 V. PROTO (2026-10-30): tira 1x3 de 2.54 mm genérica BOOMELE 2.54-1*3PPin (LCSC C49257), misma huella; la Würth no está en lcsc.com. Soldar a mano (THT).
- R401: LCSC (none) -> C116677; LCSC_PROTO (none) -> C25804; MPN_PROTO (none) -> 0603WAF1002T5E; Manufacturer_PROTO (none) -> UNI-ROYAL; Notes Pull-up de EN (RC de Espressif: 10k + 1 uF). También es el pull-up del WDO (drenador abierto) del TPS3828 en 80_supervision. -> Pull-up de EN (RC de Espressif: 10k + 1 uF). También es el pull-up del WDO (drenador abierto) del TPS3828 en 80_supervision. PROTO (2026-10-30): UNI-ROYAL 0603WAF1002T5E (LCSC C25804, JLC basic), misma especificación, sin AEC-Q200.
- R402: LCSC (none) -> C116677; LCSC_PROTO (none) -> C25804; MPN_PROTO (none) -> 0603WAF1002T5E; Manufacturer_PROTO (none) -> UNI-ROYAL; Notes Pull-up externo de GPIO0 (strapping: 1 = arranque desde flash). No depende del pull-up interno. -> Pull-up externo de GPIO0 (strapping: 1 = arranque desde flash). No depende del pull-up interno. PROTO (2026-10-30): UNI-ROYAL 0603WAF1002T5E (LCSC C25804, JLC basic), misma especificación, sin AEC-Q200.
- R403: LCSC (none) -> C125891; LCSC_PROTO (none) -> C23186; MPN_PROTO (none) -> 0603WAF5101T5E; Manufacturer_PROTO (none) -> UNI-ROYAL; Notes Rd de CC1 (5.1k a GND): identifica a la placa como dispositivo USB-C. -> Rd de CC1 (5.1k a GND): identifica a la placa como dispositivo USB-C. PROTO (2026-10-30): UNI-ROYAL 0603WAF5101T5E (LCSC C23186, JLC basic), misma especificación, sin AEC-Q200.
- R404: LCSC (none) -> C125891; LCSC_PROTO (none) -> C23186; MPN_PROTO (none) -> 0603WAF5101T5E; Manufacturer_PROTO (none) -> UNI-ROYAL; Notes Rd de CC2 (5.1k a GND): identifica a la placa como dispositivo USB-C. -> Rd de CC2 (5.1k a GND): identifica a la placa como dispositivo USB-C. PROTO (2026-10-30): UNI-ROYAL 0603WAF5101T5E (LCSC C23186, JLC basic), misma especificación, sin AEC-Q200.
- SW401, SW402: LCSC (none) -> C720477; LCSC Part C720477 -> (none)
- U401: LCSC (none) -> C2913204; Notes 8 MB flash quad + 2 MB PSRAM quad, antena PCB, -40 a +85 C (las variantes R8/R16 con PSRAM octal llegan solo a 65 C). PSRAM quad: IO35-IO37 libres (WROOM-1 v1.8, tabla 3-1, nota b). LCSC C2913204. Pad 41 (EPAD) y pines 1/40 a GND_VEH. Antena al borde de la placa con keepout (ver nota de layout). IMPORTANTE: IO35-IO37 se usan como GPIO (DO1_EN, DO2_EN, DO1_DIAG); solo es valido con PSRAM quad (N8R2) o sin PSRAM. NO reemplazar por variantes con PSRAM octal (R8). -> 8 MB flash quad + 2 MB PSRAM quad, antena PCB, -40 a +85 C (las variantes R8/R16 con PSRAM octal llegan solo a 65 C). PSRAM quad: IO35-IO37 libres (WROOM-1 v1.8, tabla 3-1, nota b). LCSC C2913204. Pad 41 (EPAD) y pines 1/40 a GND_VEH. Antena al borde de la placa con keepout (ver nota de layout). IMPORTANTE: IO35-IO37 se usan como GPIO (DO1_EN, DO2_EN, DO1_DIAG); solo es valido con PSRAM quad (N8R2) o sin PSRAM. NO reemplazar por variantes con PSRAM octal (R8). Montaje: soldar a mano; comprar en LCSC (C2913204).
- U402: LCSC (none) -> C2687116

Commit message: [Claude Code] TP de la cara inferior rotulados, TP406/TP505 GND con agujero, R803/R804 2.2k
- B.Silk: nombre de señal junto a cada TP (verificado con la red), GND con recuadro,
  nota «CAN: medir vs GND_CAN (J1-5)».
- TP406 (40_mcu) y TP505 (50_sensors): GND_VEH THT D2.5/1.2 mm, en esquema y PCB,
  fuera de BOM/CPL.
- LEDs: R803/R804 470 → 2.2k (0603WAF2201T5E C4190 basic; PROD AC0603FR-072K2L);
  ~0.61 / 0.70 mA; brillo por PWM (PENDIENTES, firmware).
- DRC 0 errores / 3 avisos aceptados, paridad 0, ERC 0 / 5; fab/proto y BOM regenerados.

Co-Authored-By: Claude Opus 5.5 <noreply@anthropic.com>
Parts:
- added TP406: GND_VEH, TestPoint:TestPoint_THTPad_D2.5mm_Drill1.2mm, symbol Connector:TestPoint
Connections:
- net GND_VEH: now also TP406.1
Changed lines of the file:
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@@
 	(wire (pts (xy 365.76 67.31) (xy 365.76 73.66)) (stroke (width 0) (type default)))
 	(label "VBUS" (at 365.76 55.88 0) (effects (font (size 1.27 1.27)) (justify left bottom)))
+	(symbol
+		(lib_id "Connector:TestPoint")
+		(at 322.58 205.74 0)
+		(unit 1)
+		(body_style 1)
+		(exclude_from_sim no)
+		(in_bom no)
+		(on_board yes)
+		(in_pos_files no)
+		(dnp no)
+		(property "Reference" "TP406"
+			(at 323.85 200.66 0)
+			(show_name no)
+			(do_not_autoplace no)
+			(effects
+				(font
+					(size 1.27 1.27)
+				)
+				(justify left)
+			)
+		)
+		(property "Value" "GND_VEH"
+			(at 323.85 202.57 0)
+			(show_name no)
+			(do_not_autoplace no)
+			(effects
+				(font
+					(size 1.27 1.27)
+				)
+				(justify left)
+			)
+		)
+		(property "Footprint" "TestPoint:TestPoint_THTPad_D2.5mm_Drill1.2mm"
+			(at 322.58 205.74 0)
+			(hide yes)
+			(show_name no)
+			(do_not_autoplace no)
+			(effects
+				(font
+					(size 1.27 1.27)
+				)
+			)
+		)
+		(property "Datasheet" "N/A (pad de prueba)"
+			(at 322.58 205.74 0)
+			(hide yes)
+			(show_name no)
+			(do_not_autoplace no)
+			(effects
+				(font
+					(size 1.27 1.27)
+				)
+			)
+		)
+		(property "Description" ""
+			(at 322.58 205.74 0)
+			(hide yes)
+			(show_name no)
+			(do_not_autoplace no)
+			(effects
+				(font
+					(size 1.27 1.27)
+				)
+			)
+		)
+		(property "MPN" "-"
+			(at 322.58 205.74 0)
+			(hide yes)
+			(show_name no)
+			(do_not_autoplace no)
+			(effects
+				(font
+					(size 1.27 1.27)
+				)
+			)
+		)
+		(property "Manufacturer" "-"
+			(at 322.58 205.74 0)
+			(hide yes)
+			(show_name no)
+			(do_not_autoplace no)
+			(effects
+				(font
+					(size 1.27 1.27)
+				)
+			)
+		)
+		(property "Notes" "Punto de prueba de GND_VEH con agujero (pad 2.5 mm, taladro 1.2 mm) para el caiman o la punta de masa del osciloscopio; admite un lazo de alambre o un Keystone 5001 soldado a mano. Fuera del BOM y del CPL de JLC."
+			(at 322.58 205.74 0)
+			(hide yes)
+			(show_name no)
+			(do_not_autoplace no)
+			(effects
+				(font
+					(size 1.27 1.27)
+				)
+			)
+		)
+		(property "DNP" ""
+			(at 322.58 205.74 0)
+			(hide yes)
+			(show_name no)
+			(do_not_autoplace no)
+			(effects
+				(font
+					(size 1.27 1.27)
+				)
+			)
+		)
+		(pin "1"
+		)
+		(instances
+			(project "INCLI-VA"
+				(path "/7fd92c2b-4254-4d73-93ba-bfde861bede3/712b3cf0-3806-4b78-89c5-204f7bed5fb6"
+					(reference "TP406")
+					(unit 1)
+				)
+			)
+		)
+	)
+	(symbol
+		(lib_id "INCLI-VA:GND_VEH")
+		(at 322.58 205.74 0)
+		(unit 1)
+		(body_style 1)
+		(exclude_from_sim no)
+		(in_bom no)
+		(on_board yes)
+		(in_pos_files no)
+		(dnp no)
+		(property "Reference" "#PWR490"
+			(at 322.58 212.09 0)
+			(hide yes)
+			(show_name no)
+			(do_not_autoplace no)
+			(effects
+				(font
+					(size 1.27 1.27)
+				)
+			)
+		)
+		(property "Value" "GND_VEH"
+			(at 322.58 209.55 0)
+			(show_name no)
+			(do_not_autoplace no)
+			(effects
+				(font
+					(size 1.27 1.27)
+				)
+			)
+		)
+		(property "Footprint" ""
+			(at 322.58 205.74 0)
+			(hide yes)
+			(show_name no)
+			(do_not_autoplace no)
+			(effects
+				(font
+					(size 1.27 1.27)
+				)
+			)
+		)
+		(property "Datasheet" ""
+			(at 322.58 205.74 0)
+			(hide yes)
+			(show_name no)
+			(do_not_autoplace no)
+			(effects
+				(font
+					(size 1.27 1.27)
+				)
+			)
+		)
+		(property "Description" ""
+			(at 322.58 205.74 0)
+			(hide yes)
+			(show_name no)
+			(do_not_autoplace no)
+			(effects
+				(font
+					(size 1.27 1.27)
+				)
+			)
+		)
+		(pin "1"
+		)
+		(instances
+			(project "INCLI-VA"
+				(path "/7fd92c2b-4254-4d73-93ba-bfde861bede3/712b3cf0-3806-4b78-89c5-204f7bed5fb6"
+					(reference "#PWR490")
+					(unit 1)
+				)
+			)
+		)
+	)
 )

Commit message: [Claude Code] bom: compra principal en LCSC + DigiKey/Mouser; consolidación de pasivos
- Plan: JLC solo PCB + stencil Top; componentes de LCSC soldados a mano.
- Consolidación (solo valor/campos): R702/R752 4k7 → 2.2k; 23 × 100 nF a un
  MPN de 100 V X7R; PROTO 1 µF 50 V y 10 µF 25 V X7R. BOM PROTO 70 → 68 líneas.
- LCSC_BOM_COMPLETO_PROTO.csv: 6 juegos, 62 líneas, USD 552.43 (3 juegos: 286.65).
- DIGIKEY_MOUSER.csv: L201, U503, Q101, Q102, F101 (0 en LCSC), ≈ USD 99.54.
- Resumen de costos en BOM_SOURCING.md; archivos de JLC al día como alternativa.
- DRC 0 errores / 3 avisos aceptados, paridad 0, ERC 0 / 5.

Co-Authored-By: Claude Opus 5.5 <noreply@anthropic.com>
Parts:
- C402: LCSC C85864 -> C415406; LCSC_PROTO C14663 -> C88219; MPN GCM188R71H104KA57D -> GCM188R72A104KA64D; MPN_PROTO CC0603KRX7R9BB104 -> 0603B104K101NT; Manufacturer_PROTO Yageo -> FH; Notes Desacople de alta frecuencia, pegado al pin 3V3 del módulo. PROTO (2026-10-30): Yageo CC0603KRX7R9BB104 (LCSC C14663, JLC basic), misma especificación, sin AEC-Q200. -> Desacople de alta frecuencia, pegado al pin 3V3 del módulo. PROTO (2026-10-30, consolidacion): un solo MPN para los 100 nF 0603: 100 V X7R (FH 0603B104K101NT, LCSC C88219), sin AEC-Q200. PROD: Murata GCM188R72A104KA64D (100 V, AEC-Q200). Mismo valor y tolerancia.
- C403: LCSC_PROTO (none) -> C559769; MPN_PROTO (none) -> CC0603KRX7R9BB105; Manufacturer_PROTO (none) -> Yageo; Notes Retardo de EN (Espressif: 1 uF; tau = 10 ms) para que EN suba después de que 3V3 esté estable. MPN a verificar (disponibilidad y especificación) antes de congelar el BOM. -> Retardo de EN (Espressif: 1 uF; tau = 10 ms) para que EN suba después de que 3V3 esté estable. MPN a verificar (disponibilidad y especificación) antes de congelar el BOM. PROTO (2026-10-30, consolidacion): Yageo CC0603KRX7R9BB105 (50 V X7R, LCSC C559769), sin AEC-Q200: mas stock y menos perdida por DC bias.
- C404: LCSC C85864 -> C415406; LCSC_PROTO C14663 -> C88219; MPN GCM188R71H104KA57D -> GCM188R72A104KA64D; MPN_PROTO CC0603KRX7R9BB104 -> 0603B104K101NT; Manufacturer_PROTO Yageo -> FH; Notes Desacople VBUS del USBLC6-2SC6: 100 nF, X7R, 50 V, 0603; no alimenta el riel +5V. Agregado despues de placement-v1, autorizado en etapa 3. PROTO (2026-10-30): Yageo CC0603KRX7R9BB104 (LCSC C14663, JLC basic), misma especificación, sin AEC-Q200. -> Desacople VBUS del USBLC6-2SC6: 100 nF, X7R, 50 V, 0603; no alimenta el riel +5V. Agregado despues de placement-v1, autorizado en etapa 3. PROTO (2026-10-30, consolidacion): un solo MPN para los 100 nF 0603: 100 V X7R (FH 0603B104K101NT, LCSC C88219), sin AEC-Q200. PROD: Murata GCM188R72A104KA64D (100 V, AEC-Q200). Mismo valor y tolerancia.
Changed lines of the file:
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@@
 			)
 		)
-		(property "MPN" "GCM188R71H104KA57D"
+		(property "MPN" "GCM188R72A104KA64D"
 			(at 180.34 95.25 0)
 			(hide yes)
@@
 			)
 		)
-		(property "Notes" "Desacople de alta frecuencia, pegado al pin 3V3 del módulo. PROTO (2026-10-30): Yageo CC0603KRX7R9BB104 (LCSC C14663, JLC basic), misma especificación, sin AEC-Q200."
+		(property "Notes" "Desacople de alta frecuencia, pegado al pin 3V3 del módulo. PROTO (2026-10-30, consolidacion): un solo MPN para los 100 nF 0603: 100 V X7R (FH 0603B104K101NT, LCSC C88219), sin AEC-Q200. PROD: Murata GCM188R72A104KA64D (100 V, AEC-Q200). Mismo valor y tolerancia."
 			(at 180.34 95.25 0)
 			(hide yes)
@@
 			)
 		)
-		(property "LCSC" "C85864"
+		(property "LCSC" "C415406"
 			(at 180.34 95.25 0)
 			(hide yes)
@@
 			)
 		)
-		(property "MPN_PROTO" "CC0603KRX7R9BB104"
+		(property "MPN_PROTO" "0603B104K101NT"
 			(at 180.34 95.25 0)
 			(hide yes)
@@
 			)
 		)
-		(property "Manufacturer_PROTO" "Yageo"
+		(property "Manufacturer_PROTO" "FH"
 			(at 180.34 95.25 0)
 			(hide yes)
@@
 			)
 		)
-		(property "LCSC_PROTO" "C14663"
+		(property "LCSC_PROTO" "C88219"
 			(at 180.34 95.25 0)
 			(hide yes)
@@
 			)
 		)
-		(property "Notes" "Retardo de EN (Espressif: 1 uF; tau = 10 ms) para que EN suba después de que 3V3 esté estable. MPN a verificar (disponibilidad y especificación) antes de congelar el BOM."
+		(property "Notes" "Retardo de EN (Espressif: 1 uF; tau = 10 ms) para que EN suba después de que 3V3 esté estable. MPN a verificar (disponibilidad y especificación) antes de congelar el BOM. PROTO (2026-10-30, consolidacion): Yageo CC0603KRX7R9BB105 (50 V X7R, LCSC C559769), sin AEC-Q200: mas stock y menos perdida por DC bias."
 			(at 116.84 120.65 0)
 			(hide yes)
@@
 		)
 		(property "LCSC" "C161212"
+			(at 116.84 120.65 0)
+			(hide yes)
+			(show_name no)
+			(do_not_autoplace no)
+			(effects
+				(font
+					(size 1.27 1.27)
+				)
+			)
+		)
+		(property "MPN_PROTO" "CC0603KRX7R9BB105"
+			(at 116.84 120.65 0)
+			(hide yes)
+			(show_name no)
+			(do_not_autoplace no)
+			(effects
+				(font
+					(size 1.27 1.27)
+				)
+			)
+		)
+		(property "Manufacturer_PROTO" "Yageo"
+			(at 116.84 120.65 0)
+			(hide yes)
+			(show_name no)
+			(do_not_autoplace no)
+			(effects
+				(font
+					(size 1.27 1.27)
+				)
+			)
+		)
+		(property "LCSC_PROTO" "C559769"
 			(at 116.84 120.65 0)
 			(hide yes)
@@
 			)
 		)
-		(property "MPN" "GCM188R71H104KA57D"
+		(property "MPN" "GCM188R72A104KA64D"
 			(at 365.7600 63.5000 0)
 			(hide yes)
@@
 			)
 		)
-		(property "Notes" "Desacople VBUS del USBLC6-2SC6: 100 nF, X7R, 50 V, 0603; no alimenta el riel +5V. Agregado despues de placement-v1, autorizado en etapa 3. PROTO (2026-10-30): Yageo CC0603KRX7R9BB104 (LCSC C14663, JLC basic), misma especificación, sin AEC-Q200."
+		(property "Notes" "Desacople VBUS del USBLC6-2SC6: 100 nF, X7R, 50 V, 0603; no alimenta el riel +5V. Agregado despues de placement-v1, autorizado en etapa 3. PROTO (2026-10-30, consolidacion): un solo MPN para los 100 nF 0603: 100 V X7R (FH 0603B104K101NT, LCSC C88219), sin AEC-Q200. PROD: Murata GCM188R72A104KA64D (100 V, AEC-Q200). Mismo valor y tolerancia."
 			(at 365.7600 63.5000 0)
 			(hide yes)
@@
 			)
 		)
-		(property "LCSC" "C85864"
+		(property "LCSC" "C415406"
 			(at 365.7600 63.5000 0)
 			(hide yes)
@@
 			)
 		)
-		(property "MPN_PROTO" "CC0603KRX7R9BB104"
+		(property "MPN_PROTO" "0603B104K101NT"
 			(at 365.7600 63.5000 0)
 			(hide yes)
@@
 			)
 		)
-		(property "Manufacturer_PROTO" "Yageo"
+		(property "Manufacturer_PROTO" "FH"
 			(at 365.7600 63.5000 0)
 			(hide yes)
@@
 			)
 		)
-		(property "LCSC_PROTO" "C14663"
+		(property "LCSC_PROTO" "C88219"
 			(at 365.7600 63.5000 0)
 			(hide yes)

Commit message: [Claude Code] rc6: grupo A de la revisión externa y JLCDFM (pcb-v1-rc6)
Esquema (hoja 10), aprobado por el usuario:
- R-01: UVLO desde VBAT_F (R113 + R106 51k 1206, cara inferior junto a TP102),
  R107 9.53k (corte 6.44 V), U101.3 (SW) con no-connect. TI SNOSDF6 fig. 8-1.
- R-02: D104 = BAV23C (Diode:BAV70): A2-K es el D1 de VA a VS de TI.
  PROTO Diodes BAV23C-7-F (C150732); PROD Nexperia BAV23C,215.
- R-26: TP105 VS, TP106 VA, TP107 UVLO (cara inferior).
- Notes C-1..C-14, R-17, R-29; README, REVISION_CODEX, BOM_SOURCING.

PCB, sin mover componentes existentes:
- UVLO por B.Cu (y90 -> x111 -> y74.5) con 10 vías de costura GND_VEH.
- VA a D104.2 por x = 132.1.
- J-01 vías a 0.15 mm de los pads (excepción C403.2), J-02 tramos a
  >= 0.11 mm de las aberturas (excepciones de la misma red), J-03 64 textos
  fuera de vías, pads y orificios.
- DRC 0 errores / 3 avisos aceptados, 0 sin rutear, paridad 0; ERC 0 / 5;
  verify_etapa3/5 OK; 710 teardrops; fab/proto/ y BOM de LCSC regenerados.

Datasheets agregados en docs/datasheets/ (STD18NF25, BAS21, BAV23C, BAV23A_C_S,
BAV23C-7-F y los renombrados por el usuario). Scripts en scripts/rc6/.

Co-Authored-By: Claude Opus 5.5 <noreply@anthropic.com>
Parts:
- C401: Notes Desacople bulk del módulo en 3V3 (Espressif). 0805 por DC bias. Parte del presupuesto de 47 uF de +3V3_D (22 uF en C304 + 22 uF aquí + desacoples); no agregar más bulk sin revisar la estabilidad del TPS62A02-Q1. MPN a verificar (disponibilidad y especificación) antes de congelar el BOM. -> Desacople bulk del módulo en 3V3 (Espressif). 0805 por DC bias. Parte del presupuesto de 47 uF de +3V3_D (22 uF en C304 + 22 uF aquí + 10 uF de C605 en la hoja 60 + desacoples = ~54.6 uF nominal; con DC bias probablemente < 47 uF: verificar el escalón 0.1 -> 0.6 A en el bring-up); no agregar más bulk sin revisar la estabilidad del TPS62A02-Q1. MPN a verificar (disponibilidad y especificación) antes de congelar el BOM.
- TP403: Notes Punto de prueba de VBUS (no alimenta la placa salvo con D40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 -> Punto de prueba de VBUS (no alimenta la placa: D401 y JP401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
- U401: Notes 8 MB flash quad + 2 MB PSRAM quad, antena PCB, -40 a +85 C (las variantes R8/R16 con PSRAM octal llegan solo a 65 C). PSRAM quad: IO35-IO37 libres (WROOM-1 v1.8, tabla 3-1, nota b). LCSC C2913204. Pad 41 (EPAD) y pines 1/40 a GND_VEH. Antena al borde de la placa con keepout (ver nota de layout). IMPORTANTE: IO35-IO37 se usan como GPIO (DO1_EN, DO2_EN, DO1_DIAG); solo es valido con PSRAM quad (N8R2) o sin PSRAM. NO reemplazar por variantes con PSRAM octal (R8). Montaje: soldar a mano; comprar en LCSC (C2913204). -> 8 MB flash quad + 2 MB PSRAM quad, antena PCB, -40 a +85 C (las variantes R8/R16 con PSRAM octal llegan solo a 65 C). PSRAM quad: IO35-IO37 libres (WROOM-1 v1.8, tabla 3-1, nota b). LCSC C2913204. Pad 41 (EPAD) y pines 1/40 a GND_VEH. Antena al borde de la placa con keepout (ver nota de layout). IMPORTANTE: IO35-IO37 se usan como GPIO (DO1_EN, DO2_EN, DO1_DIAG); solo es valido con PSRAM quad (N8R2) o sin PSRAM. NO reemplazar por variantes con PSRAM octal (R8) ni con flash de 1.8 V (variantes «V»): IO47/IO48 (CAN_TX/CAN_RX) están en el dominio VDD_SPI y quedarían a 1.8 V frente al VIO de 3.3 V del ADM3055E. Montaje: soldar a mano; comprar en LCSC (C2913204).
Changed lines of the file:
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@@
 			)
 		)
-		(property "Notes" "Desacople bulk del módulo en 3V3 (Espressif). 0805 por DC bias. Parte del presupuesto de 47 uF de +3V3_D (22 uF en C304 + 22 uF aquí + desacoples); no agregar más bulk sin revisar la estabilidad del TPS62A02-Q1. MPN a verificar (disponibilidad y especificación) antes de congelar el BOM."
+		(property "Notes" "Desacople bulk del módulo en 3V3 (Espressif). 0805 por DC bias. Parte del presupuesto de 47 uF de +3V3_D (22 uF en C304 + 22 uF aquí + 10 uF de C605 en la hoja 60 + desacoples = ~54.6 uF nominal; con DC bias probablemente < 47 uF: verificar el escalón 0.1 -> 0.6 A en el bring-up); no agregar más bulk sin revisar la estabilidad del TPS62A02-Q1. MPN a verificar (disponibilidad y especificación) antes de congelar el BOM."
 			(at 190.5 95.25 0)
 			(hide yes)
@@
 			)
 		)
-		(property "Notes" "8 MB flash quad + 2 MB PSRAM quad, antena PCB, -40 a +85 C (las variantes R8/R16 con PSRAM octal llegan solo a 65 C). PSRAM quad: IO35-IO37 libres (WROOM-1 v1.8, tabla 3-1, nota b). LCSC C2913204. Pad 41 (EPAD) y pines 1/40 a GND_VEH. Antena al borde de la placa con keepout (ver nota de layout). IMPORTANTE: IO35-IO37 se usan como GPIO (DO1_EN, DO2_EN, DO1_DIAG); solo es valido con PSRAM quad (N8R2) o sin PSRAM. NO reemplazar por variantes con PSRAM octal (R8). Montaje: soldar a mano; comprar en LCSC (C2913204)."
+		(property "Notes" "8 MB flash quad + 2 MB PSRAM quad, antena PCB, -40 a +85 C (las variantes R8/R16 con PSRAM octal llegan solo a 65 C). PSRAM quad: IO35-IO37 libres (WROOM-1 v1.8, tabla 3-1, nota b). LCSC C2913204. Pad 41 (EPAD) y pines 1/40 a GND_VEH. Antena al borde de la placa con keepout (ver nota de layout). IMPORTANTE: IO35-IO37 se usan como GPIO (DO1_EN, DO2_EN, DO1_DIAG); solo es valido con PSRAM quad (N8R2) o sin PSRAM. NO reemplazar por variantes con PSRAM octal (R8) ni con flash de 1.8 V (variantes «V»): IO47/IO48 (CAN_TX/CAN_RX) están en el dominio VDD_SPI y quedarían a 1.8 V frente al VIO de 3.3 V del ADM3055E. Montaje: soldar a mano; comprar en LCSC (C2913204)."
 			(at 200.66 139.7 0)
 			(hide yes)
@@
 			)
 		)
-		(property "Notes" "Punto de prueba de VBUS (no alimenta la placa salvo con D401 + JP401)."
+		(property "Notes" "Punto de prueba de VBUS (no alimenta la placa: D401 y JP401 se eliminaron)."
 			(at 350.52 121.92 0)
 			(hide yes)
