File: sheets/50_sensors.kicad_sch (KiCad schematic)
At the start: 18 parts, among them U501 SCL3300-D01, U502 ASM330LHHTR, U503 AS5147U-HTSM

Commit message: [Claude Code] 20_buck_5v: opción B (no aislada) con LMR38010; masas unificadas
- sheets/20_isolation -> sheets/20_buck_5v: se quitan PS201, ISO7763 y
  TPS7A1650; U201 LMR38010SQDDARQ1 (PROTO: LMR38010SDDAR, LCSC C5219310),
  5.02 V / 1 A a 400 kHz según TI SNVSC73B (L201 XAL6060-333, 3 x 22 uF,
  RT 64.9k, FB 100k/24.9k). Huella oficial HSOIC-8 con vías térmicas.
- Símbolo LMR38010 (easyeda2kicad) en lib/easyeda2kicad/INCLI-VA_easyeda,
  con tipos de pin ajustados; registrado en sym-lib-table.
- Todas las hojas: GND_ISO -> GND_VEH, +5V_ISO -> +5V_VEH.
- Raíz: EN/DIAG/FLT directos entre las hojas 40, 70 y 10; la hoja 20 sin pines.
- 10_power_input: R111 a +3V3_D, C109 = 100 nF (inrush con C105),
  C105 DNP solo en PROTO; se quita un PWR_FLAG suelto en GND_VEH.
- 70_output_ch: cambios de layout del usuario (hechos en KiCad).
- Textos de las hojas 30/40/50/80 y la raíz sin referencias al aislamiento.
- ERC: 0 en 10, 20, 30, 40, 50, 60 y 70; quedan los de 80 (hoja vacía).

Co-Authored-By: Claude Opus 5.5 <noreply@anthropic.com>
Connections:
- net GND_ISO renamed GND_VEH
Other:
- note added: "BLOQUE 50 — SENSORES [riel +3V3_A] Bus SPI compartido (SPI_SCK, SPI_MOSI, SPI_MISO) con un CS por sensor y pull-up de 10 k a +3V3_A en cada CS. MISO en alta impedancia con CS alto en los tres sensores (SCL3300 "Tri State"; AS5147U tOZ = 10 ns; ASM330LHH SDO). MODOS SPI PARA EL FIRMWARE (un spi_device por sensor en ESP-IDF; el modo cambia según el CS): U501 SCL3300-D01 modo 0 (CPOL=0, CPHA=0) fSCK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"
- note added: "NOTAS DE LAYOUT • U501 (SCL3300) cerca de los puntos de fijación de la placa; lejos de U201/L201 (buck), L301, U302, del ADM3055E y de toda fuente de calor. Plano de masa bajo el encapsulado y sin pistas bajo él en la capa superior (Murata, Doc. 4921). Capacitores pegados a cada pin. • Ejes X/Y/Z de U501 y U502 alineados entre sí y con los bordes de la placa; marcar los ejes en la serigrafía. • V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"
- note removed: "BLOQUE 50 — SENSORES [dominio ISO, riel +3V3_A] Bus SPI compartido (SPI_SCK, SPI_MOSI, SPI_MISO) con un CS por sensor y pull-up de 10 k a +3V3_A en cada CS. MISO en alta impedancia con CS alto en los tres sensores (SCL3300 "Tri State"; AS5147U tOZ = 10 ns; ASM330LHH SDO). MODOS SPI PARA EL FIRMWARE (un spi_device por sensor en ESP-IDF; el modo cambia según el CS): U501 SCL3300-D01 modo 0 (CPOL=0,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"
- note removed: "NOTAS DE LAYOUT • U501 (SCL3300) cerca de los puntos de fijación de la placa; lejos de PS201, L301, U302, del ADM3055E y de toda fuente de calor. Plano de masa bajo el encapsulado y sin pistas bajo él en la capa superior (Murata, Doc. 4921). Capacitores pegados a cada pin. • Ejes X/Y/Z de U501 y U502 alineados entre sí y con los bordes de la placa; marcar los ejes en la serigrafía. • Variante ROT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"
Changed lines of the file:
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@@
 		(comment 2 "Inclinómetro de chasis CAN/BLE — INCLI-VA")
 	)
-	(text "NOTAS DE LAYOUT\n• U501 (SCL3300) cerca de los puntos de fijación de la placa; lejos de PS201, L301, U302, del ADM3055E y de toda fuente de calor.\n  Plano de masa bajo el encapsulado y sin pistas bajo él en la capa superior (Murata, Doc. 4921). Capacitores pegados a cada pin.\n• Ejes X/Y/Z de U501 y U502 alineados entre sí y con los bordes de la placa; marcar los ejes en la serigrafía.\n• Variante ROT: la placa va CENTRADA sobre el eje del pivote; U503 centrado sobre el eje del imán diametral (on-axis),\n  a la distancia del datasheet AS5147U. Sin material ferromagnético cerca del imán.\n• U502 (LGA): sin vías en los pads; dejar acceso para aire caliente."
+	(text "NOTAS DE LAYOUT\n• U501 (SCL3300) cerca de los puntos de fijación de la placa; lejos de U201/L201 (buck), L301, U302, del ADM3055E y de toda fuente de calor.\n  Plano de masa bajo el encapsulado y sin pistas bajo él en la capa superior (Murata, Doc. 4921). Capacitores pegados a cada pin.\n• Ejes X/Y/Z de U501 y U502 alineados entre sí y con los bordes de la placa; marcar los ejes en la serigrafía.\n• Variante ROT: la placa va CENTRADA sobre el eje del pivote; U503 centrado sobre el eje del imán diametral (on-axis),\n  a la distancia del datasheet AS5147U. Sin material ferromagnético cerca del imán.\n• U502 (LGA): sin vías en los pads; dejar acceso para aire caliente."
 		(exclude_from_sim no)
 		(at 20.32 253.492 0)
@@
 		)
 	)
-	(text "BLOQUE 50 — SENSORES  [dominio ISO, riel +3V3_A]\n\nBus SPI compartido (SPI_SCK, SPI_MOSI, SPI_MISO) con un CS por sensor y pull-up de 10 k a +3V3_A en cada CS.\nMISO en alta impedancia con CS alto en los tres sensores (SCL3300 \"Tri State\"; AS5147U tOZ = 10 ns; ASM330LHH SDO).\n\nMODOS SPI PARA EL FIRMWARE (un spi_device por sensor en ESP-IDF; el modo cambia según el CS):\n  U501 SCL3300-D01   modo 0 (CPOL=0, CPHA=0)   fSCK máx. 8 MHz, recomendado 2–4 MHz     CS_INC → IO10\n  U502 ASM330LHH     modo 3 (CPOL=1, CPHA=1)   fc(SPC) máx. 10 MHz                      CS_IMU → IO9   INT1 → IO40, INT2 → IO41\n  U503 AS5147U       modo 1 (CPOL=0, CPHA=1)   fSCK máx. 10 MHz                         CS_ROT → IO14  (solo variante ROT)"
+	(text "BLOQUE 50 — SENSORES  [riel +3V3_A]\n\nBus SPI compartido (SPI_SCK, SPI_MOSI, SPI_MISO) con un CS por sensor y pull-up de 10 k a +3V3_A en cada CS.\nMISO en alta impedancia con CS alto en los tres sensores (SCL3300 \"Tri State\"; AS5147U tOZ = 10 ns; ASM330LHH SDO).\n\nMODOS SPI PARA EL FIRMWARE (un spi_device por sensor en ESP-IDF; el modo cambia según el CS):\n  U501 SCL3300-D01   modo 0 (CPOL=0, CPHA=0)   fSCK máx. 8 MHz, recomendado 2–4 MHz     CS_INC → IO10\n  U502 ASM330LHH     modo 3 (CPOL=1, CPHA=1)   fc(SPC) máx. 10 MHz                      CS_IMU → IO9   INT1 → IO40, INT2 → IO41\n  U503 AS5147U       modo 1 (CPOL=0, CPHA=1)   fSCK máx. 10 MHz                         CS_ROT → IO14  (solo variante ROT)"
 		(exclude_from_sim no)
 		(at 20.32 20.32 0)
@@
 	)
 	(symbol
-		(lib_id "INCLI-VA:GND_ISO")
+		(lib_id "INCLI-VA:GND_VEH")
 		(at 109.22 198.12 0)
 		(unit 1)
@@
 			)
 		)
-		(property "Value" "GND_ISO"
+		(property "Value" "GND_VEH"
 			(at 109.22 201.93 0)
 			(show_name no)
@@
 	)
 	(symbol
-		(lib_id "INCLI-VA:GND_ISO")
+		(lib_id "INCLI-VA:GND_VEH")
 		(at 106.68 121.92 0)
 		(unit 1)
@@
 			)
 		)
-		(property "Value" "GND_ISO"
+		(property "Value" "GND_VEH"
 			(at 106.68 125.73 0)
 			(show_name no)
@@
 	)
 	(symbol
-		(lib_id "INCLI-VA:GND_ISO")
+		(lib_id "INCLI-VA:GND_VEH")
 		(at 76.2 87.63 270)
 		(unit 1)
@@
 			)
 		)
-		(property "Value" "GND_ISO"
+		(property "Value" "GND_VEH"
 			(at 72.39 87.63 90)
 			(show_name no)
@@
 	)
 	(symbol
-		(lib_id "INCLI-VA:GND_ISO")
+		(lib_id "INCLI-VA:GND_VEH")
 		(at 93.98 121.92 0)
 		(unit 1)
@@
 			)
 		)
-		(property "Value" "GND_ISO"
+		(property "Value" "GND_VEH"
 			(at 93.98 125.73 0)
 			(show_name no)
@@
 	)
 	(symbol
-		(lib_id "INCLI-VA:GND_ISO")
+		(lib_id "INCLI-VA:GND_VEH")
 		(at 119.38 121.92 0)
 		(unit 1)
@@
 			)
 		)
-		(property "Value" "GND_ISO"
+		(property "Value" "GND_VEH"
 			(at 119.38 125.73 0)
 			(show_name no)
@@
 	)
 	(symbol
-		(lib_id "INCLI-VA:GND_ISO")
+		(lib_id "INCLI-VA:GND_VEH")
 		(at 80.01 172.72 270)
 		(unit 1)
@@
 			)
 		)
-		(property "Value" "GND_ISO"
+		(property "Value" "GND_VEH"
 			(at 76.2 172.72 90)
 			(show_name no)
@@
 	)
 	(symbol
-		(lib_id "INCLI-VA:GND_ISO")
+		(lib_id "INCLI-VA:GND_VEH")
 		(at 64.77 162.56 270)
 		(unit 1)
@@
 			)
 		)
-		(property "Value" "GND_ISO"
+		(property "Value" "GND_VEH"
 			(at 60.96 162.56 90)
 			(show_name no)
@@
 	)
 	(symbol
-		(lib_id "INCLI-VA:GND_ISO")
+		(lib_id "INCLI-VA:GND_VEH")
 		(at 83.82 198.12 0)
 		(unit 1)
@@
 			)
 		)
-		(property "Value" "GND_ISO"
+		(property "Value" "GND_VEH"
 			(at 83.82 201.93 0)
 			(show_name no)
@@
 	)
 	(symbol
-		(lib_id "INCLI-VA:GND_ISO")
+		(lib_id "INCLI-VA:GND_VEH")
 		(at 254 83.82 90)
 		(unit 1)
@@
 			)
 		)
-		(property "Value" "GND_ISO"
+		(property "Value" "GND_VEH"
 			(at 257.81 83.82 90)
 			(show_name no)
@@
 	)
 	(symbol
-		(lib_id "INCLI-VA:GND_ISO")
+		(lib_id "INCLI-VA:GND_VEH")
 		(at 81.28 121.92 0)
 		(unit 1)
@@
 			)
 		)
-		(property "Value" "GND_ISO"
+		(property "Value" "GND_VEH"
 			(at 81.28 125.73 0)
 			(show_name no)
@@
 	)
 	(symbol
-		(lib_id "INCLI-VA:GND_ISO")
+		(lib_id "INCLI-VA:GND_VEH")
 		(at 96.52 198.12 0)
 		(unit 1)
@@
 			)
 		)
-		(property "Value" "GND_ISO"
+		(property "Value" "GND_VEH"
 			(at 96.52 201.93 0)
 			(show_name no)
@@
 	)
 	(symbol
-		(lib_id "INCLI-VA:GND_ISO")
+		(lib_id "INCLI-VA:GND_VEH")
 		(at 76.2 82.55 270)
 		(unit 1)
@@
 			)
 		)
-		(property "Value" "GND_ISO"
+		(property "Value" "GND_VEH"
 			(at 72.39 82.55 90)
 			(show_name no)
@@
 	)
 	(symbol
-		(lib_id "INCLI-VA:GND_ISO")
+		(lib_id "INCLI-VA:GND_VEH")
 		(at 121.92 82.55 90)
 		(unit 1)
@@
 			)
 		)
-		(property "Value" "GND_ISO"
+		(property "Value" "GND_VEH"
 			(at 125.73 82.55 90)
 			(show_name no)
@@
 	)
 	(symbol
-		(lib_id "INCLI-VA:GND_ISO")
+		(lib_id "INCLI-VA:GND_VEH")
 		(at 203.2 91.44 270)
 		(unit 1)
@@
 			)
 		)
-		(property "Value" "GND_ISO"
+		(property "Value" "GND_VEH"
 			(at 199.39 91.44 90)
 			(show_name no)
@@
 	)
 	(symbol
-		(lib_id "INCLI-VA:GND_ISO")
+		(lib_id "INCLI-VA:GND_VEH")
 		(at 236.22 121.92 0)
 		(unit 1)
@@
 			)
 		)
-		(property "Value" "GND_ISO"
+		(property "Value" "GND_VEH"
 			(at 236.22 125.73 0)
 			(show_name no)
