File: sheets/50_sensors.kicad_sch (KiCad schematic)
At the start: 18 parts, among them U501 SCL3300-D01, U502 ASM330LHHTR, U503 AS5147U-HTSM

Commit message: [Codex] Integra cierre de Claude y valida sincronizacion previa al layout
Parts:
- C507, R503, U503: now fitted
Changed lines of the file:
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@@
 			)
 		)
-		(property "Datasheet" ""
+		(property "Datasheet" "N/A (pad de prueba)"
 			(at 154.94 162.56 0)
 			(hide yes)
@@
 		(on_board yes)
 		(in_pos_files yes)
-		(dnp yes)
+		(dnp no)
 		(property "Reference" "R503"
 			(at 187.96 86.36 0)
@@
 			)
 		)
-		(property "Datasheet" ""
+		(property "Datasheet" "N/A (pad de prueba)"
 			(at 154.94 132.08 0)
 			(hide yes)
@@
 		(on_board yes)
 		(in_pos_files yes)
-		(dnp yes)
+		(dnp no)
 		(property "Reference" "C507"
 			(at 238.76 114.3 0)
@@
 			)
 		)
-		(property "Datasheet" ""
+		(property "Datasheet" "N/A (pad de prueba)"
 			(at 154.94 152.4 0)
 			(hide yes)
@@
 		(on_board yes)
 		(in_pos_files yes)
-		(dnp yes)
+		(dnp no)
 		(property "Reference" "U503"
 			(at 229.87 76.2 0)
@@
 			)
 		)
-		(property "Datasheet" ""
+		(property "Datasheet" "N/A (pad de prueba)"
 			(at 154.94 142.24 0)
 			(hide yes)
