File: sheets/50_sensors.kicad_sch (KiCad schematic)
At the start: 18 parts, among them U501 SCL3300-D01, U502 ASM330LHHTR, U503 AS5147U-HTSM

Commit message: [Claude Code] esquema+PCB: campos LCSC y sustitutos PROTO del BOM (pcb-v1-rc2)
- Esquema (solo campos, ocultos): LCSC en todos los componentes; MPN_PROTO,
  LCSC_PROTO y Manufacturer_PROTO con los sustitutos aceptados; Notes con
  compra y montaje (Q101, Q102, F101, L201, U503 a mano desde DigiKey/Mouser).
  MPN (PROD), valores, huellas y conexiones sin cambios. LCSC Part -> LCSC.
- PCB: mismos campos en las 145 huellas, insertados como texto (equivalente
  a F8 solo para campos); nada cambia fuera de las huellas.
- ERC por hoja igual que antes (0 errores, 5 avisos). DRC 0 errores / 3 avisos
  aceptados, 0 sin rutear, paridad 0 (antes de sincronizar: 145).
- etapa6_fab.py usa los campos _PROTO y genera bom_jlc_lcsc.csv; este y
  cpl_jlc.csv salen idénticos (60 líneas, 123 piezas). Gerbers sin cambios
  de contenido.

Co-Authored-By: Claude Opus 5.5 <noreply@anthropic.com>
Parts:
- C501: LCSC (none) -> C85864; LCSC_PROTO (none) -> C14663; MPN_PROTO (none) -> CC0603KRX7R9BB104; Manufacturer_PROTO (none) -> Yageo; Notes VDD de U501. Circuito de aplicación de Murata (Doc. 4921, fig. 16 y tabla 48): 70-130 nF, ESR <= 100 mohm, junto al pin. Murata usa 0402; aquí 0603 (prototipo). -> VDD de U501. Circuito de aplicación de Murata (Doc. 4921, fig. 16 y tabla 48): 70-130 nF, ESR <= 100 mohm, junto al pin. Murata usa 0402; aquí 0603 (prototipo). PROTO (2026-10-30): Yageo CC0603KRX7R9BB104 (LCSC C14663, JLC basic), misma especificación, sin AEC-Q200.
- C502: LCSC (none) -> C85864; LCSC_PROTO (none) -> C14663; MPN_PROTO (none) -> CC0603KRX7R9BB104; Manufacturer_PROTO (none) -> Yageo; Notes A_EXTC de U501. Circuito de aplicación de Murata (Doc. 4921, fig. 16 y tabla 48): 70-130 nF, ESR <= 100 mohm, junto al pin. Murata usa 0402; aquí 0603 (prototipo). -> A_EXTC de U501. Circuito de aplicación de Murata (Doc. 4921, fig. 16 y tabla 48): 70-130 nF, ESR <= 100 mohm, junto al pin. Murata usa 0402; aquí 0603 (prototipo). PROTO (2026-10-30): Yageo CC0603KRX7R9BB104 (LCSC C14663, JLC basic), misma especificación, sin AEC-Q200.
- C503: LCSC (none) -> C85864; LCSC_PROTO (none) -> C14663; MPN_PROTO (none) -> CC0603KRX7R9BB104; Manufacturer_PROTO (none) -> Yageo; Notes D_EXTC de U501. Circuito de aplicación de Murata (Doc. 4921, fig. 16 y tabla 48): 70-130 nF, ESR <= 100 mohm, junto al pin. Murata usa 0402; aquí 0603 (prototipo). -> D_EXTC de U501. Circuito de aplicación de Murata (Doc. 4921, fig. 16 y tabla 48): 70-130 nF, ESR <= 100 mohm, junto al pin. Murata usa 0402; aquí 0603 (prototipo). PROTO (2026-10-30): Yageo CC0603KRX7R9BB104 (LCSC C14663, JLC basic), misma especificación, sin AEC-Q200.
- C504: LCSC (none) -> C85864; LCSC_PROTO (none) -> C14663; MPN_PROTO (none) -> CC0603KRX7R9BB104; Manufacturer_PROTO (none) -> Yageo; Notes DVIO de U501. Circuito de aplicación de Murata (Doc. 4921, fig. 16 y tabla 48): 70-130 nF, ESR <= 100 mohm, junto al pin. Murata usa 0402; aquí 0603 (prototipo). -> DVIO de U501. Circuito de aplicación de Murata (Doc. 4921, fig. 16 y tabla 48): 70-130 nF, ESR <= 100 mohm, junto al pin. Murata usa 0402; aquí 0603 (prototipo). PROTO (2026-10-30): Yageo CC0603KRX7R9BB104 (LCSC C14663, JLC basic), misma especificación, sin AEC-Q200.
- C505: LCSC (none) -> C85864; LCSC_PROTO (none) -> C14663; MPN_PROTO (none) -> CC0603KRX7R9BB104; Manufacturer_PROTO (none) -> Yageo; Notes VDD de U502 (ST fig. 14: C1 = 100 nF junto al pin 8). -> VDD de U502 (ST fig. 14: C1 = 100 nF junto al pin 8). PROTO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
- C506: LCSC (none) -> C85864; LCSC_PROTO (none) -> C14663; MPN_PROTO (none) -> CC0603KRX7R9BB104; Manufacturer_PROTO (none) -> Yageo; Notes VDDIO de U502 (ST fig. 14: C3 = 100 nF junto al pin 5). -> VDDIO de U502 (ST fig. 14: C3 = 100 nF junto al pin 5). PRO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
- C507: LCSC (none) -> C85864; LCSC_PROTO (none) -> C14663; MPN_PROTO (none) -> CC0603KRX7R9BB104; Manufacturer_PROTO (none) -> Yageo; Notes VDD/VDD3V3 de U503 (fig. 13, modo 3.3 V: 100 nF). Solo variante ROT: DNP en la variante estándar. -> VDD/VDD3V3 de U503 (fig. 13, modo 3.3 V: 100 nF). Solo variante ROT: DNP en la variante estándar. PROTO (2026-10-30): Yageo CC0603KRX7R9BB104 (LCSC C14663, JLC basic), misma especificación, sin AEC-Q200.
- C508: LCSC (none) -> C126586
- R501: LCSC (none) -> C116677; LCSC_PROTO (none) -> C25804; MPN_PROTO (none) -> 0603WAF1002T5E; Manufacturer_PROTO (none) -> UNI-ROYAL; Notes Pull-up de CS_INC a +3V3_A: mantiene el sensor deseleccionado mientras arranca el ESP32 (GPIO en alta impedancia). -> Pull-up de CS_INC a +3V3_A: mantiene el sensor deseleccionado mientras arranca el ESP32 (GPIO en alta impedancia). PROTO (2026-10-30): UNI-ROYAL 0603WAF1002T5E (LCSC C25804, JLC basic), misma especificación, sin AEC-Q200.
- R502: LCSC (none) -> C116677; LCSC_PROTO (none) -> C25804; MPN_PROTO (none) -> 0603WAF1002T5E; Manufacturer_PROTO (none) -> UNI-ROYAL; Notes Pull-up de CS_IMU a +3V3_A: mantiene el sensor deseleccionado mientras arranca el ESP32 (GPIO en alta impedancia). -> Pull-up de CS_IMU a +3V3_A: mantiene el sensor deseleccionado mientras arranca el ESP32 (GPIO en alta impedancia). PROTO (2026-10-30): UNI-ROYAL 0603WAF1002T5E (LCSC C25804, JLC basic), misma especificación, sin AEC-Q200.
- R503: LCSC (none) -> C116677; LCSC_PROTO (none) -> C25804; MPN_PROTO (none) -> 0603WAF1002T5E; Manufacturer_PROTO (none) -> UNI-ROYAL; Notes Pull-up de CS_ROT a +3V3_A: mantiene el sensor deseleccionado mientras arranca el ESP32 (GPIO en alta impedancia). Solo variante ROT: DNP en la variante estándar. -> Pull-up de CS_ROT a +3V3_A: mantiene el sensor deseleccionado mientras arranca el ESP32 (GPIO en alta impedancia). Solo variante ROT: DNP en la variante estándar. PROTO (2026-10-30): UNI-ROYAL 0603WAF1002T5E (LCSC C25804, JLC basic), misma especificación, sin AEC-Q200.
- U501: LCSC (none) -> C22416657; LCSC_PROTO (none) -> C3825395; MPN_PROTO (none) -> SCL3300-D01-10; Notes Inclinómetro principal, 3 ejes. SPI modo 0 (CPOL=0, CPHA=0), fSCK 0.1-8 MHz, recomendado 2-4 MHz (Doc. 4921 Rev. 4). Huella easyeda2kicad (LCSC C22416657): pads 0.65 x 1.30 mm, 0.32 mm más largos hacia afuera que el land pattern de Murata (0.61 x 0.98, fig. 11): mejor para soldar a mano; en producción volver al de Murata. Compra: sin stock en LCSC, comprar en DigiKey o Mouser. -> Inclinómetro principal, 3 ejes. SPI modo 0 (CPOL=0, CPHA=0), fSCK 0.1-8 MHz, recomendado 2-4 MHz (Doc. 4921 Rev. 4). Huella easyeda2kicad (LCSC C22416657): pads 0.65 x 1.30 mm, 0.32 mm más largos hacia afuera que el land pattern de Murata (0.61 x 0.98, fig. 11): mejor para soldar a mano; en producción volver al de Murata. PROTO (2026-10-30): Murata SCL3300-D01-10 (LCSC C3825395), mismo sensor en carrete de 1000 u (Murata Doc. 4921 Rev. 2, sec. 9); lo monta JLC.
- U502: LCSC (none) -> C459826
- U503: LCSC (none) -> C38675951; Notes Sensor de ángulo magnético 14 bit, AEC-Q100 (ángulo de pluma con imán diametral externo). Solo variante ROT: DNP en la variante estándar. SPI modo 1 (CPOL=0, CPHA=1), hasta 10 MHz (DS000639 v1-04). Modo 3.3 V: VDD y VDD3V3 unidos (fig. 13). Salidas ABI/UVW/PWM sin uso. Compra: sin stock en LCSC, comprar en DigiKey o Mouser. -> Sensor de ángulo magnético 14 bit, AEC-Q100 (ángulo de pluma con imán diametral externo). Solo variante ROT: DNP en la variante estándar. SPI modo 1 (CPOL=0, CPHA=1), hasta 10 MHz (DS000639 v1-04). Modo 3.3 V: VDD y VDD3V3 unidos (fig. 13). Salidas ABI/UVW/PWM sin uso. Compra: sin stock en LCSC, comprar en DigiKey o Mouser. Compra (2026-10-30): sin stock en JLC/LCSC; comprar en DigiKey/Mouser y soldar a mano.

Commit message: [Claude Code] TP de la cara inferior rotulados, TP406/TP505 GND con agujero, R803/R804 2.2k
- B.Silk: nombre de señal junto a cada TP (verificado con la red), GND con recuadro,
  nota «CAN: medir vs GND_CAN (J1-5)».
- TP406 (40_mcu) y TP505 (50_sensors): GND_VEH THT D2.5/1.2 mm, en esquema y PCB,
  fuera de BOM/CPL.
- LEDs: R803/R804 470 → 2.2k (0603WAF2201T5E C4190 basic; PROD AC0603FR-072K2L);
  ~0.61 / 0.70 mA; brillo por PWM (PENDIENTES, firmware).
- DRC 0 errores / 3 avisos aceptados, paridad 0, ERC 0 / 5; fab/proto y BOM regenerados.

Co-Authored-By: Claude Opus 5.5 <noreply@anthropic.com>
Parts:
- added TP505: GND_VEH, TestPoint:TestPoint_THTPad_D2.5mm_Drill1.2mm, symbol Connector:TestPoint
Connections:
- net GND_VEH: now also TP505.1
Changed lines of the file:
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@@
+		)
+	)
+	(symbol
+		(lib_id "Connector:TestPoint")
+		(at 154.94 175.26 0)
+		(unit 1)
+		(body_style 1)
+		(exclude_from_sim no)
+		(in_bom no)
+		(on_board yes)
+		(in_pos_files no)
+		(dnp no)
+		(property "Reference" "TP505"
+			(at 156.21 170.18 0)
+			(show_name no)
+			(do_not_autoplace no)
+			(effects
+				(font
+					(size 1.27 1.27)
+				)
+				(justify left)
+			)
+		)
+		(property "Value" "GND_VEH"
+			(at 156.21 172.09 0)
+			(show_name no)
+			(do_not_autoplace no)
+			(effects
+				(font
+					(size 1.27 1.27)
+				)
+				(justify left)
+			)
+		)
+		(property "Footprint" "TestPoint:TestPoint_THTPad_D2.5mm_Drill1.2mm"
+			(at 154.94 175.26 0)
+			(hide yes)
+			(show_name no)
+			(do_not_autoplace no)
+			(effects
+				(font
+					(size 1.27 1.27)
+				)
+			)
+		)
+		(property "Datasheet" "N/A (pad de prueba)"
+			(at 154.94 175.26 0)
+			(hide yes)
+			(show_name no)
+			(do_not_autoplace no)
+			(effects
+				(font
+					(size 1.27 1.27)
+				)
+			)
+		)
+		(property "Description" ""
+			(at 154.94 175.26 0)
+			(hide yes)
+			(show_name no)
+			(do_not_autoplace no)
+			(effects
+				(font
+					(size 1.27 1.27)
+				)
+			)
+		)
+		(property "MPN" "-"
+			(at 154.94 175.26 0)
+			(hide yes)
+			(show_name no)
+			(do_not_autoplace no)
+			(effects
+				(font
+					(size 1.27 1.27)
+				)
+			)
+		)
+		(property "Manufacturer" "-"
+			(at 154.94 175.26 0)
+			(hide yes)
+			(show_name no)
+			(do_not_autoplace no)
+			(effects
+				(font
+					(size 1.27 1.27)
+				)
+			)
+		)
+		(property "Notes" "Punto de prueba de GND_VEH con agujero (pad 2.5 mm, taladro 1.2 mm) para el caiman o la punta de masa del osciloscopio; admite un lazo de alambre o un Keystone 5001 soldado a mano. Fuera del BOM y del CPL de JLC."
+			(at 154.94 175.26 0)
+			(hide yes)
+			(show_name no)
+			(do_not_autoplace no)
+			(effects
+				(font
+					(size 1.27 1.27)
+				)
+			)
+		)
+		(property "DNP" ""
+			(at 154.94 175.26 0)
+			(hide yes)
+			(show_name no)
+			(do_not_autoplace no)
+			(effects
+				(font
+					(size 1.27 1.27)
+				)
+			)
+		)
+		(pin "1"
+		)
+		(instances
+			(project "INCLI-VA"
+				(path "/7fd92c2b-4254-4d73-93ba-bfde861bede3/3985e6d4-83de-4a87-a0f1-257500c83de4"
+					(reference "TP505")
+					(unit 1)
+				)
+			)
+		)
+	)
+	(symbol
+		(lib_id "INCLI-VA:GND_VEH")
+		(at 154.94 175.26 0)
+		(unit 1)
+		(body_style 1)
+		(exclude_from_sim no)
+		(in_bom no)
+		(on_board yes)
+		(in_pos_files no)
+		(dnp no)
+		(property "Reference" "#PWR590"
+			(at 154.94 181.61 0)
+			(hide yes)
+			(show_name no)
+			(do_not_autoplace no)
+			(effects
+				(font
+					(size 1.27 1.27)
+				)
+			)
+		)
+		(property "Value" "GND_VEH"
+			(at 154.94 179.07 0)
+			(show_name no)
+			(do_not_autoplace no)
+			(effects
+				(font
+					(size 1.27 1.27)
+				)
+			)
+		)
+		(property "Footprint" ""
+			(at 154.94 175.26 0)
+			(hide yes)
+			(show_name no)
+			(do_not_autoplace no)
+			(effects
+				(font
+					(size 1.27 1.27)
+				)
+			)
+		)
+		(property "Datasheet" ""
+			(at 154.94 175.26 0)
+			(hide yes)
+			(show_name no)
+			(do_not_autoplace no)
+			(effects
+				(font
+					(size 1.27 1.27)
+				)
+			)
+		)
+		(property "Description" ""
+			(at 154.94 175.26 0)
+			(hide yes)
+			(show_name no)
+			(do_not_autoplace no)
+			(effects
+				(font
+					(size 1.27 1.27)
+				)
+			)
+		)
+		(pin "1"
+		)
+		(instances
+			(project "INCLI-VA"
+				(path "/7fd92c2b-4254-4d73-93ba-bfde861bede3/3985e6d4-83de-4a87-a0f1-257500c83de4"
+					(reference "#PWR590")
+					(unit 1)
+				)
+			)
 		)
 	)
