File: sheets/50_sensors.kicad_sch (KiCad schematic)
At the start: 19 parts, among them U501 SCL3300-D01, U502 ASM330LHHTR, U503 AS5147U-HTSM

Commit message: [Claude Code] bom: compra principal en LCSC + DigiKey/Mouser; consolidación de pasivos
- Plan: JLC solo PCB + stencil Top; componentes de LCSC soldados a mano.
- Consolidación (solo valor/campos): R702/R752 4k7 → 2.2k; 23 × 100 nF a un
  MPN de 100 V X7R; PROTO 1 µF 50 V y 10 µF 25 V X7R. BOM PROTO 70 → 68 líneas.
- LCSC_BOM_COMPLETO_PROTO.csv: 6 juegos, 62 líneas, USD 552.43 (3 juegos: 286.65).
- DIGIKEY_MOUSER.csv: L201, U503, Q101, Q102, F101 (0 en LCSC), ≈ USD 99.54.
- Resumen de costos en BOM_SOURCING.md; archivos de JLC al día como alternativa.
- DRC 0 errores / 3 avisos aceptados, paridad 0, ERC 0 / 5.

Co-Authored-By: Claude Opus 5.5 <noreply@anthropic.com>
Parts:
- C501: LCSC C85864 -> C415406; LCSC_PROTO C14663 -> C88219; MPN GCM188R71H104KA57D -> GCM188R72A104KA64D; MPN_PROTO CC0603KRX7R9BB104 -> 0603B104K101NT; Manufacturer_PROTO Yageo -> FH; Notes VDD de U501. Circuito de aplicación de Murata (Doc. 4921, fig. 16 y tabla 48): 70-130 nF, ESR <= 100 mohm, junto al pin. Murata usa 0402; aquí 0603 (prototipo). PROTO (2026-10-30): Yageo CC0603KRX7R9BB104 (LCSC C14663, JLC basic), misma especificación, sin AEC-Q200. -> VDD de U501. Circuito de aplicación de Murata (Doc. 4921, fig. 16 y tabla 48): 70-130 nF, ESR <= 100 mohm, junto al pin. Murata usa 0402; aquí 0603 (prototipo). PROTO (2026-10-30, consolidacion): un solo MPN para los 100 nF 0603: 100 V X7R (FH 0603B104K101NT, LCSC C88219), sin AEC-Q200. PROD: Murata GCM188R72A104KA64D (100 V, AEC-Q200). Mismo valor y tolerancia.
- C502: LCSC C85864 -> C415406; LCSC_PROTO C14663 -> C88219; MPN GCM188R71H104KA57D -> GCM188R72A104KA64D; MPN_PROTO CC0603KRX7R9BB104 -> 0603B104K101NT; Manufacturer_PROTO Yageo -> FH; Notes A_EXTC de U501. Circuito de aplicación de Murata (Doc. 4921, fig. 16 y tabla 48): 70-130 nF, ESR <= 100 mohm, junto al pin. Murata usa 0402; aquí 0603 (prototipo). PROTO (2026-10-30): Yageo CC0603KRX7R9BB104 (LCSC C14663, JLC basic), misma especificación, sin AEC-Q200. -> A_EXTC de U501. Circuito de aplicación de Murata (Doc. 4921, fig. 16 y tabla 48): 70-130 nF, ESR <= 100 mohm, junto al pin. Murata usa 0402; aquí 0603 (prototipo). PROTO (2026-10-30, consolidacion): un solo MPN para los 100 nF 0603: 100 V X7R (FH 0603B104K101NT, LCSC C88219), sin AEC-Q200. PROD: Murata GCM188R72A104KA64D (100 V, AEC-Q200). Mismo valor y tolerancia.
- C503: LCSC C85864 -> C415406; LCSC_PROTO C14663 -> C88219; MPN GCM188R71H104KA57D -> GCM188R72A104KA64D; MPN_PROTO CC0603KRX7R9BB104 -> 0603B104K101NT; Manufacturer_PROTO Yageo -> FH; Notes D_EXTC de U501. Circuito de aplicación de Murata (Doc. 4921, fig. 16 y tabla 48): 70-130 nF, ESR <= 100 mohm, junto al pin. Murata usa 0402; aquí 0603 (prototipo). PROTO (2026-10-30): Yageo CC0603KRX7R9BB104 (LCSC C14663, JLC basic), misma especificación, sin AEC-Q200. -> D_EXTC de U501. Circuito de aplicación de Murata (Doc. 4921, fig. 16 y tabla 48): 70-130 nF, ESR <= 100 mohm, junto al pin. Murata usa 0402; aquí 0603 (prototipo). PROTO (2026-10-30, consolidacion): un solo MPN para los 100 nF 0603: 100 V X7R (FH 0603B104K101NT, LCSC C88219), sin AEC-Q200. PROD: Murata GCM188R72A104KA64D (100 V, AEC-Q200). Mismo valor y tolerancia.
- C504: LCSC C85864 -> C415406; LCSC_PROTO C14663 -> C88219; MPN GCM188R71H104KA57D -> GCM188R72A104KA64D; MPN_PROTO CC0603KRX7R9BB104 -> 0603B104K101NT; Manufacturer_PROTO Yageo -> FH; Notes DVIO de U501. Circuito de aplicación de Murata (Doc. 4921, fig. 16 y tabla 48): 70-130 nF, ESR <= 100 mohm, junto al pin. Murata usa 0402; aquí 0603 (prototipo). PROTO (2026-10-30): Yageo CC0603KRX7R9BB104 (LCSC C14663, JLC basic), misma especificación, sin AEC-Q200. -> DVIO de U501. Circuito de aplicación de Murata (Doc. 4921, fig. 16 y tabla 48): 70-130 nF, ESR <= 100 mohm, junto al pin. Murata usa 0402; aquí 0603 (prototipo). PROTO (2026-10-30, consolidacion): un solo MPN para los 100 nF 0603: 100 V X7R (FH 0603B104K101NT, LCSC C88219), sin AEC-Q200. PROD: Murata GCM188R72A104KA64D (100 V, AEC-Q200). Mismo valor y tolerancia.
- C505: LCSC C85864 -> C415406; LCSC_PROTO C14663 -> C88219; MPN GCM188R71H104KA57D -> GCM188R72A104KA64D; MPN_PROTO CC0603KRX7R9BB104 -> 0603B104K101NT; Manufacturer_PROTO Yageo -> FH; Notes VDD de U502 (ST fig. 14: C1 = 100 nF junto al pin 8). PROTO (2026-10-30): Yageo CC0603KRX7R9BB104 (LCSC C14663, JLC basic), misma especificación, sin AEC-Q200. -> VDD de U502 (ST fig. 14: C1 = 100 nF junto al pin 8). PROTO (2026-10-30, consolidacion): un solo MPN para los 100 nF 0603: 100 V X7R (FH 0603B104K101NT, LCSC C88219), sin AEC-Q200. PROD: Murata GCM188R72A104KA64D (100 V, AEC-Q200). Mismo valor y tolerancia.
- C506: LCSC C85864 -> C415406; LCSC_PROTO C14663 -> C88219; MPN GCM188R71H104KA57D -> GCM188R72A104KA64D; MPN_PROTO CC0603KRX7R9BB104 -> 0603B104K101NT; Manufacturer_PROTO Yageo -> FH; Notes VDDIO de U502 (ST fig. 14: C3 = 100 nF junto al pin 5). PROTO (2026-10-30): Yageo CC0603KRX7R9BB104 (LCSC C14663, JLC basic), misma especificación, sin AEC-Q200. -> VDDIO de U502 (ST fig. 14: C3 = 100 nF junto al pin 5). PROTO (2026-10-30, consolidacion): un solo MPN para los 100 nF 0603: 100 V X7R (FH 0603B104K101NT, LCSC C88219), sin AEC-Q200. PROD: Murata GCM188R72A104KA64D (100 V, AEC-Q200). Mismo valor y tolerancia.
- C507: LCSC C85864 -> C415406; LCSC_PROTO C14663 -> C88219; MPN GCM188R71H104KA57D -> GCM188R72A104KA64D; MPN_PROTO CC0603KRX7R9BB104 -> 0603B104K101NT; Manufacturer_PROTO Yageo -> FH; Notes VDD/VDD3V3 de U503 (fig. 13, modo 3.3 V: 100 nF). Solo variante ROT: DNP en la variante estándar. PROTO (2026-10-30): Yageo CC0603KRX7R9BB104 (LCSC C14663, JLC basic), misma especificación, sin AEC-Q200. -> VDD/VDD3V3 de U503 (fig. 13, modo 3.3 V: 100 nF). Solo variante ROT: DNP en la variante estándar. PROTO (2026-10-30, consolidacion): un solo MPN para los 100 nF 0603: 100 V X7R (FH 0603B104K101NT, LCSC C88219), sin AEC-Q200. PROD: Murata GCM188R72A104KA64D (100 V, AEC-Q200). Mismo valor y tolerancia.
- C508: LCSC_PROTO (none) -> C3039694; MPN_PROTO (none) -> CL21B106KAYQNNE; Manufacturer_PROTO (none) -> Samsung; Notes VDD de U502 (ST fig. 14: C2 = 10 uF; ST sugiere aluminio, aquí cerámico X7R). 0805 por DC bias. MPN a verificar (disponibilidad y especificación) antes de congelar el BOM. -> VDD de U502 (ST fig. 14: C2 = 10 uF; ST sugiere aluminio, aquí cerámico X7R). 0805 por DC bias. MPN a verificar (disponibilidad y especificación) antes de congelar el BOM. PROTO (2026-10-30, consolidacion): Samsung CL21B106KAYQNNE (25 V X7R, LCSC C3039694), sin AEC-Q200: el original no tiene stock en lcsc.com.
