File: sheets/20_buck_5v.kicad_sch (KiCad schematic)
At the start: 12 parts, among them U201 LMR38010SQDDARQ1

Commit message: [Codex] Integra cierre de Claude y valida sincronizacion previa al layout
Changed lines of the file:
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@@
 			(do_not_autoplace no)
 			(effects
+				(hide yes)
 				(font
 					(size 1.27 1.27)
@@
 			)
 		)
-		(property "Datasheet" ""
+		(property "Datasheet" "N/A (pad de prueba)"
 			(at 294.64 104.14 0)
 			(hide yes)

Commit message: update pcb layout
Other:
- moved on the sheet: C201, C202, C203, C204, C205, C206, L201, R201, R202, R203, TP201, U201
