File: sheets/20_buck_5v.kicad_sch (KiCad schematic)
At the start: 12 parts, among them U201 LMR38010SQDDARQ1

Commit message: [Claude Code] esquema+PCB: campos LCSC y sustitutos PROTO del BOM (pcb-v1-rc2)
- Esquema (solo campos, ocultos): LCSC en todos los componentes; MPN_PROTO,
  LCSC_PROTO y Manufacturer_PROTO con los sustitutos aceptados; Notes con
  compra y montaje (Q101, Q102, F101, L201, U503 a mano desde DigiKey/Mouser).
  MPN (PROD), valores, huellas y conexiones sin cambios. LCSC Part -> LCSC.
- PCB: mismos campos en las 145 huellas, insertados como texto (equivalente
  a F8 solo para campos); nada cambia fuera de las huellas.
- ERC por hoja igual que antes (0 errores, 5 avisos). DRC 0 errores / 3 avisos
  aceptados, 0 sin rutear, paridad 0 (antes de sincronizar: 145).
- etapa6_fab.py usa los campos _PROTO y genera bom_jlc_lcsc.csv; este y
  cpl_jlc.csv salen idénticos (60 líneas, 123 piezas). Gerbers sin cambios
  de contenido.

Co-Authored-By: Claude Opus 5.5 <noreply@anthropic.com>
Parts:
- C201: LCSC (none) -> C2168848; LCSC_PROTO (none) -> C17288249; MPN_PROTO (none) -> CL32B475KCVZNWE; Manufacturer_PROTO (none) -> Samsung; Notes C_IN del LMR38010 (TI: >= 4.7 uF ceramico, X7R, idealmente 2 x VIN max). 100 V X7S AEC-Q200. 1210 por tension y DC bias. Pegado a VIN/GND de U201. MPN a verificar. -> C_IN del LMR38010 (TI: >= 4.7 uF ceramico, X7R, idealmente 2 x VIN max). 100 V X7S AEC-Q200. 1210 por tension y DC bias. Pegado a VIN/GND de U201. MPN a verificar. PROTO (2026-10-30): Samsung CL32B475KCVZNWE (LCSC C17288249), sin AEC-Q200, solo para el prototipo. PROD: este MPN (AEC-Q200); sin stock en JLC/LCSC, comprar en DigiKey/Mouser.
- C202: LCSC (none) -> C415406
- C203: LCSC (none) -> C85864; LCSC_PROTO (none) -> C14663; MPN_PROTO (none) -> CC0603KRX7R9BB104; Manufacturer_PROTO (none) -> Yageo; Notes C_BOOT entre BOOT (7) y SW (8): 100 nF >= 16 V (TI 9.2.2.7). -> C_BOOT entre BOOT (7) y SW (8): 100 nF >= 16 V (TI 9.2.2.7)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
- C204, C205, C206: LCSC (none) -> C126598
- L201: LCSC (none) -> C5119929; Notes 33 uH (TI tabla 9-1, 400 kHz, 5 V). Isat 3.7 A > limite high-side max del LMR38010 (1.9 A); DCR 105 mohm max. AEC-Q200. -> 33 uH (TI tabla 9-1, 400 kHz, 5 V). Isat 3.7 A > limite high-side max del LMR38010 (1.9 A); DCR 105 mohm max. AEC-Q200. Compra (2026-10-30): sin stock en JLC/LCSC; comprar en DigiKey/Mouser y soldar a mano.
- R201: LCSC (none) -> C116674; LCSC_PROTO (none) -> C25803; MPN_PROTO (none) -> 0603WAF1003T5E; Manufacturer_PROTO (none) -> UNI-ROYAL; Notes R_FBT (TI recomienda 100k). VOUT = 1 V x (1 + 100k/24.9k) = 5.02 V. -> R_FBT (TI recomienda 100k). VOUT = 1 V x (1 + 100k/24.9k) = 5.02 V. PROTO (2026-10-30): UNI-ROYAL 0603WAF1003T5E (LCSC C25803, JLC basic), misma especificación, sin AEC-Q200.
- R202: LCSC (none) -> C227732
- R203: LCSC (none) -> C228007
- U201: LCSC (none) -> C18198885; Notes Buck 80 V / 1 A, PFM + spread spectrum. PROD: LMR38010SQDDARQ1 (AEC-Q100, SNVSC72B). PROTO: LMR38010SDDAR (LCSC C5219310), equivalente comercial: mismo modo, pinout y DDA0008B (ver PENDIENTES 'Equivalencia LMR38010'). EP con 6 vias de 0.2 mm a GND_VEH (soldable con aire caliente). Pin a pin con LMR38020 (2 A). Simbolo de easyeda2kicad con tipos de pin ajustados. -> Buck 80 V / 1 A, PFM + spread spectrum. PROD: LMR38010SQDDARQ1 (AEC-Q100, SNVSC72B). PROTO: LMR38010SDDAR (LCSC C5219310), equivalente comercial: mismo modo, pinout y DDA0008B (ver PENDIENTES 'Equivalencia LMR38010'). EP con 6 vias de 0.2 mm a GND_VEH (soldable con aire caliente). Pin a pin con LMR38020 (2 A). Simbolo de easyeda2kicad con tipos de pin ajustados. PROD (2026-10-30): sin stock suficiente en JLC/LCSC para 100 placas; comprar en DigiKey/Mouser.
Changed lines of the file:
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@@
+			)
+		)
+		(property "LCSC" "C415406"
+			(at 92.71 140.97 0)
+			(hide yes)
+			(show_name no)
+			(do_not_autoplace no)
+			(effects
+				(font
+					(size 1.27 1.27)
+				)
 			)
 		)
@@
 			)
 		)
+		(property "LCSC" "C126598"
+			(at 267.97 140.97 0)
+			(hide yes)
+			(show_name no)
+			(do_not_autoplace no)
+			(effects
+				(font
+					(size 1.27 1.27)
+				)
+			)
+		)
 		(pin "1"
 		)
@@
 			)
 		)
-		(property "Notes" "33 uH (TI tabla 9-1, 400 kHz, 5 V). Isat 3.7 A > limite high-side max del LMR38010 (1.9 A); DCR 105 mohm max. AEC-Q200."
+		(property "Notes" "33 uH (TI tabla 9-1, 400 kHz, 5 V). Isat 3.7 A > limite high-side max del LMR38010 (1.9 A); DCR 105 mohm max. AEC-Q200. Compra (2026-10-30): sin stock en JLC/LCSC; comprar en DigiKey/Mouser y soldar a mano."
 			(at 229.87 133.35 0)
 			(hide yes)
@@
 		)
 		(property "DNP" ""
+			(at 229.87 133.35 0)
+			(hide yes)
+			(show_name no)
+			(do_not_autoplace no)
+			(effects
+				(font
+					(size 1.27 1.27)
+				)
+			)
+		)
+		(property "LCSC" "C5119929"
 			(at 229.87 133.35 0)
 			(hide yes)
@@
 			)
 		)
-		(property "Notes" "Buck 80 V / 1 A, PFM + spread spectrum. PROD: LMR38010SQDDARQ1 (AEC-Q100, SNVSC72B). PROTO: LMR38010SDDAR (LCSC C5219310), equivalente comercial: mismo modo, pinout y DDA0008B (ver PENDIENTES 'Equivalencia LMR38010'). EP con 6 vias de 0.2 mm a GND_VEH (soldable con aire caliente). Pin a pin con LMR38020 (2 A). Simbolo de easyeda2kicad con tipos de pin ajustados."
+		(property "Notes" "Buck 80 V / 1 A, PFM + spread spectrum. PROD: LMR38010SQDDARQ1 (AEC-Q100, SNVSC72B). PROTO: LMR38010SDDAR (LCSC C5219310), equivalente comercial: mismo modo, pinout y DDA0008B (ver PENDIENTES 'Equivalencia LMR38010'). EP con 6 vias de 0.2 mm a GND_VEH (soldable con aire caliente). Pin a pin con LMR38020 (2 A). Simbolo de easyeda2kicad con tipos de pin ajustados. PROD (2026-10-30): sin stock suficiente en JLC/LCSC para 100 placas; comprar en DigiKey/Mouser."
 			(at 153.67 138.43 0)
 			(hide yes)
@@
 		)
 		(property "DNP" ""
+			(at 153.67 138.43 0)
+			(hide yes)
+			(show_name no)
+			(do_not_autoplace no)
+			(effects
+				(font
+					(size 1.27 1.27)
+				)
+			)
+		)
+		(property "LCSC" "C18198885"
 			(at 153.67 138.43 0)
 			(hide yes)
@@
 			)
 		)
-		(property "Notes" "C_IN del LMR38010 (TI: >= 4.7 uF ceramico, X7R, idealmente 2 x VIN max). 100 V X7S AEC-Q200. 1210 por tension y DC bias. Pegado a VIN/GND de U201. MPN a verificar."
+		(property "Notes" "C_IN del LMR38010 (TI: >= 4.7 uF ceramico, X7R, idealmente 2 x VIN max). 100 V X7S AEC-Q200. 1210 por tension y DC bias. Pegado a VIN/GND de U201. MPN a verificar. PROTO (2026-10-30): Samsung CL32B475KCVZNWE (LCSC C17288249), sin AEC-Q200, solo para el prototipo. PROD: este MPN (AEC-Q200); sin stock en JLC/LCSC, comprar en DigiKey/Mouser."
 			(at 80.01 140.97 0)
 			(hide yes)
@@
 		)
 		(property "DNP" ""
+			(at 80.01 140.97 0)
+			(hide yes)
+			(show_name no)
+			(do_not_autoplace no)
+			(effects
+				(font
+					(size 1.27 1.27)
+				)
+			)
+		)
+		(property "LCSC" "C2168848"
+			(at 80.01 140.97 0)
+			(hide yes)
+			(show_name no)
+			(do_not_autoplace no)
+			(effects
+				(font
+					(size 1.27 1.27)
+				)
+			)
+		)
+		(property "MPN_PROTO" "CL32B475KCVZNWE"
+			(at 80.01 140.97 0)
+			(hide yes)
+			(show_name no)
+			(do_not_autoplace no)
+			(effects
+				(font
+					(size 1.27 1.27)
+				)
+			)
+		)
+		(property "Manufacturer_PROTO" "Samsung"
+			(at 80.01 140.97 0)
+			(hide yes)
+			(show_name no)
+			(do_not_autoplace no)
+			(effects
+				(font
+					(size 1.27 1.27)
+				)
+			)
+		)
+		(property "LCSC_PROTO" "C17288249"
 			(at 80.01 140.97 0)
 			(hide yes)
@@
 			)
 		)
-		(property "Notes" "R_FBT (TI recomienda 100k). VOUT = 1 V x (1 + 100k/24.9k) = 5.02 V."
+		(property "Notes" "R_FBT (TI recomienda 100k). VOUT = 1 V x (1 + 100k/24.9k) = 5.02 V. PROTO (2026-10-30): UNI-ROYAL 0603WAF1003T5E (LCSC C25803, JLC basic), misma especificación, sin AEC-Q200."
 			(at 298.45 133.35 0)
 			(hide yes)
@@
 		)
 		(property "DNP" ""
+			(at 298.45 133.35 0)
+			(hide yes)
+			(show_name no)
+			(do_not_autoplace no)
+			(effects
+				(font
+					(size 1.27 1.27)
+				)
+			)
+		)
+		(property "LCSC" "C116674"
+			(at 298.45 133.35 0)
+			(hide yes)
+			(show_name no)
+			(do_not_autoplace no)
+			(effects
+				(font
+					(size 1.27 1.27)
+				)
+			)
+		)
+		(property "MPN_PROTO" "0603WAF1003T5E"
+			(at 298.45 133.35 0)
+			(hide yes)
+			(show_name no)
+			(do_not_autoplace no)
+			(effects
+				(font
+					(size 1.27 1.27)
+				)
+			)
+		)
+		(property "Manufacturer_PROTO" "UNI-ROYAL"
+			(at 298.45 133.35 0)
+			(hide yes)
+			(show_name no)
+			(do_not_autoplace no)
+			(effects
+				(font
+					(size 1.27 1.27)
+				)
+			)
+		)
+		(property "LCSC_PROTO" "C25803"
 			(at 298.45 133.35 0)
 			(hide yes)
@@
 			)
 		)
+		(property "LCSC" "C126598"
+			(at 280.67 140.97 0)
+			(hide yes)
+			(show_name no)
+			(do_not_autoplace no)
+			(effects
+				(font
+					(size 1.27 1.27)
+				)
+			)
+		)
 		(pin "1"
 		)
@@
 			)
 		)
-		(property "Notes" "C_BOOT entre BOOT (7) y SW (8): 100 nF >= 16 V (TI 9.2.2.7)."
+		(property "Notes" "C_BOOT entre BOOT (7) y SW (8): 100 nF >= 16 V (TI 9.2.2.7). PROTO (2026-10-30): Yageo CC0603KRX7R9BB104 (LCSC C14663, JLC basic), misma especificación, sin AEC-Q200."
 			(at 204.47 140.97 0)
 			(hide yes)
@@
 		)
 		(property "DNP" ""
+			(at 204.47 140.97 0)
+			(hide yes)
+			(show_name no)
+			(do_not_autoplace no)
+			(effects
+				(font
+					(size 1.27 1.27)
+				)
+			)
+		)
+		(property "LCSC" "C85864"
+			(at 204.47 140.97 0)
+			(hide yes)
+			(show_name no)
+			(do_not_autoplace no)
+			(effects
+				(font
+					(size 1.27 1.27)
+				)
+			)
+		)
+		(property "MPN_PROTO" "CC0603KRX7R9BB104"
+			(at 204.47 140.97 0)
+			(hide yes)
+			(show_name no)
+			(do_not_autoplace no)
+			(effects
+				(font
+					(size 1.27 1.27)
+				)
+			)
+		)
+		(property "Manufacturer_PROTO" "Yageo"
+			(at 204.47 140.97 0)
+			(hide yes)
+			(show_name no)
+			(do_not_autoplace no)
+			(effects
+				(font
+					(size 1.27 1.27)
+				)
+			)
+		)
+		(property "LCSC_PROTO" "C14663"
 			(at 204.47 140.97 0)
 			(hide yes)
@@
 			)
 		)
+		(property "LCSC" "C227732"
+			(at 298.45 148.59 0)
+			(hide yes)
+			(show_name no)
+			(do_not_autoplace no)
+			(effects
+				(font
+					(size 1.27 1.27)
+				)
+			)
+		)
 		(pin "1"
 		)
@@
 			)
 		)
+		(property "LCSC" "C228007"
+			(at 316.23 140.97 0)
+			(hide yes)
+			(show_name no)
+			(do_not_autoplace no)
+			(effects
+				(font
+					(size 1.27 1.27)
+				)
+			)
+		)
 		(pin "1"
 		)
@@
 			(at 255.27 140.97 0)
 			(hide yes)
+			(show_name no)
+			(do_not_autoplace no)
+			(effects
+				(font
+					(size 1.27 1.27)
+				)
+			)
+		)
+		(property "LCSC" "C126598"
+			(at 255.27 140.97 0)
+			(hide yes)

Commit message: [Claude Code] bom: compra principal en LCSC + DigiKey/Mouser; consolidación de pasivos
- Plan: JLC solo PCB + stencil Top; componentes de LCSC soldados a mano.
- Consolidación (solo valor/campos): R702/R752 4k7 → 2.2k; 23 × 100 nF a un
  MPN de 100 V X7R; PROTO 1 µF 50 V y 10 µF 25 V X7R. BOM PROTO 70 → 68 líneas.
- LCSC_BOM_COMPLETO_PROTO.csv: 6 juegos, 62 líneas, USD 552.43 (3 juegos: 286.65).
- DIGIKEY_MOUSER.csv: L201, U503, Q101, Q102, F101 (0 en LCSC), ≈ USD 99.54.
- Resumen de costos en BOM_SOURCING.md; archivos de JLC al día como alternativa.
- DRC 0 errores / 3 avisos aceptados, paridad 0, ERC 0 / 5.

Co-Authored-By: Claude Opus 5.5 <noreply@anthropic.com>
Parts:
- C202: LCSC_PROTO (none) -> C88219; MPN_PROTO (none) -> 0603B104K101NT; Manufacturer_PROTO (none) -> FH; Notes Bypass de alta frecuencia de VIN (TI: 100-220 nF, 100 V X7R), lo mas cerca posible de los pines 3 y 1. -> Bypass de alta frecuencia de VIN (TI: 100-220 nF, 100 V X7R), lo mas cerca posible de los pines 3 y 1. PROTO (2026-10-30, consolidacion): un solo MPN para los 100 nF 0603: 100 V X7R (FH 0603B104K101NT, LCSC C88219), sin AEC-Q200. PROD: Murata GCM188R72A104KA64D (100 V, AEC-Q200). Mismo valor y tolerancia.
- C203: LCSC C85864 -> C415406; LCSC_PROTO C14663 -> C88219; MPN GCM188R71H104KA57D -> GCM188R72A104KA64D; MPN_PROTO CC0603KRX7R9BB104 -> 0603B104K101NT; Manufacturer_PROTO Yageo -> FH; Notes C_BOOT entre BOOT (7) y SW (8): 100 nF >= 16 V (TI 9.2.2.7). PROTO (2026-10-30): Yageo CC0603KRX7R9BB104 (LCSC C14663, JLC basic), misma especificación, sin AEC-Q200. -> C_BOOT entre BOOT (7) y SW (8): 100 nF >= 16 V (TI 9.2.2.7). PROTO (2026-10-30, consolidacion): un solo MPN para los 100 nF 0603: 100 V X7R (FH 0603B104K101NT, LCSC C88219), sin AEC-Q200. PROD: Murata GCM188R72A104KA64D (100 V, AEC-Q200). Mismo valor y tolerancia.
Changed lines of the file:
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@@
 			)
 		)
-		(property "Notes" "Bypass de alta frecuencia de VIN (TI: 100-220 nF, 100 V X7R), lo mas cerca posible de los pines 3 y 1."
+		(property "Notes" "Bypass de alta frecuencia de VIN (TI: 100-220 nF, 100 V X7R), lo mas cerca posible de los pines 3 y 1. PROTO (2026-10-30, consolidacion): un solo MPN para los 100 nF 0603: 100 V X7R (FH 0603B104K101NT, LCSC C88219), sin AEC-Q200. PROD: Murata GCM188R72A104KA64D (100 V, AEC-Q200). Mismo valor y tolerancia."
 			(at 92.71 140.97 0)
 			(hide yes)
@@
 		)
 		(property "LCSC" "C415406"
+			(at 92.71 140.97 0)
+			(hide yes)
+			(show_name no)
+			(do_not_autoplace no)
+			(effects
+				(font
+					(size 1.27 1.27)
+				)
+			)
+		)
+		(property "MPN_PROTO" "0603B104K101NT"
+			(at 92.71 140.97 0)
+			(hide yes)
+			(show_name no)
+			(do_not_autoplace no)
+			(effects
+				(font
+					(size 1.27 1.27)
+				)
+			)
+		)
+		(property "Manufacturer_PROTO" "FH"
+			(at 92.71 140.97 0)
+			(hide yes)
+			(show_name no)
+			(do_not_autoplace no)
+			(effects
+				(font
+					(size 1.27 1.27)
+				)
+			)
+		)
+		(property "LCSC_PROTO" "C88219"
 			(at 92.71 140.97 0)
 			(hide yes)
@@
 			)
 		)
-		(property "MPN" "GCM188R71H104KA57D"
+		(property "MPN" "GCM188R72A104KA64D"
 			(at 204.47 140.97 0)
 			(hide yes)
@@
 			)
 		)
-		(property "Notes" "C_BOOT entre BOOT (7) y SW (8): 100 nF >= 16 V (TI 9.2.2.7). PROTO (2026-10-30): Yageo CC0603KRX7R9BB104 (LCSC C14663, JLC basic), misma especificación, sin AEC-Q200."
+		(property "Notes" "C_BOOT entre BOOT (7) y SW (8): 100 nF >= 16 V (TI 9.2.2.7). PROTO (2026-10-30, consolidacion): un solo MPN para los 100 nF 0603: 100 V X7R (FH 0603B104K101NT, LCSC C88219), sin AEC-Q200. PROD: Murata GCM188R72A104KA64D (100 V, AEC-Q200). Mismo valor y tolerancia."
 			(at 204.47 140.97 0)
 			(hide yes)
@@
 			)
 		)
-		(property "LCSC" "C85864"
+		(property "LCSC" "C415406"
 			(at 204.47 140.97 0)
 			(hide yes)
@@
 			)
 		)
-		(property "MPN_PROTO" "CC0603KRX7R9BB104"
+		(property "MPN_PROTO" "0603B104K101NT"
 			(at 204.47 140.97 0)
 			(hide yes)
@@
 			)
 		)
-		(property "Manufacturer_PROTO" "Yageo"
+		(property "Manufacturer_PROTO" "FH"
 			(at 204.47 140.97 0)
 			(hide yes)
@@
 			)
 		)
-		(property "LCSC_PROTO" "C14663"
+		(property "LCSC_PROTO" "C88219"
 			(at 204.47 140.97 0)
 			(hide yes)
