File: sheets/80_supervision.kicad_sch (KiCad schematic)
At the start: 11 parts, among them U801 TPS3828-33Q1

Commit message: [Codex] Integra cierre de Claude y valida sincronizacion previa al layout
Parts:
- U801: Alt_MPN (none) -> TPS3828-33DBVR; MPN_PROTO (none) -> TPS3828-33DBVR
Changed lines of the file:
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@@
+			)
+		)
+		(property "MPN_PROTO" "TPS3828-33DBVR"
+			(at 127 76.2 0)
+			(hide yes)
+			(show_name no)
+			(do_not_autoplace no)
+			(effects
+				(font
+					(size 1.27 1.27)
+				)
+			)
+		)
+		(property "Alt_MPN" "TPS3828-33DBVR"
+			(at 127 76.2 0)
+			(hide yes)
+			(show_name no)
+			(do_not_autoplace no)
+			(effects
+				(font
+					(size 1.27 1.27)
+				)
 			)
 		)

Commit message: update
Other:
- moved on the sheet: C801
Changed lines of the file:
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@@
 	(wire
 		(pts
-			(xy 165.1 67.31) (xy 165.1 69.85)
+			(xy 181.61 77.47) (xy 181.61 80.01)
 		)
 		(stroke
@@
 	(wire
 		(pts
-			(xy 165.1 59.69) (xy 165.1 57.15)
+			(xy 181.61 69.85) (xy 181.61 67.31)
 		)
 		(stroke
@@
 		(dnp no)
 		(property "Reference" "R804"
-			(at 109.22 110.49 90)
+			(at 111.506 112.268 90)
 			(show_name no)
 			(do_not_autoplace no)
@@
 		)
 		(property "Value" "470"
-			(at 109.22 113.03 90)
+			(at 110.998 114.3 90)
 			(show_name no)
 			(do_not_autoplace no)
@@
 		(dnp no)
 		(property "Reference" "R803"
-			(at 109.22 97.79 90)
+			(at 111.506 99.568 90)
 			(show_name no)
 			(do_not_autoplace no)
@@
 		)
 		(property "Value" "470"
-			(at 109.22 100.33 90)
+			(at 111.252 101.6 90)
 			(show_name no)
 			(do_not_autoplace no)
@@
 	(symbol
 		(lib_id "INCLI-VA:+3V3_D")
-		(at 165.1 57.15 0)
+		(at 181.61 67.31 0)
 		(unit 1)
 		(body_style 1)
@@
 		(dnp no)
 		(property "Reference" "#PWR0578"
-			(at 167.64 55.88 0)
+			(at 184.15 66.04 0)
 			(hide yes)
 			(show_name no)
@@
 		)
 		(property "Value" "+3V3_D"
-			(at 165.1 52.07 0)
+			(at 181.61 62.23 0)
 			(show_name no)
 			(do_not_autoplace no)
@@
 		)
 		(property "Footprint" ""
-			(at 165.1 57.15 0)
+			(at 181.61 67.31 0)
 			(hide yes)
 			(show_name no)
@@
 		)
 		(property "Datasheet" ""
-			(at 165.1 57.15 0)
+			(at 181.61 67.31 0)
 			(hide yes)
 			(show_name no)
@@
 		)
 		(property "Description" ""
-			(at 165.1 57.15 0)
+			(at 181.61 67.31 0)
 			(hide yes)
 			(show_name no)
@@
 	(symbol
 		(lib_id "Device:C")
-		(at 165.1 63.5 0)
+		(at 181.61 73.66 0)
 		(unit 1)
 		(body_style 1)
@@
 		(dnp no)
 		(property "Reference" "C801"
-			(at 167.64 62.23 0)
+			(at 184.15 72.39 0)
 			(show_name no)
 			(do_not_autoplace no)
@@
 		)
 		(property "Value" "100nF"
-			(at 167.64 64.77 0)
+			(at 184.15 74.93 0)
 			(show_name no)
 			(do_not_autoplace no)
@@
 		)
 		(property "Footprint" "Capacitor_SMD:C_0603_1608Metric"
-			(at 165.1 63.5 0)
+			(at 181.61 73.66 0)
 			(hide yes)
 			(show_name no)
@@
 		)
 		(property "Datasheet" "https://www.murata.com/en-global/products/productdetail?partno=GCM188R71H104KA57D"
-			(at 165.1 63.5 0)
+			(at 181.61 73.66 0)
 			(hide yes)
 			(show_name no)
@@
 		)
 		(property "Description" ""
-			(at 165.1 63.5 0)
+			(at 181.61 73.66 0)
 			(hide yes)
 			(show_name no)
@@
 		)
 		(property "MPN" "GCM188R71H104KA57D"
-			(at 165.1 63.5 0)
+			(at 181.61 73.66 0)
 			(hide yes)
 			(show_name no)
@@
 		)
 		(property "Manufacturer" "Murata"
-			(at 165.1 63.5 0)
+			(at 181.61 73.66 0)
 			(hide yes)
 			(show_name no)
@@
 		)
 		(property "DNP" ""
-			(at 165.1 63.5 0)
+			(at 181.61 73.66 0)
 			(hide yes)
 			(show_name no)
@@
 		)
 		(property "Notes" "Desacople de U801."
-			(at 165.1 63.5 0)
+			(at 181.61 73.66 0)
 			(hide yes)
 			(show_name no)
@@
 	(symbol
 		(lib_id "INCLI-VA:GND_VEH")
-		(at 165.1 69.85 0)
+		(at 181.61 80.01 0)
 		(unit 1)
 		(body_style 1)
@@
 		(dnp no)
 		(property "Reference" "#PWR0579"
-			(at 167.64 68.58 0)
+			(at 184.15 78.74 0)
 			(hide yes)
 			(show_name no)
@@
 		)
 		(property "Value" "GND_VEH"
-			(at 165.1 73.66 0)
+			(at 181.61 83.82 0)
 			(show_name no)
 			(do_not_autoplace no)
@@
 		)
 		(property "Footprint" ""
-			(at 165.1 69.85 0)
+			(at 181.61 80.01 0)
 			(hide yes)
 			(show_name no)
@@
 		)
 		(property "Datasheet" ""
-			(at 165.1 69.85 0)
+			(at 181.61 80.01 0)
 			(hide yes)
 			(show_name no)
@@
 		)
 		(property "Description" ""
-			(at 165.1 69.85 0)
-			(hide yes)
-			(show_name no)
+			(at 181.61 80.01 0)
+			(hide yes)
+			(show_name no)
