File: sheets/80_supervision.kicad_sch (KiCad schematic)
At the start: 11 parts, among them U801 TPS3828-33Q1

Commit message: [Claude Code] esquema+PCB: campos LCSC y sustitutos PROTO del BOM (pcb-v1-rc2)
- Esquema (solo campos, ocultos): LCSC en todos los componentes; MPN_PROTO,
  LCSC_PROTO y Manufacturer_PROTO con los sustitutos aceptados; Notes con
  compra y montaje (Q101, Q102, F101, L201, U503 a mano desde DigiKey/Mouser).
  MPN (PROD), valores, huellas y conexiones sin cambios. LCSC Part -> LCSC.
- PCB: mismos campos en las 145 huellas, insertados como texto (equivalente
  a F8 solo para campos); nada cambia fuera de las huellas.
- ERC por hoja igual que antes (0 errores, 5 avisos). DRC 0 errores / 3 avisos
  aceptados, 0 sin rutear, paridad 0 (antes de sincronizar: 145).
- etapa6_fab.py usa los campos _PROTO y genera bom_jlc_lcsc.csv; este y
  cpl_jlc.csv salen idénticos (60 líneas, 123 piezas). Gerbers sin cambios
  de contenido.

Co-Authored-By: Claude Opus 5.5 <noreply@anthropic.com>
Parts:
- C801: LCSC (none) -> C85864; LCSC_PROTO (none) -> C14663; MPN_PROTO (none) -> CC0603KRX7R9BB104; Manufacturer_PROTO (none) -> Yageo; Notes Desacople de U801. -> Desacople de U801. PROTO (2026-10-30): Yageo CC0603KRX7R9BB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
- D801: LCSC (none) -> C98224
- D802: LCSC (none) -> C284871
- R801: LCSC (none) -> C116692
- R802: LCSC (none) -> C141796; LCSC_PROTO (none) -> C21189; MPN_PROTO (none) -> 0603WAF0000T5E; Manufacturer_PROTO (none) -> UNI-ROYAL; Notes 0 ohm en serie con RESET. Sin montar, la placa funciona sin supervisor (depuracion). -> 0 ohm en serie con RESET. Sin montar, la placa funciona sin supervisor (depuracion). PROTO (2026-10-30): UNI-ROYAL 0603WAF0000T5E (LCSC C21189, JLC basic), misma especificación, sin AEC-Q200.
- R803, R804: LCSC (none) -> C144657; LCSC_PROTO (none) -> C23179; MPN_PROTO (none) -> 0603WAF4700T5E; Manufacturer_PROTO (none) -> UNI-ROYAL; Notes 470 ohm: ~3 mA desde 3.3 V. DNP en PROD (caja ABS opaca). -> 470 ohm: ~3 mA desde 3.3 V. DNP en PROD (caja ABS opaca). P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
- R805: LCSC (none) -> C141796; LCSC_PROTO (none) -> C21189; MPN_PROTO (none) -> 0603WAF0000T5E; Manufacturer_PROTO (none) -> UNI-ROYAL; Notes VAR_ID0 (IO4) = 0 si la variante lleva CAN. Tabla (ID1 ID0): 11 base | 10 CAN | 01 solo DO | 00 CAN + DO. ROT se detecta por SPI (AS5147U). -> VAR_ID0 (IO4) = 0 si la variante lleva CAN. Tabla (ID1 ID0): 11 base | 10 CAN | 01 solo DO | 00 CAN + DO. ROT se detecta por SPI (AS5147U). PROTO (2026-10-30): UNI-ROYAL 0603WAF0000T5E (LCSC C21189, JLC basic), misma especificación, sin AEC-Q200.
- R806: LCSC (none) -> C141796; LCSC_PROTO (none) -> C21189; MPN_PROTO (none) -> 0603WAF0000T5E; Manufacturer_PROTO (none) -> UNI-ROYAL; Notes VAR_ID1 (IO5) = 0 si la variante lleva salidas DO. Tabla (ID1 ID0): 11 base | 10 CAN | 01 solo DO | 00 CAN + DO. ROT se detecta por SPI (AS5147U). -> VAR_ID1 (IO5) = 0 si la variante lleva salidas DO. Tabla (ID1 ID0): 11 base | 10 CAN | 01 solo DO | 00 CAN + DO. ROT se detecta por SPI (AS5147U). PROTO (2026-10-30): UNI-ROYAL 0603WAF0000T5E (LCSC C21189, JLC basic), misma especificación, sin AEC-Q200.
- R807: LCSC (none) -> C141796
- U801: LCSC (none) -> C2872895; LCSC_PROTO (none) -> C20032; Notes Supervisor de +3V3_D + watchdog, AEC-Q100 (TI SGLS143E). VIT- 2.84/2.93/3.0 V, reset 120/200/300 ms, ttout 0.9/1.6/2.5 s. RESET drenador abierto (TPS3828) -> MCU_RST_N (wire-OR con R401 10k + C403 1 uF + SW401). WDI en alta impedancia = watchdog deshabilitado (7.3.4): GPIO17 queda en alta Z en boot/flasheo. Simbolo oficial TPS3823-xxDBV: mismo pinout (1 RESET, 2 GND, 3 MR, 4 WDI, 5 VDD). -> Supervisor de +3V3_D + watchdog, AEC-Q100 (TI SGLS143E). VIT- 2.84/2.93/3.0 V, reset 120/200/300 ms, ttout 0.9/1.6/2.5 s. RESET drenador abierto (TPS3828) -> MCU_RST_N (wire-OR con R401 10k + C403 1 uF + SW401). WDI en alta impedancia = watchdog deshabilitado (7.3.4): GPIO17 queda en alta Z en boot/flasheo. Simbolo oficial TPS3823-xxDBV: mismo pinout (1 RESET, 2 GND, 3 MR, 4 WDI, 5 VDD). PROD (2026-10-30): sin stock suficiente en JLC/LCSC para 100 placas; comprar en DigiKey/Mouser.

Commit message: [Claude Code] TP de la cara inferior rotulados, TP406/TP505 GND con agujero, R803/R804 2.2k
- B.Silk: nombre de señal junto a cada TP (verificado con la red), GND con recuadro,
  nota «CAN: medir vs GND_CAN (J1-5)».
- TP406 (40_mcu) y TP505 (50_sensors): GND_VEH THT D2.5/1.2 mm, en esquema y PCB,
  fuera de BOM/CPL.
- LEDs: R803/R804 470 → 2.2k (0603WAF2201T5E C4190 basic; PROD AC0603FR-072K2L);
  ~0.61 / 0.70 mA; brillo por PWM (PENDIENTES, firmware).
- DRC 0 errores / 3 avisos aceptados, paridad 0, ERC 0 / 5; fab/proto y BOM regenerados.

Co-Authored-By: Claude Opus 5.5 <noreply@anthropic.com>
Parts:
- R803, R804: value 470 -> 2.2k; LCSC C144657 -> C125931; LCSC_PROTO C23179 -> C4190; MPN AC0603FR-07470RL -> AC0603FR-072K2L; MPN_PROTO 0603WAF4700T5E -> 0603WAF2201T5E; Notes 470 ohm: ~3 mA desde 3.3 V. DNP en PROD (caja ABS opaca). P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 -> 2.2 kohm: ~0.6 mA (verde, Vf ~1.95 V) y ~0.7 mA (rojo, Vf ~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
Changed lines of the file:
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@@
 			)
 		)
-		(property "Value" "470"
+		(property "Value" "2.2k"
 			(at 110.998 114.3 90)
 			(show_name no)
@@
 			)
 		)
-		(property "MPN" "AC0603FR-07470RL"
+		(property "MPN" "AC0603FR-072K2L"
 			(at 109.22 114.3 0)
 			(hide yes)
@@
 			)
 		)
-		(property "Notes" "470 ohm: ~3 mA desde 3.3 V. DNP en PROD (caja ABS opaca). PROTO (2026-10-30): UNI-ROYAL 0603WAF4700T5E (LCSC C23179, JLC basic), misma especificación, sin AEC-Q200."
-			(at 109.22 114.3 0)
-			(hide yes)
-			(show_name no)
-			(do_not_autoplace no)
-			(effects
-				(font
-					(size 1.27 1.27)
-				)
-			)
-		)
-		(property "LCSC" "C144657"
-			(at 109.22 114.3 0)
-			(hide yes)
-			(show_name no)
-			(do_not_autoplace no)
-			(effects
-				(font
-					(size 1.27 1.27)
-				)
-			)
-		)
-		(property "MPN_PROTO" "0603WAF4700T5E"
+		(property "Notes" "2.2 kohm: ~0.6 mA (verde, Vf ~1.95 V) y ~0.7 mA (rojo, Vf ~1.75 V) desde 3.3 V (Lite-On LTST-C171KGKT rev. F / LTST-C171KRKT rev. E, fig. 2). Un solo valor para R803 y R804 (una linea de BOM); el brillo se iguala por PWM en firmware. DNP en PROD (caja ABS opaca). PROTO (2026-10-30): UNI-ROYAL 0603WAF2201T5E (LCSC C4190, JLC basic), misma especificacion, sin AEC-Q200."
+			(at 109.22 114.3 0)
+			(hide yes)
+			(show_name no)
+			(do_not_autoplace no)
+			(effects
+				(font
+					(size 1.27 1.27)
+				)
+			)
+		)
+		(property "LCSC" "C125931"
+			(at 109.22 114.3 0)
+			(hide yes)
+			(show_name no)
+			(do_not_autoplace no)
+			(effects
+				(font
+					(size 1.27 1.27)
+				)
+			)
+		)
+		(property "MPN_PROTO" "0603WAF2201T5E"
 			(at 109.22 114.3 0)
 			(hide yes)
@@
 			)
 		)
-		(property "LCSC_PROTO" "C23179"
+		(property "LCSC_PROTO" "C4190"
 			(at 109.22 114.3 0)
 			(hide yes)
@@
 			)
 		)
-		(property "Value" "470"
+		(property "Value" "2.2k"
 			(at 111.252 101.6 90)
 			(show_name no)
@@
 			)
 		)
-		(property "MPN" "AC0603FR-07470RL"
+		(property "MPN" "AC0603FR-072K2L"
 			(at 109.22 101.6 0)
 			(hide yes)
@@
 			)
 		)
-		(property "Notes" "470 ohm: ~3 mA desde 3.3 V. DNP en PROD (caja ABS opaca). PROTO (2026-10-30): UNI-ROYAL 0603WAF4700T5E (LCSC C23179, JLC basic), misma especificación, sin AEC-Q200."
-			(at 109.22 101.6 0)
-			(hide yes)
-			(show_name no)
-			(do_not_autoplace no)
-			(effects
-				(font
-					(size 1.27 1.27)
-				)
-			)
-		)
-		(property "LCSC" "C144657"
-			(at 109.22 101.6 0)
-			(hide yes)
-			(show_name no)
-			(do_not_autoplace no)
-			(effects
-				(font
-					(size 1.27 1.27)
-				)
-			)
-		)
-		(property "MPN_PROTO" "0603WAF4700T5E"
+		(property "Notes" "2.2 kohm: ~0.6 mA (verde, Vf ~1.95 V) y ~0.7 mA (rojo, Vf ~1.75 V) desde 3.3 V (Lite-On LTST-C171KGKT rev. F / LTST-C171KRKT rev. E, fig. 2). Un solo valor para R803 y R804 (una linea de BOM); el brillo se iguala por PWM en firmware. DNP en PROD (caja ABS opaca). PROTO (2026-10-30): UNI-ROYAL 0603WAF2201T5E (LCSC C4190, JLC basic), misma especificacion, sin AEC-Q200."
+			(at 109.22 101.6 0)
+			(hide yes)
+			(show_name no)
+			(do_not_autoplace no)
+			(effects
+				(font
+					(size 1.27 1.27)
+				)
+			)
+		)
+		(property "LCSC" "C125931"
+			(at 109.22 101.6 0)
+			(hide yes)
+			(show_name no)
+			(do_not_autoplace no)
+			(effects
+				(font
+					(size 1.27 1.27)
+				)
+			)
+		)
+		(property "MPN_PROTO" "0603WAF2201T5E"
 			(at 109.22 101.6 0)
 			(hide yes)
@@
 			)
 		)
-		(property "LCSC_PROTO" "C23179"
-			(at 109.22 101.6 0)
-			(hide yes)
+		(property "LCSC_PROTO" "C4190"
+			(at 109.22 101.6 0)
+			(hide yes)

Commit message: [Claude Code] bom: compra principal en LCSC + DigiKey/Mouser; consolidación de pasivos
- Plan: JLC solo PCB + stencil Top; componentes de LCSC soldados a mano.
- Consolidación (solo valor/campos): R702/R752 4k7 → 2.2k; 23 × 100 nF a un
  MPN de 100 V X7R; PROTO 1 µF 50 V y 10 µF 25 V X7R. BOM PROTO 70 → 68 líneas.
- LCSC_BOM_COMPLETO_PROTO.csv: 6 juegos, 62 líneas, USD 552.43 (3 juegos: 286.65).
- DIGIKEY_MOUSER.csv: L201, U503, Q101, Q102, F101 (0 en LCSC), ≈ USD 99.54.
- Resumen de costos en BOM_SOURCING.md; archivos de JLC al día como alternativa.
- DRC 0 errores / 3 avisos aceptados, paridad 0, ERC 0 / 5.

Co-Authored-By: Claude Opus 5.5 <noreply@anthropic.com>
Parts:
- C801: LCSC C85864 -> C415406; LCSC_PROTO C14663 -> C88219; MPN GCM188R71H104KA57D -> GCM188R72A104KA64D; MPN_PROTO CC0603KRX7R9BB104 -> 0603B104K101NT; Manufacturer_PROTO Yageo -> FH; Notes Desacople de U801. PROTO (2026-10-30): Yageo CC0603KRX7R9BB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 -> Desacople de U801. PROTO (2026-10-30, consolidacion): un so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
Changed lines of the file:
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@@
 			)
 		)
-		(property "MPN" "GCM188R71H104KA57D"
+		(property "MPN" "GCM188R72A104KA64D"
 			(at 181.61 73.66 0)
 			(hide yes)
@@
 			)
 		)
-		(property "Notes" "Desacople de U801. PROTO (2026-10-30): Yageo CC0603KRX7R9BB104 (LCSC C14663, JLC basic), misma especificación, sin AEC-Q200."
+		(property "Notes" "Desacople de U801. PROTO (2026-10-30, consolidacion): un solo MPN para los 100 nF 0603: 100 V X7R (FH 0603B104K101NT, LCSC C88219), sin AEC-Q200. PROD: Murata GCM188R72A104KA64D (100 V, AEC-Q200). Mismo valor y tolerancia."
 			(at 181.61 73.66 0)
 			(hide yes)
@@
 			)
 		)
-		(property "LCSC" "C85864"
+		(property "LCSC" "C415406"
 			(at 181.61 73.66 0)
 			(hide yes)
@@
 			)
 		)
-		(property "MPN_PROTO" "CC0603KRX7R9BB104"
+		(property "MPN_PROTO" "0603B104K101NT"
 			(at 181.61 73.66 0)
 			(hide yes)
@@
 			)
 		)
-		(property "Manufacturer_PROTO" "Yageo"
+		(property "Manufacturer_PROTO" "FH"
 			(at 181.61 73.66 0)
 			(hide yes)
@@
 			)
 		)
-		(property "LCSC_PROTO" "C14663"
+		(property "LCSC_PROTO" "C88219"
 			(at 181.61 73.66 0)
 			(hide yes)
