File: INCLI-VA.kicad_pcb (KiCad board)
At the start: 2 copper layers, 151 parts, among them J1 MSTB 2,5/5-GF-5,08, J2 MSTB 2,5/2-GF-5,08, J401 USB4105-GF-A, J402 UART0, Q101 STD18NF25, Q102 IPD30N10S3L-34, Q701 FDD7N25LZ, Q702 BC817-40, Q703 BC807-40, Q751 FDD7N25LZ, Q752 BC817-40, Q753 BC807-40, SW401 RESET, SW402 BOOT, U1 ADM3055E, U101 LM74930QRGERQ1, U201 TPS7A1650QDGNRQ1, U202 ISO7763FQDWRQ1, U301 TPS62A02QDRLRQ1, U302 LP5907QMFX-3.3Q1, U401 ESP32-S3-WROOM-1-N8R2, U402 USBLC6-2SC6, U501 SCL3300-D01, U502 ASM330LHHTR, U503 AS5147U-HTSM

Commit message: move pcb
Parts:
- moved U101 211.5 mm to (61.5, 55.2)
- moved C204 204.3 mm to (58.0, 81.1), turned to -90 degrees
- moved C206 197.1 mm to (67.4, 76.5)
- moved U201 195.8 mm to (68.0, 81.0)
- moved C205 195.2 mm to (62.0, 81.1), turned to -90 degrees
- moved D701 154.9 mm to (43.5, 116.0), turned to 90 degrees
- moved R709 154.1 mm to (37.0, 113.5), turned to 90 degrees
- moved R708 153.0 mm to (37.0, 118.5), turned to 90 degrees
- moved D703 150.5 mm to (36.5, 106.1), turned to -90 degrees
- moved R710 147.6 mm to (37.0, 110.0)
- moved R707 145.5 mm to (41.0, 101.3), turned to -90 degrees
- moved Q701 144.9 mm to (51.0, 116.4), turned to -90 degrees
- moved R701 142.7 mm to (48.5, 107.3), turned to 90 degrees
- moved Q703 140.8 mm to (52.0, 96.3), turned to 180 degrees
- moved C701 138.6 mm to (44.0, 101.3), turned to -90 degrees
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
Commit message: order pcb
Parts:
- added H1: MountingHole_3.2mm_M3_ISO7380_Pad, MountingHole:MountingHole_3.2mm_M3_ISO7380_Pad, F.Cu at (105.0, 55.0)
- added H2: MountingHole_3.2mm_M3_ISO7380_Pad, MountingHole:MountingHole_3.2mm_M3_ISO7380_Pad, F.Cu at (195.0, 55.0)
- added H3: MountingHole_3.2mm_M3_ISO7380_Pad, MountingHole:MountingHole_3.2mm_M3_ISO7380_Pad, F.Cu at (195.0, 115.0)
- added H4: MountingHole_3.2mm_M3_ISO7380_Pad, MountingHole:MountingHole_3.2mm_M3_ISO7380_Pad, F.Cu at (105.0, 115.0)
- TP401, TP402, TP403, TP404, TP405: moved to B.Cu
- moved C301 166.3 mm to (123.0, 264.5), turned to -90 degrees
- moved TP301 165.7 mm to (95.9, 255.0)
- moved TP303 165.7 mm to (95.9, 262.1)
- moved TP304 165.7 mm to (95.9, 265.6)
- moved TP305 165.7 mm to (95.9, 269.2)
- moved TP302 165.7 mm to (95.9, 258.5)
- moved Q751 162.6 mm to (56.5, 34.4)
- moved FB301 158.9 mm to (102.0, 243.5)
- moved C302 157.7 mm to (126.1, 264.5), turned to -90 degrees
- moved R301 156.2 mm to (129.0, 264.5), turned to -90 degrees
- moved R753 154.7 mm to (47.5, 33.6)
- moved D752 153.4 mm to (47.5, 40.1), turned to 90 degrees
- moved R751 153.2 mm to (52.4, 40.9)
- moved D701 152.4 mm to (171.3, 33.0), turned to 180 degrees
- moved Q752 152.0 mm to (46.0, 55.1), turned to 90 degrees
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Connections:
- U1 pad 1: Net-(U1-GND_{1}-Pad1) -> GND_ISO
- U1 pad 10: Net-(U1-GND_{1}-Pad1) -> GND_ISO
- U1 pad 11: Net-(U1-GND_{2}-Pad11) -> GND_CAN
- U1 pad 13: unconnected-(U1-CANL-Pad13) -> /BUS_CAN_L
- U1 pad 14: unconnected-(U1-CANH-Pad14) -> /BUS_CAN_H
- U1 pad 15: Net-(U1-GND_{2}-Pad11) -> GND_CAN
- U1 pad 16: unconnected-(U1-V_{ISOIN}-Pad16) -> /60_can/V_SOIN
- U1 pad 18: Net-(U1-GND_{ISO}-Pad18) -> GND_CAN
- U1 pad 19: unconnected-(U1-V_{ISOOUT}-Pad19) -> /60_can/V_SOOUT
- U1 pad 2: Net-(U1-GND_{1}-Pad1) -> GND_ISO
- U1 pad 20: Net-(U1-GND_{ISO}-Pad18) -> GND_CAN
- U1 pad 3: unconnected-(U1-V_{CC}-Pad3) -> +5V_ISO
- U1 pad 4: unconnected-(U1-V_{IO}-Pad4) -> +3V3_D
- U1 pad 5: unconnected-(U1-RXD-Pad5) -> /CAN_RX
- U1 pad 7: unconnected-(U1-TXD-Pad7) -> /CAN_TX
- U1 pad 8: unconnected-(U1-STBY-Pad8) -> /CAN_STBY
Other:
- board outline added: 100 x 70 mm
