File: INCLI-VA.kicad_pcb (KiCad board)
At the start: 2 copper layers, 100 x 70 mm, 183 parts, among them J1 MSTBV 2,5/5-GF-5,08, J2 MSTBV 2,5/2-GF-5,08, J401 USB4105-GF-A, J402 UART0, Q101 STD18NF25, Q102 IPD30N10S3L-34, Q701 DMN10H220LQ, Q702 BC817-40, Q703 BC807-40, Q751 DMN10H220LQ, Q752 BC817-40, Q753 BC807-40, SW401 RESET, SW402 BOOT, U101 LM74930QRGERQ1, U201 LMR38010SQDDARQ1, U301 TPS62A02QDRLRQ1, U302 LP5907QMFX-3.3Q1, U401 ESP32-S3-WROOM-1-N8R2, U402 USBLC6-2SC6, U501 SCL3300-D01, U502 ASM330LHHTR, U503 AS5147U-HTSM, U601 ADM3055E, U701 74AHCT1G126, U751 74AHCT1G126, U801 TPS3828-33Q1

Commit message: [Codex] Integra cierre de Claude y valida sincronizacion previa al layout
Parts:
- removed D401: PMEG3020EH, Diode_SMD:D_SOD-123F
- removed JP401: BANCO_USB, Jumper:SolderJumper-2_P1.3mm_Open_RoundedPad1.0x1.5mm
- added H1: MountingHole_M3, MountingHole:MountingHole_3.2mm_M3, F.Cu at (220.0, 50.0)
- added H2: MountingHole_M3, MountingHole:MountingHole_3.2mm_M3, F.Cu at (230.0, 50.0)
- added H3: MountingHole_M3, MountingHole:MountingHole_3.2mm_M3, F.Cu at (240.0, 50.0)
- added H4: MountingHole_M3, MountingHole:MountingHole_3.2mm_M3, F.Cu at (250.0, 50.0)
- added H5: MountingHole_M3, MountingHole:MountingHole_3.2mm_M3, F.Cu at (260.0, 50.0)
- C105: value 1000uF -> 1000uF 50V
- F101: footprint INCLI-VA:FUSE-SMD_L6.1-W2.5-1 -> INCLI-VA:Fuse_Bourns_SF-2410
