File: INCLI-VA.kicad_pcb (KiCad board)
At the start: 2 copper layers, 100 x 100 mm, 168 parts, among them J1 MSTBV 2,5/5-GF-5,08, J2 MSTBV 2,5/2-GF-5,08, J401 USB4105-GF-A, J402 UART0, Q101 STD18NF25, Q102 IPD30N10S3L-34, Q701 DMN10H220LQ, Q751 DMN10H220LQ, SW401 RESET, SW402 BOOT, U101 LM74930QRGERQ1, U201 LMR38010SQDDARQ1, U301 TPS62A02QDRLRQ1, U302 LP5907QMFX-3.3Q1, U401 ESP32-S3-WROOM-1-N8R2, U402 USBLC6-2SC6, U501 SCL3300-D01, U502 ASM330LHHTR, U503 AS5147U-HTSM, U601 ADM3055E, U701 74AHCT1G126, U751 74AHCT1G126, U801 TPS3828-33Q1

Commit message: update pcb layout
Parts:
- removed H5: MountingHole_M3, MountingHole:MountingHole_3.2mm_M3
- SW401, SW402: footprint Button_Switch_THT:SW_PUSH_6mm -> easyeda2kicad:SW-SMD_L3.9-W3.0-P4.45
- moved SW401 56.8 mm to (160.8, 145.7), turned to 90 degrees
- moved R103 23.9 mm to (103.4, 89.8), turned to 90 degrees
- moved R112 21.4 mm to (135.9, 93.7), turned to 90 degrees
- moved L101 16.1 mm to (119.1, 55.2)
- moved C105 15.8 mm to (109.9, 71.4), turned to 90 degrees
- moved C109 14.6 mm to (120.4, 77.8)
- moved C107 14.3 mm to (126.5, 57.5), turned to 0 degrees
- moved R304 14.3 mm to (145.0, 146.9), turned to -90 degrees
- moved Q102 14.1 mm to (109.5, 89.6), turned to -90 degrees
- moved C106 13.3 mm to (126.5, 53.4), turned to 0 degrees
- moved R104 13.0 mm to (123.7, 69.1), turned to 180 degrees
- moved R107 11.0 mm to (120.4, 70.9), turned to 90 degrees
- moved C303 9.52 mm to (147.9, 143.5), turned to -90 degrees
- moved R111 9.28 mm to (128.8, 79.6)
- moved C102 9.21 mm to (127.3, 64.5), turned to 90 degrees
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Routing:
- net /BUS_CAN_H: track 0.00 -> 8.22 mm
- net /BUS_CAN_L: track 0.00 -> 8.22 mm
- net /60_can/V_SOIN: track 0.00 -> 5.92 mm
- net /CAN_STBY: track 0.00 -> 5.28 mm
- net /60_can/V_SOOUT: track 0.00 -> 3.48 mm
- net Net-(C609-Pad1): track 0.00 -> 3.28 mm
- net /60_can/CAN_RS: track 0.00 -> 3.09 mm
- net /60_can/GNDISO_CAN: track 0.00 -> 0.59 mm
Other:
- outline, holes or cut-outs redrawn

Commit message: update
Parts:
- moved D801 55.3 mm to (154.6, 53.6), turned to -90 degrees
- moved D802 51.6 mm to (158.1, 53.6), turned to -90 degrees
- moved C403 47.1 mm to (164.6, 146.4), turned to -90 degrees
- moved R401 46.5 mm to (162.0, 146.4), turned to 90 degrees
- moved R804 46.3 mm to (158.1, 57.5), turned to 90 degrees
- moved U801 45.1 mm to (166.1, 136.5)
- moved R803 44.8 mm to (154.6, 57.5)
- moved R802 43.8 mm to (162.6, 136.5)
- moved R801 41.5 mm to (170.3, 137.5), turned to 0 degrees
- moved C801 40.9 mm to (170.3, 135.5), turned to 0 degrees
- moved R402 19.2 mm to (169.8, 147.2), turned to 0 degrees
- moved L201 19.1 mm to (139.4, 55.5), turned to 0 degrees
- moved C204 16.4 mm to (146.4, 53.0), turned to 0 degrees
- moved R805 16.1 mm to (186.6, 103.5), turned to -90 degrees
- moved R806 12.9 mm to (184.7, 103.5), turned to -90 degrees
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Routing:
- net /60_can/V_SOIN: track 5.92 -> 0.00 mm
- net /CAN_STBY: track 5.28 -> 0.00 mm
- net /60_can/V_SOOUT: track 3.48 -> 0.09 mm
- net Net-(C609-Pad1): track 3.28 -> 0.03 mm
- net /60_can/CAN_RS: track 3.09 -> 0.16 mm
