File: INCLI-VA.kicad_pcb (KiCad board)
At the start: 2 copper layers, 100 x 100 mm, 168 parts, among them J1 MSTBV 2,5/5-GF-5,08, J2 MSTBV 2,5/2-GF-5,08, J401 USB4105-GF-A, J402 UART0, Q101 STD18NF25, Q102 IPD30N10S3L-34, Q701 DMN10H220LQ, Q751 DMN10H220LQ, SW401 RESET, SW402 BOOT, U101 LM74930QRGERQ1, U201 LMR38010SQDDARQ1, U301 TPS62A02QDRLRQ1, U302 LP5907QMFX-3.3Q1, U401 ESP32-S3-WROOM-1-N8R2, U402 USBLC6-2SC6, U501 SCL3300-D01, U502 ASM330LHHTR, U503 AS5147U-HTSM, U601 ADM3055E, U701 74AHCT1G126, U751 74AHCT1G126, U801 TPS3828-33Q1

Commit message: update layout position screen
Parts:
- moved C609 2.51 mm to (114.4, 128.5)
- moved R711 0.24 mm to (185.9, 72.3)
- moved C109 0.10 mm to (120.4, 76.6)
- moved R105 0.10 mm to (120.4, 80.7)
- moved R106 0.10 mm to (120.4, 72.6)
- moved R107 0.10 mm to (120.4, 68.5)
Routing:
- net /BUS_CAN_H: track 0.82 -> 0.00 mm
- net /60_can/GNDISO_CAN: track 0.59 -> 0.00 mm
