File: INCLI-VA.kicad_pcb (KiCad board)
At the start: 2 copper layers, 100 x 100 mm, 169 parts, among them J1 MSTBV 2,5/5-GF-5,08, J2 MSTBV 2,5/2-GF-5,08, J401 USB4105-GF-A, J402 UART0, Q101 STD18NF25, Q102 IPD30N10S3L-34, Q701 DMN10H220LQ, Q751 DMN10H220LQ, SW401 RESET, SW402 BOOT, U101 LM74930QRGERQ1, U201 LMR38010SQDDARQ1, U301 TPS62A02QDRLRQ1, U302 LP5907QMFX-3.3Q1, U401 ESP32-S3-WROOM-1-N8R2, U402 USBLC6-2SC6, U501 SCL3300-D01, U502 ASM330LHHTR, U503 AS5147U-HTSM, U601 ADM3055E, U701 74AHCT1G126, U751 74AHCT1G126, U801 TPS3828-33Q1

Commit message: [Claude Code] ruteo etapa 4 parcial: U101, RESET, bus bajo el modulo, DO, supervision
- Perifericos de U101 con los saltos B.Cu reservados; pad 25 RTN intacto.
- RESET: tramo B.Cu movido de bajo las salidas SPI a un carril bajo el modulo
  (autorizado). SW401 68.92 mm, R802 61.59 mm.
- DO1/DO2_EN, DO1/DO2_DIAG, PWR_FLT_N y LED por B.Cu bajo el modulo, con un
  unico cruce del par USB (autorizado). Salidas DO, +5V, LED, VAR_ID, WDI, VMON,
  R305/R307 y PG_3V3D.
- DRC 0 errores, paridad 0, ERC sin cambios, verify_etapa3 OK. Quedan 39
  conexiones de sensores: pendiente reasignar GPIO del SPI (decision del usuario).

Co-Authored-By: Claude Opus 5.5 <noreply@anthropic.com>
Routing:
- net /PWR_FLT_N: track 0.00 -> 112.9 mm, vias 0 -> 6
- net +5V_VEH: track 159.6 -> 262.4 mm, vias 2 -> 6
- net /LED_G: track 0.00 -> 79.1 mm, vias 0 -> 2
- net /LED_R: track 0.00 -> 74.7 mm, vias 0 -> 2
- net /DO2_DIAG: track 0.00 -> 74.0 mm, vias 0 -> 4
- net /DO1_DIAG: track 0.00 -> 73.7 mm, vias 0 -> 2
- net /DO2_EN: track 0.00 -> 65.6 mm, vias 0 -> 2
- net /DO1_EN: track 0.00 -> 65.2 mm, vias 0 -> 2
- net /WDI: track 0.00 -> 56.2 mm, vias 0 -> 4
- net +3V3_D: track 199.1 -> 240.5 mm, vias 8 -> 10
- net /10_power_input/VS: track 0.00 -> 40.3 mm, vias 0 -> 4
- net /10_power_input/OV: track 0.00 -> 33.1 mm, vias 0 -> 2
- net /VEH_DO2: track 0.00 -> 31.0 mm
- net /VEH_DO1: track 0.00 -> 24.3 mm
- net Net-(D704-K): track 0.00 -> 22.1 mm
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
Commit message: [Claude Code] ruteo etapa 4: sensores (opcion C, U503 girado 180), cierre de etapa
- SPI/CS, INT1/INT2, +3V3_A y SCL_AEXTC/DEXTC ruteados con GPIO actuales.
- U503 r180, C501/C502 girados, pasivos y TP501-504 reubicados; referencias de serigrafia.
- 12 cruces B.Cu perpendiculares con costura GND; cruce 12 (3.6 mm) aceptado.
- Tres vias GND en el circulo del iman, tapadas en ambas caras.
- DRC 0 errores, paridad 0, ERC 0 errores, verify_etapa3 OK; 132 pendientes, todas de masa.
- Traspaso y pendientes: cambios de ubicacion, cifra +5V/U503 corregida a 7.6 mm, ZPOS, islas para etapa 5.

Co-Authored-By: Claude Opus 5.5 <noreply@anthropic.com>
Parts:
- moved TP501 22.6 mm to (162.4, 91.0)
- moved TP504 16.0 mm to (170.1, 104.6)
- moved R503 11.3 mm to (151.9, 104.6)
- moved C507 8.71 mm to (145.3, 100.5), turned to -90 degrees
- moved R502 7.64 mm to (171.3, 92.0), turned to -90 degrees
- moved TP502 5.52 mm to (155.8, 108.0)
- moved TP503 4.31 mm to (162.2, 108.2)
- moved C505 4.17 mm to (167.1, 98.0), turned to 0 degrees
- moved C506 3.46 mm to (169.5, 98.2), turned to -90 degrees
- moved R501 1.53 mm to (161.6, 110.4)
- moved C508 1.29 mm to (168.7, 90.3), turned to 180 degrees
- turned C501 to -90 degrees
- turned C502 to -90 degrees
- turned U503 to 180 degrees
Routing:
- net +3V3_A: track 2.56 -> 160.1 mm, vias 0 -> 9
- net /SPI_SCK: track 0.00 -> 72.1 mm, vias 0 -> 3
- net /SPI_MOSI: track 0.00 -> 65.0 mm, vias 0 -> 5
- net /SPI_MISO: track 0.00 -> 63.2 mm, vias 0 -> 3
- net /IMU_INT1: track 0.00 -> 47.7 mm, vias 0 -> 3
- net /IMU_INT2: track 0.00 -> 46.7 mm, vias 0 -> 2
- net /CS_ROT: track 0.00 -> 35.8 mm
- net /CS_IMU: track 0.00 -> 23.9 mm
- net /CS_INC: track 0.00 -> 17.0 mm, vias 0 -> 2
- net GND_VEH: track 72.0 -> 83.2 mm, vias 50 -> 76
- net /50_sensors/SCL_DEXTC: track 0.00 -> 3.30 mm
- net /50_sensors/SCL_AEXTC: track 0.00 -> 1.98 mm
