File: INCLI-VA.kicad_sch (KiCad schematic)
At the start: 5 parts

Commit message: update pcb layout
Parts:
- removed H5: MountingHole_M3, MountingHole:MountingHole_3.2mm_M3, symbol Mechanical:MountingHole
Other:
- note added: "AGUJEROS DE FIJACION: H1-H4, 4 agujeros M3 sin cobre: H1-H4 en las esquinas, fuera del eje de ROT (en el esquematico para que 'Update PCB from Schematic' no los borre)."
- note removed: "AGUJEROS DE FIJACION: H1-H5, cinco agujeros M3 sin cobre: H1-H4 en las esquinas y H5 intermedio junto a los sensores, fuera del eje de ROT (en el esquematico para que 'Update PCB from Schematic' no los borre)."
