File: docs/layout/INCLI-VA-100x100.kicad_pcb (KiCad board)
At the start: 2 copper layers, 100 x 100 mm, 186 parts, among them J1 MSTBV 2,5/5-GF-5,08, J2 MSTBV 2,5/2-GF-5,08, J401 USB4105-GF-A, J402 UART0, Q101 STD18NF25, Q102 IPD30N10S3L-34, Q701 DMN10H220LQ, Q702 BC817-40, Q703 BC807-40, Q751 DMN10H220LQ, Q752 BC817-40, Q753 BC807-40, SW401 RESET, SW402 BOOT, U101 LM74930QRGERQ1, U201 LMR38010SQDDARQ1, U301 TPS62A02QDRLRQ1, U302 LP5907QMFX-3.3Q1, U401 ESP32-S3-WROOM-1-N8R2, U402 USBLC6-2SC6, U501 SCL3300-D01, U502 ASM330LHHTR, U503 AS5147U-HTSM, U601 ADM3055E, U701 74AHCT1G126, U751 74AHCT1G126, U801 TPS3828-33Q1

Commit message: [Codex] Pasa TP a Bottom y deja cuatro fijaciones en propuesta 100x100
Parts:
- removed H5: MountingHole_M3, MountingHole:MountingHole_3.2mm_M3
- TP101, TP102, TP103, TP104, TP201, TP301, TP302, TP303, TP304, TP305, TP501, TP502, TP503, TP504: moved to B.Cu
- turned TP101 to 180 degrees
- turned TP102 to 180 degrees
- turned TP103 to 180 degrees
- turned TP104 to 180 degrees
- turned TP201 to 180 degrees
- turned TP301 to 180 degrees
- turned TP302 to 180 degrees
- turned TP303 to 180 degrees
- turned TP304 to 180 degrees
- turned TP305 to 180 degrees
- turned TP501 to 180 degrees
- turned TP502 to 180 degrees
- turned TP503 to 180 degrees
- turned TP504 to 180 degrees
